Commit message: Unify use of arm_id (arm.xacro) and ns (hand.xacro) to prefix
IMO, prefix much better describes the purpose of these two variables
in the present context, namely providing a name prefix to joints and links.

File: franka_description/robots/arm.xacro (robot description, xacro)
@@ -2,14 +2,14 @@
 <robot xmlns:xacro="http://www.ros.org/wiki/xacro" name="panda">
   <!-- safety_distance: Minimum safety distance in [m] by which the collision volumes are expanded and which is enforced during robot motions -->
-  <!-- arm_id: Namespace of the panda arm. Serves to differentiate between arms in case of multiple instances. -->
-  <xacro:macro name="arm" params="arm_id:='panda' description_pkg:='franka_description' connected_to:='' xyz:='0 0 0' rpy:='0 0 0' safety_distance:=0">
+  <!-- prefix: used for joint and link names. Needed to distinguish joints and TFs in case of multiple arm instances. -->
+  <xacro:macro name="arm" params="prefix:=^| description_pkg:='franka_description' connected_to:='' xyz:='0 0 0' rpy:='0 0 0' safety_distance:=0">
     <xacro:unless value="${not connected_to}">
-      <joint name="${arm_id}_joint_${connected_to}" type="fixed">
+      <joint name="${prefix}joint_${connected_to}" type="fixed">
         <parent link="${connected_to}"/>
-        <child link="${arm_id}_link0"/>
+        <child link="${prefix}link0"/>
         <origin rpy="${rpy}" xyz="${xyz}"/>
       </joint>
     </xacro:unless>
-    <link name="${arm_id}_link0">
+    <link name="${prefix}link0">
       <visual>
         <geometry>
@@ -36,5 +36,5 @@
       </collision>
     </link>
-    <link name="${arm_id}_link1">
+    <link name="${prefix}link1">
       <visual>
         <geometry>
@@ -61,13 +61,13 @@
       </collision>
     </link>
-    <joint name="${arm_id}_joint1" type="revolute">
+    <joint name="${prefix}joint1" type="revolute">
       <safety_controller k_position="100.0" k_velocity="40.0" soft_lower_limit="-2.8973" soft_upper_limit="2.8973"/>
       <origin rpy="0 0 0" xyz="0 0 0.333"/>
-      <parent link="${arm_id}_link0"/>
-      <child link="${arm_id}_link1"/>
+      <parent link="${prefix}link0"/>
+      <child link="${prefix}link1"/>
       <axis xyz="0 0 1"/>
       <limit effort="87" lower="-2.8973" upper="2.8973" velocity="2.1750"/>
     </joint>
-    <link name="${arm_id}_link2">
+    <link name="${prefix}link2">
       <visual>
         <geometry>
@@ -94,13 +94,13 @@
       </collision>
     </link>
-    <joint name="${arm_id}_joint2" type="revolute">
+    <joint name="${prefix}joint2" type="revolute">
       <safety_controller k_position="100.0" k_velocity="40.0" soft_lower_limit="-1.7628" soft_upper_limit="1.7628"/>
       <origin rpy="${-pi/2} 0 0" xyz="0 0 0"/>
-      <parent link="${arm_id}_link1"/>
-      <child link="${arm_id}_link2"/>
+      <parent link="${prefix}link1"/>
+      <child link="${prefix}link2"/>
       <axis xyz="0 0 1"/>
       <limit effort="87" lower="-1.7628" upper="1.7628" velocity="2.1750"/>
     </joint>
-    <link name="${arm_id}_link3">
+    <link name="${prefix}link3">
       <visual>
         <geometry>
@@ -127,13 +127,13 @@
       </collision>
     </link>
-    <joint name="${arm_id}_joint3" type="revolute">
+    <joint name="${prefix}joint3" type="revolute">
       <safety_controller k_position="100.0" k_velocity="40.0" soft_lower_limit="-2.8973" soft_upper_limit="2.8973"/>
       <origin rpy="${pi/2} 0 0" xyz="0 -0.316 0"/>
-      <parent link="${arm_id}_link2"/>
-      <child link="${arm_id}_link3"/>
+      <parent link="${prefix}link2"/>
+      <child link="${prefix}link3"/>
       <axis xyz="0 0 1"/>
       <limit effort="87" lower="-2.8973" upper="2.8973" velocity="2.1750"/>
     </joint>
-    <link name="${arm_id}_link4">
+    <link name="${prefix}link4">
       <visual>
         <geometry>
@@ -160,13 +160,13 @@
       </collision>
     </link>
-    <joint name="${arm_id}_joint4" type="revolute">
+    <joint name="${prefix}joint4" type="revolute">
       <safety_controller k_position="100.0" k_velocity="40.0" soft_lower_limit="-3.0718" soft_upper_limit="-0.0698"/>
       <origin rpy="${pi/2} 0 0" xyz="0.0825 0 0"/>
-      <parent link="${arm_id}_link3"/>
-      <child link="${arm_id}_link4"/>
+      <parent link="${prefix}link3"/>
+      <child link="${prefix}link4"/>
       <axis xyz="0 0 1"/>
       <limit effort="87" lower="-3.0718" upper="-0.0698" velocity="2.1750"/>
     </joint>
-    <link name="${arm_id}_link5">
+    <link name="${prefix}link5">
       <visual>
         <geometry>
@@ -211,13 +211,13 @@
       </collision>
     </link>
-    <joint name="${arm_id}_joint5" type="revolute">
+    <joint name="${prefix}joint5" type="revolute">
       <safety_controller k_position="100.0" k_velocity="40.0" soft_lower_limit="-2.8973" soft_upper_limit="2.8973"/>
       <origin rpy="${-pi/2} 0 0" xyz="-0.0825 0.384 0"/>
-      <parent link="${arm_id}_link4"/>
-      <child link="${arm_id}_link5"/>
+      <parent link="${prefix}link4"/>
+      <child link="${prefix}link5"/>
       <axis xyz="0 0 1"/>
       <limit effort="12" lower="-2.8973" upper="2.8973" velocity="2.6100"/>
     </joint>
-    <link name="${arm_id}_link6">
+    <link name="${prefix}link6">
       <visual>
         <geometry>
@@ -244,13 +244,13 @@
       </collision>
     </link>
-    <joint name="${arm_id}_joint6" type="revolute">
+    <joint name="${prefix}joint6" type="revolute">
       <safety_controller k_position="100.0" k_velocity="40.0" soft_lower_limit="-0.0175" soft_upper_limit="3.7525"/>
       <origin rpy="${pi/2} 0 0" xyz="0 0 0"/>
-      <parent link="${arm_id}_link5"/>
-      <child link="${arm_id}_link6"/>
+      <parent link="${prefix}link5"/>
+      <child link="${prefix}link6"/>
       <axis xyz="0 0 1"/>
       <limit effort="12" lower="-0.0175" upper="3.7525" velocity="2.6100"/>
     </joint>
-    <link name="${arm_id}_link7">
+    <link name="${prefix}link7">
       <visual>
         <geometry>
@@ -277,13 +277,13 @@
       </collision>
     </link>
-    <joint name="${arm_id}_joint7" type="revolute">
+    <joint name="${prefix}joint7" type="revolute">
       <safety_controller k_position="100.0" k_velocity="40.0" soft_lower_limit="-2.8973" soft_upper_limit="2.8973"/>
       <origin rpy="${pi/2} 0 0" xyz="0.088 0 0"/>
-      <parent link="${arm_id}_link6"/>
-      <child link="${arm_id}_link7"/>
+      <parent link="${prefix}link6"/>
+      <child link="${prefix}link7"/>
       <axis xyz="0 0 1"/>
       <limit effort="12" lower="-2.8973" upper="2.8973" velocity="2.6100"/>
     </joint>
-    <link name="${arm_id}_link8">
+    <link name="${prefix}link8">
       <collision>
         <origin xyz="0.0424 0.0424 -0.0250" rpy="${pi} ${pi/2} ${pi/2}"/>
@@ -305,8 +305,8 @@
       </collision>
     </link>
-    <joint name="${arm_id}_joint8" type="fixed">
+    <joint name="${prefix}joint8" type="fixed">
       <origin rpy="0 0 0" xyz="0 0 0.107"/>
-      <parent link="${arm_id}_link7"/>
-      <child link="${arm_id}_link8"/>
+      <parent link="${prefix}link7"/>
+      <child link="${prefix}link8"/>
     </joint>
   </xacro:macro>

File: franka_description/robots/dual_panda_example.urdf.xacro (robot description, xacro)
@@ -24,8 +24,8 @@
   </link>
   <!-- right arm with gripper -->
-  <xacro:arm arm_id="$(arg arm_id_1)" connected_to="base"  xyz="0 -0.5 1" safety_distance="0.03"/>
-  <xacro:hand ns="$(arg arm_id_1)" rpy="0 0 ${-pi/4}" connected_to="$(arg arm_id_1)_link8" safety_distance="0.03"/>
+  <xacro:arm prefix="$(arg arm_id_1)" connected_to="base"  xyz="0 -0.5 1" safety_distance="0.03"/>
+  <xacro:hand prefix="$(arg arm_id_1)" rpy="0 0 ${-pi/4}" connected_to="$(arg arm_id_1)_link8" safety_distance="0.03"/>
   <!-- left arm with gripper -->
-  <xacro:arm arm_id="$(arg arm_id_2)" connected_to="base"  xyz="0 0.5 1" safety_distance="0.03"/>
-  <xacro:hand ns="$(arg arm_id_2)" rpy="0 0 ${-pi/4}" connected_to="$(arg arm_id_2)_link8" safety_distance="0.03"/>
+  <xacro:arm prefix="$(arg arm_id_2)" connected_to="base"  xyz="0 0.5 1" safety_distance="0.03"/>
+  <xacro:hand prefix="$(arg arm_id_2)" rpy="0 0 ${-pi/4}" connected_to="$(arg arm_id_2)_link8" safety_distance="0.03"/>
 </robot>

File: franka_description/robots/hand.urdf.xacro (robot description, xacro)
@@ -2,4 +2,4 @@
 <robot xmlns:xacro="http://www.ros.org/wiki/xacro" name="hand">
   <xacro:include filename="hand.xacro"/>
-  <xacro:hand ns="panda" safety_distance="0.03"/>
+  <xacro:hand prefix="panda_" safety_distance="0.03" />
 </robot>

File: franka_description/robots/hand.xacro (robot description, xacro)
@@ -2,13 +2,14 @@
 <robot xmlns:xacro="http://www.ros.org/wiki/xacro" name="hand">
   <!-- safety_distance: Minimum safety distance in [m] by which the collision volumes are expanded and which is enforced during robot motions -->
-  <xacro:macro name="hand" params="connected_to:='' ns:='' rpy:='0 0 0' xyz:='0 0 0' safety_distance:=0">
+  <!-- prefix: used for joint and link names. Needed to distinguish joints and TFs in case of multiple arm instances. -->
+  <xacro:macro name="hand" params="connected_to:='' prefix:=^| rpy:='0 0 0' xyz:='0 0 0' safety_distance:=0">
     <xacro:unless value="${connected_to == ''}">
-      <joint name="${ns}_hand_joint" type="fixed">
+      <joint name="${prefix}hand_joint" type="fixed">
         <parent link="${connected_to}"/>
-        <child link="${ns}_hand"/>
+        <child link="${prefix}hand"/>
         <origin xyz="${xyz}" rpy="${rpy}"/>
       </joint>
     </xacro:unless>
-    <link name="${ns}_hand">
+    <link name="${prefix}hand">
       <visual>
         <geometry>
@@ -53,5 +54,5 @@
       </collision>
     </link>
-    <link name="${ns}_leftfinger">
+    <link name="${prefix}leftfinger">
       <visual>
         <geometry>
@@ -60,5 +61,5 @@
       </visual>
     </link>
-    <link name="${ns}_rightfinger">
+    <link name="${prefix}rightfinger">
       <visual>
         <origin xyz="0 0 0" rpy="0 0 ${pi}"/>
@@ -68,18 +69,18 @@
       </visual>
    </link>
-    <joint name="${ns}_finger_joint1" type="prismatic">
-      <parent link="${ns}_hand"/>
-      <child link="${ns}_leftfinger"/>
+    <joint name="${prefix}finger_joint1" type="prismatic">
+      <parent link="${prefix}hand"/>
+      <child link="${prefix}leftfinger"/>
       <origin xyz="0 0 0.0584" rpy="0 0 0"/>
       <axis xyz="0 1 0"/>
       <limit effort="20" lower="0.0" upper="0.04" velocity="0.2"/>
     </joint>
-    <joint name="${ns}_finger_joint2" type="prismatic">
-      <parent link="${ns}_hand"/>
-      <child link="${ns}_rightfinger"/>
+    <joint name="${prefix}finger_joint2" type="prismatic">
+      <parent link="${prefix}hand"/>
+      <child link="${prefix}rightfinger"/>
       <origin xyz="0 0 0.0584" rpy="0 0 0"/>
       <axis xyz="0 -1 0"/>
       <limit effort="20" lower="0.0" upper="0.04" velocity="0.2"/>
-      <mimic joint="${ns}_finger_joint1" />
+      <mimic joint="${prefix}finger_joint1" />
     </joint>
   </xacro:macro>

File: franka_description/robots/panda_arm.urdf.xacro (robot description, xacro)
@@ -7,11 +7,13 @@
   <!-- Is the robot being simulated in gazebo?" -->
   <xacro:arg name="gazebo" default="false" />
+  <!-- Name prefix used for joints and links. Property is implicitly passed to macros. -->
+  <xacro:property name="prefix" value="$(arg arm_id)_" />
   <xacro:unless value="$(arg gazebo)">
     <!-- Create a URDF for a real hardware -->
     <xacro:include filename="$(find franka_description)/robots/arm.xacro" />
-    <xacro:arm arm_id="$(arg arm_id)" safety_distance="0.03" />
+    <xacro:arm safety_distance="0.03" />
     <xacro:if value="$(arg hand)">
       <xacro:include filename="$(find franka_description)/robots/hand.xacro"/>
-      <xacro:hand ns="$(arg arm_id)" rpy="0 0 ${-pi/4}" connected_to="$(arg arm_id)_link8" safety_distance="0.03"/>
+      <xacro:hand rpy="0 0 ${-pi/4}" connected_to="${prefix}link8" safety_distance="0.03"/>
     </xacro:if>
   </xacro:unless>
@@ -22,9 +24,9 @@
     <xacro:include filename="$(find franka_description)/robots/utils.xacro" />
     <xacro:include filename="$(find franka_description)/robots/panda_gazebo.xacro" />
-    <xacro:arm arm_id="$(arg arm_id)" />
+    <xacro:arm />
     <xacro:if value="$(arg hand)">
-      <xacro:hand ns="$(arg arm_id)" rpy="0 0 ${-pi/4}" connected_to="$(arg arm_id)_link8" />
-      <xacro:gazebo-joint joint="$(arg arm_id)_finger_joint1" transmission="hardware_interface/EffortJointInterface" />
-      <xacro:gazebo-joint joint="$(arg arm_id)_finger_joint2" transmission="hardware_interface/EffortJointInterface" />
+      <xacro:hand rpy="0 0 ${-pi/4}" connected_to="${prefix}link8" />
+      <xacro:gazebo-joint joint="${prefix}finger_joint1" transmission="hardware_interface/EffortJointInterface" />
+      <xacro:gazebo-joint joint="${prefix}finger_joint2" transmission="hardware_interface/EffortJointInterface" />
     </xacro:if>
     <!-- Gazebo requires a joint to a link called "world" for statically mounted robots -->
@@ -33,18 +35,15 @@
       <origin xyz="$(arg xyz)" rpy="$(arg rpy)" />
       <parent link="world" />
-      <child  link="$(arg arm_id)_link0" />
+      <child  link="${prefix}link0" />
     </joint>
-    <xacro:gazebo-joint joint="$(arg arm_id)_joint1" transmission="hardware_interface/EffortJointInterface" />
-    <xacro:gazebo-joint joint="$(arg arm_id)_joint2" transmission="hardware_interface/EffortJointInterface" />
-    <xacro:gazebo-joint joint="$(arg arm_id)_joint3" transmission="hardware_interface/EffortJointInterface" />
-    <xacro:gazebo-joint joint="$(arg arm_id)_joint4" transmission="hardware_interface/EffortJointInterface" />
-    <xacro:gazebo-joint joint="$(arg arm_id)_joint5" transmission="hardware_interface/EffortJointInterface" />
-    <xacro:gazebo-joint joint="$(arg arm_id)_joint6" transmission="hardware_interface/EffortJointInterface" />
-    <xacro:gazebo-joint joint="$(arg arm_id)_joint7" transmission="hardware_interface/EffortJointInterface" />
-    <xacro:transmission-franka-state arm_id="$(arg arm_id)" />
-    <xacro:transmission-franka-model arm_id="$(arg arm_id)"
-       root="$(arg arm_id)_joint1"
-       tip="$(arg arm_id)_joint8"
-     />
+    <xacro:gazebo-joint joint="${prefix}joint1" transmission="hardware_interface/EffortJointInterface" />
+    <xacro:gazebo-joint joint="${prefix}joint2" transmission="hardware_interface/EffortJointInterface" />
+    <xacro:gazebo-joint joint="${prefix}joint3" transmission="hardware_interface/EffortJointInterface" />
+    <xacro:gazebo-joint joint="${prefix}joint4" transmission="hardware_interface/EffortJointInterface" />
+    <xacro:gazebo-joint joint="${prefix}joint5" transmission="hardware_interface/EffortJointInterface" />
+    <xacro:gazebo-joint joint="${prefix}joint6" transmission="hardware_interface/EffortJointInterface" />
+    <xacro:gazebo-joint joint="${prefix}joint7" transmission="hardware_interface/EffortJointInterface" />
+    <xacro:transmission-franka-state />
+    <xacro:transmission-franka-model root="${prefix}joint1" tip="${prefix}joint8" />
     <gazebo>
       <plugin name="gazebo_ros_control" filename="libgazebo_ros_control.so">

File: franka_description/robots/panda_gazebo.xacro (robot description, xacro)
@@ -10,6 +10,6 @@
   <!-- || Paolo Robuffo Giordano, Alessandro de Luca                || -->
   <!-- =============================================================== -->
-  <xacro:macro name="arm" params="arm_id:='panda'">
-    <link name="${arm_id}_link0">
+  <xacro:macro name="arm" params="prefix:=^|">
+    <link name="${prefix}link0">
       <visual>
         <origin rpy="0 0 0" xyz="0 0 0"/>
@@ -33,5 +33,5 @@
       </inertial>
     </link>
-    <link name="${arm_id}_link1">
+    <link name="${prefix}link1">
       <visual>
         <origin rpy="0 0 0" xyz="0 0 0"/>
@@ -54,14 +54,14 @@
       </inertial>
     </link>
-    <joint name="${arm_id}_joint1" type="revolute">
+    <joint name="${prefix}joint1" type="revolute">
       <safety_controller k_position="100.0" k_velocity="40.0" soft_lower_limit="-2.8973" soft_upper_limit="2.8973"/>
       <origin rpy="0 0 0" xyz="0 0 0.333"/>
-      <parent link="${arm_id}_link0"/>
-      <child link="${arm_id}_link1"/>
+      <parent link="${prefix}link0"/>
+      <child link="${prefix}link1"/>
       <axis xyz="0 0 1"/>
       <limit acceleration="15" lower="-2.9671" effort="87" upper="2.9671" velocity="2.5"/>
       <dynamics D="1" K="7000" mu_coulomb="0" mu_viscous="16" damping="0.003" friction="0.0"/>
     </joint>
-    <link name="${arm_id}_link2">
+    <link name="${prefix}link2">
       <visual>
         <origin rpy="0 0 0" xyz="0 0 0"/>
@@ -84,14 +84,14 @@
       </inertial>
     </link>
-    <joint name="${arm_id}_joint2" type="revolute">
+    <joint name="${prefix}joint2" type="revolute">
       <safety_controller k_position="100.0" k_velocity="40.0" soft_lower_limit="-1.7628" soft_upper_limit="1.7628"/>
       <origin rpy="${-pi/2} 0 0" xyz="0 0 0"/>
-      <parent link="${arm_id}_link1"/>
-      <child link="${arm_id}_link2"/>
+      <parent link="${prefix}link1"/>
+      <child link="${prefix}link2"/>
       <axis xyz="0 0 1"/>
       <limit acceleration="7.5" lower="-1.8326" effort="87" upper="1.8326" velocity="2.5"/>
       <dynamics D="1" K="7000" mu_coulomb="0" mu_viscous="16" damping="0.003" friction="0.0"/>
     </joint>
-    <link name="${arm_id}_link3">
+    <link name="${prefix}link3">
       <visual>
         <origin rpy="0 0 0" xyz="0 0 0"/>
@@ -114,14 +114,14 @@
       </inertial>
     </link>
-    <joint name="${arm_id}_joint3" type="revolute">
+    <joint name="${prefix}joint3" type="revolute">
       <safety_controller k_position="100.0" k_velocity="40.0" soft_lower_limit="-2.8973" soft_upper_limit="2.8973"/>
       <origin rpy="${pi/2} 0 0" xyz="0 -0.316 0"/>
-      <parent link="${arm_id}_link2"/>
-      <child link="${arm_id}_link3"/>
+      <parent link="${prefix}link2"/>
+      <child link="${prefix}link3"/>
       <axis xyz="0 0 1"/>
       <limit acceleration="12.5" lower="-2.9671" effort="87" upper="2.9671" velocity="2.5"/>
       <dynamics D="1" K="7000" mu_coulomb="0" mu_viscous="16" damping="0.003" friction="0.0"/>
     </joint>
-    <link name="${arm_id}_link4">
+    <link name="${prefix}link4">
       <visual>
         <origin rpy="0 0 0" xyz="0 0 0"/>
@@ -144,14 +144,14 @@
       </inertial>
     </link>
-    <joint name="${arm_id}_joint4" type="revolute">
+    <joint name="${prefix}joint4" type="revolute">
       <safety_controller k_position="100.0" k_velocity="40.0" soft_lower_limit="-3.0718" soft_upper_limit="-0.0698"/>
       <origin rpy="${pi/2} 0 0" xyz="0.0825 0 0"/>
-      <parent link="${arm_id}_link3"/>
-      <child link="${arm_id}_link4"/>
+      <parent link="${prefix}link3"/>
+      <child link="${prefix}link4"/>
       <axis xyz="0 0 1"/>
       <limit acceleration="12.5" lower="-3.1416" effort="87" upper="-0.4" velocity="2.5"/>
       <dynamics D="1" K="7000" mu_coulomb="0" mu_viscous="16" damping="0.003" friction="0.0"/>
     </joint>
-    <link name="${arm_id}_link5">
+    <link name="${prefix}link5">
       <visual>
         <origin rpy="0 0 0" xyz="0 0 0"/>
@@ -174,14 +174,14 @@
       </inertial>
     </link>
-    <joint name="${arm_id}_joint5" type="revolute">
+    <joint name="${prefix}joint5" type="revolute">
       <safety_controller k_position="100.0" k_velocity="40.0" soft_lower_limit="-2.8973" soft_upper_limit="2.8973"/>
       <origin rpy="${-pi/2} 0 0" xyz="-0.0825 0.384 0"/>
-      <parent link="${arm_id}_link4"/>
-      <child link="${arm_id}_link5"/>
+      <parent link="${prefix}link4"/>
+      <child link="${prefix}link5"/>
       <axis xyz="0 0 1"/>
       <limit acceleration="15" lower="-2.9671" effort="12" upper="2.9671" velocity="3"/>
       <dynamics D="1" K="7000" mu_coulomb="0" mu_viscous="16" damping="0.003" friction="0.0"/>
     </joint>
-    <link name="${arm_id}_link6">
+    <link name="${prefix}link6">
       <visual>
         <origin rpy="0 0 0" xyz="0 0 0"/>
@@ -204,14 +204,14 @@
       </inertial>
     </link>
-    <joint name="${arm_id}_joint6" type="revolute">
+    <joint name="${prefix}joint6" type="revolute">
       <safety_controller k_position="100.0" k_velocity="40.0" soft_lower_limit="-0.0175" soft_upper_limit="3.7525"/>
       <origin rpy="${pi/2} 0 0" xyz="0 0 0"/>
-      <parent link="${arm_id}_link5"/>
-      <child link="${arm_id}_link6"/>
+      <parent link="${prefix}link5"/>
+      <child link="${prefix}link6"/>
       <axis xyz="0 0 1"/>
       <limit acceleration="20" lower="-0.0873" effort="12" upper="3.8223" velocity="3"/>
       <dynamics D="1" K="7000" mu_coulomb="0" mu_viscous="16" damping="0.003" friction="0.0"/>
     </joint>
-    <link name="${arm_id}_link7">
+    <link name="${prefix}link7">
       <visual>
         <origin rpy="0 0 0" xyz="0 0 0"/>
@@ -234,18 +234,18 @@
       </inertial>
     </link>
-    <joint name="${arm_id}_joint7" type="revolute">
+    <joint name="${prefix}joint7" type="revolute">
       <safety_controller k_position="100.0" k_velocity="40.0" soft_lower_limit="-2.8973" soft_upper_limit="2.8973"/>
       <origin rpy="${pi/2} 0 0" xyz="0.088 0 0"/>
-      <parent link="${arm_id}_link6"/>
-      <child link="${arm_id}_link7"/>
+      <parent link="${prefix}link6"/>
+      <child link="${prefix}link7"/>
       <axis xyz="0 0 1"/>
       <limit acceleration="20" lower="-2.9671" effort="12" upper="2.9671" velocity="3"/>
       <dynamics D="1" K="7000" mu_coulomb="0" mu_viscous="16" damping="0.003" friction="0.0"/>
     </joint>
-    <link name="${arm_id}_link8" />
-    <joint name="${arm_id}_joint8" type="fixed">
+    <link name="${prefix}link8" />
+    <joint name="${prefix}joint8" type="fixed">
       <origin rpy="0 0 0" xyz="0 0 0.107"/>
-      <parent link="${arm_id}_link7"/>
-      <child link="${arm_id}_link8"/>
+      <parent link="${prefix}link7"/>
+      <child link="${prefix}link8"/>
       <axis xyz="0 0 0"/>
     </joint>
