Commit message: Unify use of arm_id (arm.xacro) and ns (hand.xacro) to prefix
IMO, prefix much better describes the purpose of these two variables
in the present context, namely providing a name prefix to joints and links.

File: franka_description/robots/utils.xacro (robot description, xacro)
@@ -51,23 +51,23 @@
   <!-- when simulating with franka_hw_sim plugin                  -->
   <!--                                                            -->
-  <!-- arm_id - Arm ID of the panda to simulate (default 'panda') -->
+  <!-- prefix - prefix used for joint and link names              -->
   <!-- ========================================================== -->
-  <xacro:macro name="transmission-franka-state" params="arm_id:=panda">
-    <transmission name="${arm_id}_franka_state">
+  <xacro:macro name="transmission-franka-state" params="prefix:=^|">
+    <transmission name="${prefix}franka_state">
       <type>franka_hw/FrankaStateInterface</type>
-      <joint name="${arm_id}_joint1"><hardwareInterface>franka_hw/FrankaStateInterface</hardwareInterface></joint>
-      <joint name="${arm_id}_joint2"><hardwareInterface>franka_hw/FrankaStateInterface</hardwareInterface></joint>
-      <joint name="${arm_id}_joint3"><hardwareInterface>franka_hw/FrankaStateInterface</hardwareInterface></joint>
-      <joint name="${arm_id}_joint4"><hardwareInterface>franka_hw/FrankaStateInterface</hardwareInterface></joint>
-      <joint name="${arm_id}_joint5"><hardwareInterface>franka_hw/FrankaStateInterface</hardwareInterface></joint>
-      <joint name="${arm_id}_joint6"><hardwareInterface>franka_hw/FrankaStateInterface</hardwareInterface></joint>
-      <joint name="${arm_id}_joint7"><hardwareInterface>franka_hw/FrankaStateInterface</hardwareInterface></joint>
-      <actuator name="${arm_id}_motor1"><hardwareInterface>franka_hw/FrankaStateInterface</hardwareInterface></actuator>
-      <actuator name="${arm_id}_motor2"><hardwareInterface>franka_hw/FrankaStateInterface</hardwareInterface></actuator>
-      <actuator name="${arm_id}_motor3"><hardwareInterface>franka_hw/FrankaStateInterface</hardwareInterface></actuator>
-      <actuator name="${arm_id}_motor4"><hardwareInterface>franka_hw/FrankaStateInterface</hardwareInterface></actuator>
-      <actuator name="${arm_id}_motor5"><hardwareInterface>franka_hw/FrankaStateInterface</hardwareInterface></actuator>
-      <actuator name="${arm_id}_motor6"><hardwareInterface>franka_hw/FrankaStateInterface</hardwareInterface></actuator>
-      <actuator name="${arm_id}_motor7"><hardwareInterface>franka_hw/FrankaStateInterface</hardwareInterface></actuator>
+      <joint name="${prefix}joint1"><hardwareInterface>franka_hw/FrankaStateInterface</hardwareInterface></joint>
+      <joint name="${prefix}joint2"><hardwareInterface>franka_hw/FrankaStateInterface</hardwareInterface></joint>
+      <joint name="${prefix}joint3"><hardwareInterface>franka_hw/FrankaStateInterface</hardwareInterface></joint>
+      <joint name="${prefix}joint4"><hardwareInterface>franka_hw/FrankaStateInterface</hardwareInterface></joint>
+      <joint name="${prefix}joint5"><hardwareInterface>franka_hw/FrankaStateInterface</hardwareInterface></joint>
+      <joint name="${prefix}joint6"><hardwareInterface>franka_hw/FrankaStateInterface</hardwareInterface></joint>
+      <joint name="${prefix}joint7"><hardwareInterface>franka_hw/FrankaStateInterface</hardwareInterface></joint>
+      <actuator name="${prefix}motor1"><hardwareInterface>franka_hw/FrankaStateInterface</hardwareInterface></actuator>
+      <actuator name="${prefix}motor2"><hardwareInterface>franka_hw/FrankaStateInterface</hardwareInterface></actuator>
+      <actuator name="${prefix}motor3"><hardwareInterface>franka_hw/FrankaStateInterface</hardwareInterface></actuator>
+      <actuator name="${prefix}motor4"><hardwareInterface>franka_hw/FrankaStateInterface</hardwareInterface></actuator>
+      <actuator name="${prefix}motor5"><hardwareInterface>franka_hw/FrankaStateInterface</hardwareInterface></actuator>
+      <actuator name="${prefix}motor6"><hardwareInterface>franka_hw/FrankaStateInterface</hardwareInterface></actuator>
+      <actuator name="${prefix}motor7"><hardwareInterface>franka_hw/FrankaStateInterface</hardwareInterface></actuator>
     </transmission>
   </xacro:macro>
@@ -76,10 +76,10 @@
   <!-- when simulating with franka_hw_sim plugin                    -->
   <!--                                                              -->
-  <!-- arm_id - Arm ID of the panda to simulate (default 'panda')   -->
+  <!-- prefix - prefix for joint and link names                     -->
   <!-- root   - Joint name of the base of the robot                 -->
   <!-- tip    - Joint name of the tip of the robot (flange or hand) -->
   <!-- ============================================================ -->
-  <xacro:macro name="transmission-franka-model" params="arm_id:=panda root:=panda_joint1 tip:=panda_joint7">
-    <transmission name="${arm_id}_franka_model">
+  <xacro:macro name="transmission-franka-model" params="root tip prefix:=^|">
+    <transmission name="${prefix}franka_model">
       <type>franka_hw/FrankaModelInterface</type>
       <joint name="${root}">

Commit message: Use both, detailed meshes and coarse collision geometries
They serve different purposes:
- coarse collision geometries mimic the internal self-collision checking
  of the real-robot controller
- mesh models should be use for collision checking with environmental objects

File: franka_description/robots/arm.xacro (robot description, xacro)
@@ -3,5 +3,5 @@
   <!-- safety_distance: Minimum safety distance in [m] by which the collision volumes are expanded and which is enforced during robot motions -->
   <!-- prefix: used for joint and link names. Needed to distinguish joints and TFs in case of multiple arm instances. -->
-  <xacro:macro name="arm" params="prefix:=^| description_pkg:='franka_description' connected_to:='' xyz:='0 0 0' rpy:='0 0 0' safety_distance:=0">
+  <xacro:macro name="arm" params="prefix:=^| connected_to:='' xyz:='0 0 0' rpy:='0 0 0' safety_distance:=0 description_pkg:=franka_description">
     <xacro:unless value="${not connected_to}">
       <joint name="${prefix}joint_${connected_to}" type="fixed">
@@ -11,10 +11,6 @@
       </joint>
     </xacro:unless>
-    <link name="${prefix}link0">
-      <visual>
-        <geometry>
-          <mesh filename="package://${description_pkg}/meshes/visual/link0.dae"/>
-        </geometry>
-      </visual>
+    <xacro:link name="link0">
+      <self_collision_geometries>
       <collision>
         <origin xyz="-0.075 0 0.06" rpy="0 ${pi/2} 0"/>
@@ -35,11 +31,8 @@
         </geometry>
       </collision>
-    </link>
-    <link name="${prefix}link1">
-      <visual>
-        <geometry>
-          <mesh filename="package://${description_pkg}/meshes/visual/link1.dae"/>
-        </geometry>
-      </visual>
+      </self_collision_geometries>
+    </xacro:link>
+    <xacro:link name="link1">
+      <self_collision_geometries>
       <collision>
         <origin xyz="0 0 -0.1915" rpy="0 0 0"/>
@@ -60,5 +53,6 @@
         </geometry>
       </collision>
-    </link>
+      </self_collision_geometries>
+    </xacro:link>
     <joint name="${prefix}joint1" type="revolute">
       <safety_controller k_position="100.0" k_velocity="40.0" soft_lower_limit="-2.8973" soft_upper_limit="2.8973"/>
@@ -69,10 +63,6 @@
       <limit effort="87" lower="-2.8973" upper="2.8973" velocity="2.1750"/>
     </joint>
-    <link name="${prefix}link2">
-      <visual>
-        <geometry>
-          <mesh filename="package://${description_pkg}/meshes/visual/link2.dae"/>
-        </geometry>
-      </visual>
+    <xacro:link name="link2">
+      <self_collision_geometries>
       <collision>
         <origin xyz="0 0 0" rpy="0 0 0"/>
@@ -93,5 +83,6 @@
         </geometry>
       </collision>
-    </link>
+      </self_collision_geometries>
+    </xacro:link>
     <joint name="${prefix}joint2" type="revolute">
       <safety_controller k_position="100.0" k_velocity="40.0" soft_lower_limit="-1.7628" soft_upper_limit="1.7628"/>
@@ -102,10 +93,6 @@
       <limit effort="87" lower="-1.7628" upper="1.7628" velocity="2.1750"/>
     </joint>
-    <link name="${prefix}link3">
-      <visual>
-        <geometry>
-          <mesh filename="package://${description_pkg}/meshes/visual/link3.dae"/>
-        </geometry>
-      </visual>
+    <xacro:link name="link3">
+      <self_collision_geometries>
       <collision>
         <origin xyz="0 0 -0.145" rpy="0 0 0"/>
@@ -126,5 +113,6 @@
         </geometry>
       </collision>
-    </link>
+      </self_collision_geometries>
+    </xacro:link>
     <joint name="${prefix}joint3" type="revolute">
       <safety_controller k_position="100.0" k_velocity="40.0" soft_lower_limit="-2.8973" soft_upper_limit="2.8973"/>
@@ -135,10 +123,6 @@
       <limit effort="87" lower="-2.8973" upper="2.8973" velocity="2.1750"/>
     </joint>
-    <link name="${prefix}link4">
-      <visual>
-        <geometry>
-          <mesh filename="package://${description_pkg}/meshes/visual/link4.dae"/>
-        </geometry>
-      </visual>
+    <xacro:link name="link4">
+      <self_collision_geometries>
       <collision>
         <origin xyz="0 0 0" rpy="0 0 0"/>
@@ -159,5 +143,6 @@
         </geometry>
       </collision>
-    </link>
+      </self_collision_geometries>
+    </xacro:link>
     <joint name="${prefix}joint4" type="revolute">
       <safety_controller k_position="100.0" k_velocity="40.0" soft_lower_limit="-3.0718" soft_upper_limit="-0.0698"/>
@@ -168,10 +153,6 @@
       <limit effort="87" lower="-3.0718" upper="-0.0698" velocity="2.1750"/>
     </joint>
-    <link name="${prefix}link5">
-      <visual>
-        <geometry>
-          <mesh filename="package://${description_pkg}/meshes/visual/link5.dae"/>
-        </geometry>
-      </visual>
+    <xacro:link name="link5">
+      <self_collision_geometries>
       <collision>
         <origin xyz="0 0 -0.26" rpy="0 0 0"/>
@@ -210,5 +191,6 @@
         </geometry>
       </collision>
-    </link>
+      </self_collision_geometries>
+    </xacro:link>
     <joint name="${prefix}joint5" type="revolute">
       <safety_controller k_position="100.0" k_velocity="40.0" soft_lower_limit="-2.8973" soft_upper_limit="2.8973"/>
@@ -219,10 +201,6 @@
       <limit effort="12" lower="-2.8973" upper="2.8973" velocity="2.6100"/>
     </joint>
-    <link name="${prefix}link6">
-      <visual>
-        <geometry>
-          <mesh filename="package://${description_pkg}/meshes/visual/link6.dae"/>
-        </geometry>
-      </visual>
+    <xacro:link name="link6">
+      <self_collision_geometries>
       <collision>
         <origin xyz="0 0 -0.03" rpy="0 0 0"/>
@@ -243,5 +221,6 @@
         </geometry>
       </collision>
-    </link>
+      </self_collision_geometries>
+    </xacro:link>
     <joint name="${prefix}joint6" type="revolute">
       <safety_controller k_position="100.0" k_velocity="40.0" soft_lower_limit="-0.0175" soft_upper_limit="3.7525"/>
@@ -252,10 +231,6 @@
       <limit effort="12" lower="-0.0175" upper="3.7525" velocity="2.6100"/>
     </joint>
-    <link name="${prefix}link7">
-      <visual>
-        <geometry>
-          <mesh filename="package://${description_pkg}/meshes/visual/link7.dae"/>
-        </geometry>
-      </visual>
+    <xacro:link name="link7">
+      <self_collision_geometries>
       <collision>
         <origin xyz="0 0 0.01" rpy="0 0 0"/>
@@ -276,5 +251,6 @@
         </geometry>
       </collision>
-    </link>
+      </self_collision_geometries>
+    </xacro:link>
     <joint name="${prefix}joint7" type="revolute">
       <safety_controller k_position="100.0" k_velocity="40.0" soft_lower_limit="-2.8973" soft_upper_limit="2.8973"/>

File: franka_description/robots/hand.urdf.xacro (robot description, xacro)
@@ -1,4 +1,5 @@
 <?xml version="1.0" encoding="utf-8"?>
 <robot xmlns:xacro="http://www.ros.org/wiki/xacro" name="hand">
+  <xacro:include filename="utils.xacro" />
   <xacro:include filename="hand.xacro"/>
   <xacro:hand prefix="panda_" safety_distance="0.03" />

File: franka_description/robots/hand.xacro (robot description, xacro)
@@ -3,5 +3,5 @@
   <!-- safety_distance: Minimum safety distance in [m] by which the collision volumes are expanded and which is enforced during robot motions -->
   <!-- prefix: used for joint and link names. Needed to distinguish joints and TFs in case of multiple arm instances. -->
-  <xacro:macro name="hand" params="connected_to:='' prefix:=^| rpy:='0 0 0' xyz:='0 0 0' safety_distance:=0">
+  <xacro:macro name="hand" params="connected_to:='' prefix:=^| rpy:='0 0 0' xyz:='0 0 0' safety_distance:=0 description_pkg:=franka_description">
     <xacro:unless value="${connected_to == ''}">
       <joint name="${prefix}hand_joint" type="fixed">
@@ -11,10 +11,6 @@
       </joint>
     </xacro:unless>
-    <link name="${prefix}hand">
-      <visual>
-        <geometry>
-          <mesh filename="package://franka_description/meshes/visual/hand.dae"/>
-        </geometry>
-      </visual>
+    <xacro:link name="hand">
+      <self_collision_geometries>
       <collision>
         <origin xyz="0 0 0.04" rpy="0 ${pi/2} ${pi/2}"/>
@@ -53,5 +49,6 @@
         </geometry>
       </collision>
-    </link>
+      </self_collision_geometries>
+    </xacro:link>
     <link name="${prefix}leftfinger">
       <visual>

File: franka_description/robots/panda_arm.urdf.xacro (robot description, xacro)
@@ -11,4 +11,5 @@
   <xacro:unless value="$(arg gazebo)">
     <!-- Create a URDF for a real hardware -->
+    <xacro:include filename="utils.xacro" />
     <xacro:include filename="arm.xacro" />
     <xacro:arm safety_distance="0.03" />

File: franka_description/robots/utils.xacro (robot description, xacro)
@@ -1,4 +1,38 @@
 <?xml version="1.0"?>
 <robot xmlns:xacro="http://www.ros.org/wiki/xacro">
+  <!-- ========================================================== -->
+  <!-- Macro to add a single link, both with                      -->
+  <!--  * detailed meshes for environmental collision checking    -->
+  <!--  * and coarse geometry models for self-collision checking  -->
+  <!--                                                            -->
+  <!-- name:  Name of the robot link (without prefix)             -->
+  <!-- self_collision_geometries:  self <collision> models        -->
+  <!-- ========================================================== -->
+  <xacro:macro name="link" params="name **self_collision_geometries">
+    <!-- sub-link defining detailed meshes for collision with environment -->
+    <link name="${prefix}${name}">
+      <visual>
+        <geometry>
+          <mesh filename="package://${description_pkg}/meshes/visual/${name}.dae" />
+        </geometry>
+      </visual>
+      <collision>
+        <geometry>
+          <mesh filename="package://franka_description/meshes/collision/${name}.stl" />
+        </geometry>
+      </collision>
+    </link>
+    <!-- sub-link defining coarse geometries of real robot's internal self-collision -->
+    <link name="${prefix}${name}_sc">
+      <xacro:unless value="$(arg gazebo)">
+        <xacro:insert_block name="self_collision_geometries" />
+      </xacro:unless>
+    </link>
+    <!-- fixed joint between both sub-links -->
+    <joint name="${prefix}${name}_sc_joint" type="fixed">
+      <parent link="${prefix}${name}" />
+      <child link="${prefix}${name}_sc" />
+    </joint>
+  </xacro:macro>
   <!-- ========================================================== -->
   <!-- Adds the required tags to simulate one joint in gazebo     -->

Commit message: Add dynamics parameters for joints from panda_gazebo

File: franka_description/robots/arm.xacro (robot description, xacro)
@@ -62,4 +62,5 @@
       <axis xyz="0 0 1"/>
       <limit effort="87" lower="-2.8973" upper="2.8973" velocity="2.1750"/>
+      <dynamics D="1" K="7000" damping="0.003" friction="0.0" mu_coulomb="0" mu_viscous="16"/>
     </joint>
     <xacro:link name="link2">
@@ -92,4 +93,5 @@
       <axis xyz="0 0 1"/>
       <limit effort="87" lower="-1.7628" upper="1.7628" velocity="2.1750"/>
+      <dynamics D="1" K="7000" damping="0.003" friction="0.0" mu_coulomb="0" mu_viscous="16"/>
     </joint>
     <xacro:link name="link3">
@@ -122,4 +124,5 @@
       <axis xyz="0 0 1"/>
       <limit effort="87" lower="-2.8973" upper="2.8973" velocity="2.1750"/>
+      <dynamics D="1" K="7000" damping="0.003" friction="0.0" mu_coulomb="0" mu_viscous="16"/>
     </joint>
     <xacro:link name="link4">
@@ -152,4 +155,5 @@
       <axis xyz="0 0 1"/>
       <limit effort="87" lower="-3.0718" upper="-0.0698" velocity="2.1750"/>
+      <dynamics D="1" K="7000" damping="0.003" friction="0.0" mu_coulomb="0" mu_viscous="16"/>
     </joint>
     <xacro:link name="link5">
@@ -200,4 +204,5 @@
       <axis xyz="0 0 1"/>
       <limit effort="12" lower="-2.8973" upper="2.8973" velocity="2.6100"/>
+      <dynamics D="1" K="7000" damping="0.003" friction="0.0" mu_coulomb="0" mu_viscous="16"/>
     </joint>
     <xacro:link name="link6">
@@ -230,4 +235,5 @@
       <axis xyz="0 0 1"/>
       <limit effort="12" lower="-0.0175" upper="3.7525" velocity="2.6100"/>
+      <dynamics D="1" K="7000" damping="0.003" friction="0.0" mu_coulomb="0" mu_viscous="16"/>
     </joint>
     <xacro:link name="link7">
@@ -260,4 +266,5 @@
       <axis xyz="0 0 1"/>
       <limit effort="12" lower="-2.8973" upper="2.8973" velocity="2.6100"/>
+      <dynamics D="1" K="7000" damping="0.003" friction="0.0" mu_coulomb="0" mu_viscous="16"/>
     </joint>
     <link name="${prefix}link8">

File: franka_description/robots/hand.xacro (robot description, xacro)
@@ -85,4 +85,5 @@
       <axis xyz="0 1 0"/>
       <limit effort="20" lower="0.0" upper="0.04" velocity="0.2"/>
+      <dynamics damping="0.3"/>
     </joint>
     <joint name="${prefix}finger_joint2" type="prismatic">
@@ -92,4 +93,5 @@
       <axis xyz="0 -1 0"/>
       <limit effort="20" lower="0.0" upper="0.04" velocity="0.2"/>
+      <dynamics damping="0.3"/>
       <mimic joint="${prefix}finger_joint1" />
     </joint>

Commit message: Distinguish link8 and link8_sc

File: franka_description/robots/arm.xacro (robot description, xacro)
@@ -268,5 +268,6 @@
       <dynamics D="1" K="7000" damping="0.003" friction="0.0" mu_coulomb="0" mu_viscous="16"/>
     </joint>
-    <link name="${prefix}link8">
+    <link name="${prefix}link8"/>
+    <link name="${prefix}link8_sc">
       <collision>
         <origin xyz="0.0424 0.0424 -0.0250" rpy="${pi} ${pi/2} ${pi/2}"/>
@@ -288,4 +289,8 @@
       </collision>
     </link>
+    <joint name="${prefix}link8_sc_joint" type="fixed">
+      <parent link="${prefix}link8" />
+      <child link="${prefix}link8_sc" />
+    </joint>
     <joint name="${prefix}joint8" type="fixed">
       <origin rpy="0 0 0" xyz="0 0 0.107"/>
