Commit message: Replace ns -> prefix

File: franka_description/robots/dual_panda_example.urdf.xacro (robot description, xacro)
@@ -25,7 +25,7 @@
   <!-- right arm with gripper -->
   <xacro:panda_arm arm_id="$(arg arm_id_1)" connected_to="base"  xyz="0 -0.5 1" safety_distance="0.03"/>
-  <xacro:hand ns="$(arg arm_id_1)" rpy="0 0 ${-pi/4}" connected_to="$(arg arm_id_1)_link8" safety_distance="0.03"/>
+  <xacro:hand prefix="$(arg arm_id_1)" rpy="0 0 ${-pi/4}" connected_to="$(arg arm_id_1)_link8" safety_distance="0.03" />
   <!-- left arm with gripper -->
   <xacro:panda_arm arm_id="$(arg arm_id_2)" connected_to="base"  xyz="0 0.5 1" safety_distance="0.03"/>
-  <xacro:hand ns="$(arg arm_id_2)" rpy="0 0 ${-pi/4}" connected_to="$(arg arm_id_2)_link8" safety_distance="0.03"/>
+  <xacro:hand prefix="$(arg arm_id_2)" rpy="0 0 ${-pi/4}" connected_to="$(arg arm_id_2)_link8" safety_distance="0.03" />
 </robot>

File: franka_description/robots/hand.urdf.xacro (robot description, xacro)
@@ -2,4 +2,4 @@
 <robot xmlns:xacro="http://www.ros.org/wiki/xacro" name="hand">
   <xacro:include filename="hand.xacro"/>
-  <xacro:hand ns="panda" safety_distance="0.03"/>
+  <xacro:hand prefix="panda" safety_distance="0.03" />
 </robot>

File: franka_description/robots/hand.xacro (robot description, xacro)
@@ -2,13 +2,13 @@
 <robot xmlns:xacro="http://www.ros.org/wiki/xacro" name="hand">
   <!-- safety_distance: Minimum safety distance in [m] by which the collision volumes are expanded and which is enforced during robot motions -->
-  <xacro:macro name="hand" params="connected_to:='' ns:='' rpy:='0 0 0' xyz:='0 0 0' safety_distance:=0">
+  <xacro:macro name="hand" params="connected_to:='' prefix:='' ns:='' rpy:='0 0 0' xyz:='0 0 0' safety_distance:=0">
     <xacro:unless value="${connected_to == ''}">
-      <joint name="${ns}_hand_joint" type="fixed">
+      <joint name="${prefix}_hand_joint" type="fixed">
         <parent link="${connected_to}"/>
-        <child link="${ns}_hand"/>
+        <child link="${prefix}_hand" />
         <origin xyz="${xyz}" rpy="${rpy}"/>
       </joint>
     </xacro:unless>
-    <link name="${ns}_hand">
+    <link name="${prefix}_hand">
       <visual>
         <geometry>
@@ -54,11 +54,11 @@
     </link>
     <!-- Define the hand_tcp frame -->
-    <link name="${ns}_hand_tcp" />
-    <joint name="${ns}_hand_tcp_joint" type="fixed">
+    <link name="${prefix}_hand_tcp" />
+    <joint name="${prefix}_hand_tcp_joint" type="fixed">
       <origin xyz="0 0 0.1034" rpy="0 0 0" />
-      <parent link="${ns}_hand" />
-      <child link="${ns}_hand_tcp" />
+      <parent link="${prefix}_hand" />
+      <child link="${prefix}_hand_tcp" />
     </joint>
-    <link name="${ns}_leftfinger">
+    <link name="${prefix}_leftfinger">
       <visual>
         <geometry>
@@ -67,5 +67,5 @@
       </visual>
     </link>
-    <link name="${ns}_rightfinger">
+    <link name="${prefix}_rightfinger">
       <visual>
         <origin xyz="0 0 0" rpy="0 0 ${pi}"/>
@@ -75,18 +75,18 @@
       </visual>
    </link>
-    <joint name="${ns}_finger_joint1" type="prismatic">
-      <parent link="${ns}_hand"/>
-      <child link="${ns}_leftfinger"/>
+    <joint name="${prefix}_finger_joint1" type="prismatic">
+      <parent link="${prefix}_hand" />
+      <child link="${prefix}_leftfinger" />
       <origin xyz="0 0 0.0584" rpy="0 0 0"/>
       <axis xyz="0 1 0"/>
       <limit effort="20" lower="0.0" upper="0.04" velocity="0.2"/>
     </joint>
-    <joint name="${ns}_finger_joint2" type="prismatic">
-      <parent link="${ns}_hand"/>
-      <child link="${ns}_rightfinger"/>
+    <joint name="${prefix}_finger_joint2" type="prismatic">
+      <parent link="${prefix}_hand" />
+      <child link="${prefix}_rightfinger" />
       <origin xyz="0 0 0.0584" rpy="0 0 0"/>
       <axis xyz="0 -1 0"/>
       <limit effort="20" lower="0.0" upper="0.04" velocity="0.2"/>
-      <mimic joint="${ns}_finger_joint1" />
+      <mimic joint="${prefix}_finger_joint1" />
     </joint>
   </xacro:macro>

File: franka_description/robots/panda_arm.urdf.xacro (robot description, xacro)
@@ -13,5 +13,5 @@
     <xacro:if value="$(arg hand)">
       <xacro:include filename="$(find franka_description)/robots/hand.xacro"/>
-      <xacro:hand ns="$(arg arm_id)" rpy="0 0 ${-pi/4}" connected_to="$(arg arm_id)_link8" safety_distance="0.03"/>
+      <xacro:hand prefix="$(arg arm_id)" rpy="0 0 ${-pi/4}" connected_to="$(arg arm_id)_link8" safety_distance="0.03" />
     </xacro:if>
   </xacro:unless>
@@ -24,5 +24,5 @@
     <xacro:panda_arm arm_id="$(arg arm_id)" />
     <xacro:if value="$(arg hand)">
-      <xacro:hand ns="$(arg arm_id)" rpy="0 0 ${-pi/4}" connected_to="$(arg arm_id)_link8" />
+      <xacro:hand prefix="$(arg arm_id)" rpy="0 0 ${-pi/4}" connected_to="$(arg arm_id)_link8" />
       <xacro:gazebo-joint joint="$(arg arm_id)_finger_joint1" transmission="hardware_interface/EffortJointInterface" />
       <xacro:gazebo-joint joint="$(arg arm_id)_finger_joint2" transmission="hardware_interface/EffortJointInterface" />

File: franka_description/robots/panda_gazebo.xacro (robot description, xacro)
@@ -251,14 +251,14 @@
     </joint>
   </xacro:macro>
-  <xacro:macro name="hand" params="connected_to:='' ns:='' xyz:='0 0 0' rpy:='0 0 0'">
+  <xacro:macro name="hand" params="connected_to:='' prefix:='' ns:='' xyz:='0 0 0' rpy:='0 0 0'">
     <xacro:include filename="$(find franka_description)/robots/utils.xacro"/>
     <xacro:unless value="${connected_to == ''}">
-      <joint name="${ns}_hand_joint" type="fixed">
+      <joint name="${prefix}_hand_joint" type="fixed">
         <parent link="${connected_to}"/>
-        <child link="${ns}_hand"/>
+        <child link="${prefix}_hand" />
         <origin xyz="${xyz}" rpy="${rpy}"/>
       </joint>
     </xacro:unless>
-    <link name="${ns}_hand">
+    <link name="${prefix}_hand">
       <visual>
         <geometry>
@@ -309,5 +309,5 @@
       </collision>
     </xacro:macro>
-    <link name="${ns}_leftfinger">
+    <link name="${prefix}_leftfinger">
       <xacro:inertia-cylinder mass="15e-3" radius="0.01" h="0.04"/>
       <visual>
@@ -318,5 +318,5 @@
       <xacro:finger-collision sign="+" />
     </link>
-    <link name="${ns}_rightfinger">
+    <link name="${prefix}_rightfinger">
       <xacro:inertia-cylinder mass="15e-3" radius="0.01" h="0.04"/>
       <visual>
@@ -330,9 +330,9 @@
     <!-- Friction specific material for Rubber/Rubber contact -->
     <!-- See: -->
-    <xacro:gazebo-friction link="${ns}_leftfinger" mu="1.13" />
-    <xacro:gazebo-friction link="${ns}_rightfinger" mu="1.13" />
-    <joint name="${ns}_finger_joint1" type="prismatic">
-      <parent link="${ns}_hand"/>
-      <child link="${ns}_leftfinger"/>
+    <xacro:gazebo-friction link="${prefix}_leftfinger" mu="1.13" />
+    <xacro:gazebo-friction link="${prefix}_rightfinger" mu="1.13" />
+    <joint name="${prefix}_finger_joint1" type="prismatic">
+      <parent link="${prefix}_hand" />
+      <child link="${prefix}_leftfinger" />
       <origin xyz="0 0 0.0584" rpy="0 0 0"/>
       <axis xyz="0 1 0"/>
@@ -340,7 +340,7 @@
       <dynamics friction="0.0" damping="0.03"/>
     </joint>
-    <joint name="${ns}_finger_joint2" type="prismatic">
-      <parent link="${ns}_hand"/>
-      <child link="${ns}_rightfinger"/>
+    <joint name="${prefix}_finger_joint2" type="prismatic">
+      <parent link="${prefix}_hand" />
+      <child link="${prefix}_rightfinger" />
       <origin xyz="0 0 0.0584" rpy="0 0 0"/>
       <axis xyz="0 -1 0"/>
