Commit message: FIX: Use correct naming for `gazebo-friction`
Friction acts on links not joints

File: franka_description/robots/panda_gazebo.xacro (robot description, xacro)
@@ -323,6 +323,6 @@
     <!-- Friction specific material for Rubber/Rubber contact -->
     <!-- See: -->
-    <xacro:gazebo-friction joint="${ns}_leftfinger" mu="1.13" />
-    <xacro:gazebo-friction joint="${ns}_rightfinger" mu="1.13" />
+    <xacro:gazebo-friction link="${ns}_leftfinger" mu="1.13" />
+    <xacro:gazebo-friction link="${ns}_rightfinger" mu="1.13" />
     <joint name="${ns}_finger_joint1" type="prismatic">
       <parent link="${ns}_hand"/>

File: franka_description/robots/utils.xacro (robot description, xacro)
@@ -22,6 +22,6 @@
     </transmission>
   </xacro:macro>
-  <xacro:macro name="gazebo-friction" params="joint mu">
-    <gazebo reference="${joint}">
+  <xacro:macro name="gazebo-friction" params="link mu">
+    <gazebo reference="${link}">
       <collision>
         <max_contacts>10</max_contacts>

Commit message: FIX: Don't mimic fingers in gazebo
This is unfortunately not possible, since gazebo cannot reflect external force
acting on one finger onto the mimicked other finger

File: franka_description/robots/panda_gazebo.xacro (robot description, xacro)
@@ -340,5 +340,4 @@
       <limit effort="20" lower="0.0" upper="0.04" velocity="0.2"/>
       <dynamics damping="0.3"/>
-      <mimic joint="${ns}_finger_joint1" />
     </joint>
   </xacro:macro>

Commit message: Add realistic hand/finger collision meshes to the gazebo robot description
This commit replaces the hand/finger collision geometries that are used in the Gazebo
robot description with more accurate meshes. These meshes were taken from
[AndrejOrsula/panda_ign](https://github.com/AndrejOrsula/panda_ign/blob/master/panda/meshes/collision/finger.stl).

File: franka_description/robots/panda_gazebo.xacro (robot description, xacro)
@@ -267,7 +267,6 @@
       </visual>
       <collision>
-        <origin xyz="0.0 0 0.0375" rpy="0 ${pi/2} ${pi/2}"/>
-        <geometry>
-          <box size="0.055 0.04 0.198"  />
+        <geometry>
+          <mesh filename="package://franka_description/meshes/collision/hand.stl" />
         </geometry>
       </collision>
@@ -288,13 +287,6 @@
       </visual>
       <collision>
-        <origin xyz="0 0.015 0.03" rpy="0 0 0"/>
-        <geometry>
-          <box size="0.03 0.005 0.047" />
-        </geometry>
-      </collision>
-      <collision>
-        <origin xyz="0 0.007 0.045" rpy="0 0 0"/>
-        <geometry>
-          <box size="0.03 0.015 0.017" />
+        <geometry>
+          <mesh filename="package://franka_description/meshes/collision/finger.stl" />
         </geometry>
       </collision>
@@ -309,13 +301,7 @@
       </visual>
       <collision>
-        <origin xyz="0 -0.015 0.03" rpy="0 0 0"/>
-        <geometry>
-          <box size="0.03 0.005 0.047" />
-        </geometry>
-      </collision>
-      <collision>
-        <origin xyz="0 -0.007 0.045" rpy="0 0 0"/>
-        <geometry>
-          <box size="0.03 0.015 0.017" />
+        <origin xyz="0 0 0" rpy="0 0 ${pi}"/>
+        <geometry>
+          <mesh filename="package://franka_description/meshes/collision/finger.stl" />
         </geometry>
       </collision>

Commit message: Fixes hand real/gazebo discrepacy
This commit makes sure that the hand joint control behavoir between the
real and simulated robot is equal. Previously the 'franka_finger_joint2'
mimics the 'franka_finger_joint1' in the real robot but not in the
simulation.

File: franka_description/robots/panda_gazebo.xacro (robot description, xacro)
@@ -340,4 +340,5 @@
       <limit effort="20" lower="0.0" upper="0.04" velocity="0.2"/>
       <dynamics damping="0.3"/>
+      <mimic joint="${ns}_finger_joint1" />
     </joint>
   </xacro:macro>

Commit message: Fixes gazebo gripper action bug
This commit fixes a bug that was introduced by #147. In #147 the
finger collision geometries were replaced by more accurate meshes.
These more accurate messages however broke the 'gripper_action' action.
This commit migrates back to using geometries for the finger collision geometries.
The action server works fine when geometriesare used.

File: franka_description/robots/panda_gazebo.xacro (robot description, xacro)
@@ -287,6 +287,19 @@
       </visual>
       <collision>
-        <geometry>
-          <mesh filename="package://franka_description/meshes/collision/finger.stl" />
+        <origin xyz="0 0.0184 0.0101" rpy="0 0 0"/>
+        <geometry>
+          <box size="0.022 0.014 0.0177" />
+        </geometry>
+      </collision>
+      <collision>
+        <origin xyz="0 0.01655 0.02755" rpy="${3.257/(2*pi)} 0 0"/>
+        <geometry>
+          <box size="0.022 0.00686 0.0237" />
+        </geometry>
+      </collision>
+      <collision>
+        <origin xyz="0 0.0073 0.045" rpy="0 0 0"/>
+        <geometry>
+          <box size="0.022 0.0147 0.0178" />
         </geometry>
       </collision>
@@ -301,7 +314,19 @@
       </visual>
       <collision>
-        <origin xyz="0 0 0" rpy="0 0 ${pi}"/>
-        <geometry>
-          <mesh filename="package://franka_description/meshes/collision/finger.stl" />
+        <origin xyz="0 -0.0184 0.0101" rpy="0 0 0"/>
+        <geometry>
+          <box size="0.022 0.014 0.0177" />
+        </geometry>
+      </collision>
+      <collision>
+        <origin xyz="0 -0.01655 0.02755" rpy="${-3.257/(2*pi)} 0 0"/>
+        <geometry>
+          <box size="0.022 0.00686 0.0237" />
+        </geometry>
+      </collision>
+      <collision>
+        <origin xyz="0 -0.0073 0.045" rpy="0 0 0"/>
+        <geometry>
+          <box size="0.022 0.0147 0.0178" />
         </geometry>
       </collision>

Commit message: Define finger_joint2 as mimic joint of finger_joint1
Although, Gazebo doesn't support mimic joints natively,
FrankaHWSim does and MoveIt - for planning - should know
that the fingers will move in sync.

File: franka_description/robots/panda_gazebo.xacro (robot description, xacro)
@@ -354,4 +354,5 @@
       <limit effort="20" lower="0.0" upper="0.04" velocity="0.2"/>
       <dynamics friction="0.0" damping="0.03"/>
+      <mimic joint="${ns}_finger_joint1" />
     </joint>
   </xacro:macro>
