Commit message: TEST: Stick URDF
Launch the UNROTATED (working) example with:

```bash
roslaunch franka_gazebo panda.launch \
  use_gripper:=false \
  headless:=false \
  paused:=true \
  initial_joint_positions:="-J panda_joint6 $(calc 'deg2rad(-90)')"
```

and step the simulation a few times.

For the bugged example switch the commented region in `panda_gazebo.xacro` for
joint6 and launch the ROTATED (bugged) example with:

```bash
roslaunch franka_gazebo panda.launch \
  use_gripper:=false \
  headless:=false \
  paused:=true \
  initial_joint_positions:="-J panda_joint6 $(calc 'deg2rad(90)')"
```

File: franka_description/robots/panda_gazebo.xacro (robot description, xacro)
@@ -13,317 +13,209 @@
     <link name="${arm_id}_link0">
       <visual>
-        <origin rpy="0 0 0" xyz="0 0 0"/>
-        <geometry>
-          <mesh filename="package://franka_description/meshes/visual/link0.dae"/>
-        </geometry>
-      </visual>
-      <collision>
-        <origin rpy="0 0 0" xyz="0 0 0"/>
-        <geometry>
-          <mesh filename="package://franka_description/meshes/collision/link0.stl"/>
-        </geometry>
-      </collision>
-      <inertial>
-        <!-- Estimated guesses from CAD -->
-        <origin rpy="0 0 0" xyz="-0.041018 -0.00014 0.049974"/>
-        <mass value="0.629769"/>
-        <inertia ixx="0.00315" ixy="8.2904E-07" ixz="0.00015"
-                               iyy="0.00388"    iyz="8.2299E-06"
-                                                izz="0.004285" />
+        <origin xyz="0 0 0.05" />
+        <geometry><box size="0.02 0.02 0.08" /></geometry>
+      </visual>
+      <collision>
+        <origin xyz="0 0 0.05" />
+        <geometry><box size="0.02 0.02 0.08" /></geometry>
+      </collision>
+      <inertial>
+        <origin xyz="0 0 0.05" />
+        <mass value="${0.5*10./9.80}" />
+        <inertia ixx="0.1" iyy="0.1" izz="0.1"
+                 ixy="0"   ixz="0"   iyz="0" />
       </inertial>
     </link>
     <link name="${arm_id}_link1">
       <visual>
-        <origin rpy="0 0 0" xyz="0 0 0"/>
-        <geometry>
-          <mesh filename="package://franka_description/meshes/visual/link1.dae"/>
-        </geometry>
-      </visual>
-      <collision>
-        <origin rpy="0 0 0" xyz="0 0 0"/>
-        <geometry>
-          <mesh filename="package://franka_description/meshes/collision/link1.stl"/>
-        </geometry>
-      </collision>
-      <inertial>
-        <origin rpy="0 0 0" xyz="0.003875 0.002081 -0.04762"/>
-        <mass value="4.970684"/>
-        <inertia ixx="0.70337" ixy="-0.00013900" ixz="0.0067720"
-                               iyy="0.70661"     iyz="0.019169"
-                                                 izz="0.0091170" />
-      </inertial>
-    </link>
+        <origin xyz="0 0 0.05" />
+        <geometry><box size="0.02 0.02 0.08" /></geometry>
+      </visual>
+      <collision>
+        <origin xyz="0 0 0.05" />
+        <geometry><box size="0.02 0.02 0.08" /></geometry>
+      </collision>
+      <inertial>
+        <origin xyz="0 0 0.05" />
+        <mass value="${0.5*10./9.80}" />
+        <inertia ixx="0.1" iyy="0.1" izz="0.1"
+                 ixy="0"   ixz="0"   iyz="0" />
+      </inertial>
+    </link>
+    <link name="${arm_id}_link2">
+      <visual>
+        <origin xyz="0 0 0.05" />
+        <geometry><box size="0.02 0.02 0.08" /></geometry>
+      </visual>
+      <collision>
+        <origin xyz="0 0 0.05" />
+        <geometry><box size="0.02 0.02 0.08" /></geometry>
+      </collision>
+      <inertial>
+        <origin xyz="0 0 0.05" />
+        <mass value="${0.5*10./9.80}" />
+        <inertia ixx="0.1" iyy="0.1" izz="0.1"
+                 ixy="0"   ixz="0"   iyz="0" />
+      </inertial>
+    </link>
+    <link name="${arm_id}_link3">
+      <visual>
+        <origin xyz="0 0 0.05" />
+        <geometry><box size="0.02 0.02 0.08" /></geometry>
+      </visual>
+      <collision>
+        <origin xyz="0 0 0.05" />
+        <geometry><box size="0.02 0.02 0.08" /></geometry>
+      </collision>
+      <inertial>
+        <origin xyz="0 0 0.05" />
+        <mass value="${0.5*10./9.80}" />
+        <inertia ixx="0.1" iyy="0.1" izz="0.1"
+                 ixy="0"   ixz="0"   iyz="0" />
+      </inertial>
+    </link>
+    <link name="${arm_id}_link4">
+      <visual>
+        <origin xyz="0 0 0.05" />
+        <geometry><box size="0.02 0.02 0.08" /></geometry>
+      </visual>
+      <collision>
+        <origin xyz="0 0 0.05" />
+        <geometry><box size="0.02 0.02 0.08" /></geometry>
+      </collision>
+      <inertial>
+        <origin xyz="0 0 0.05" />
+        <mass value="${0.5*10./9.80}" />
+        <inertia ixx="0.1" iyy="0.1" izz="0.1"
+                 ixy="0"   ixz="0"   iyz="0" />
+      </inertial>
+    </link>
+    <link name="${arm_id}_link5">
+      <visual>
+        <origin xyz="0 0 0.05" />
+        <geometry><box size="0.02 0.02 0.08" /></geometry>
+      </visual>
+      <collision>
+        <origin xyz="0 0 0.05" />
+        <geometry><box size="0.02 0.02 0.08" /></geometry>
+      </collision>
+      <inertial>
+        <origin xyz="0 0 0.05" />
+        <mass value="${0.5*10./9.80}" />
+        <inertia ixx="0.1" iyy="0.1" izz="0.1"
+                 ixy="0"   ixz="0"   iyz="0" />
+      </inertial>
+    </link>
+    <link name="${arm_id}_link6">
+      <visual>
+        <origin xyz="0 0 0.05" />
+        <geometry><box size="0.02 0.02 0.08" /></geometry>
+      </visual>
+      <collision>
+        <origin xyz="0 0 0.05" />
+        <geometry><box size="0.02 0.02 0.08" /></geometry>
+      </collision>
+      <inertial>
+        <mass value="${0.5*10./9.80}" />
+        <origin xyz="0 0 0.05" />
+        <inertia ixx="0.1" iyy="0.1" izz="0.1"
+                 ixy="0"   ixz="0"   iyz="0" />
+      </inertial>
+    </link>
+    <link name="${arm_id}_link7">
+      <visual>
+        <origin xyz="0 0 0.05" />
+        <geometry><box size="0.02 0.02 0.08" /></geometry>
+      </visual>
+      <collision>
+        <origin xyz="0 0 0.05" />
+        <geometry><box size="0.02 0.02 0.08" /></geometry>
+      </collision>
+      <inertial>
+        <origin xyz="0 0 0.05" />
+        <mass value="${0.5*10./9.80}" />
+        <inertia ixx="0.1" iyy="0.1" izz="0.1"
+                 ixy="0"   ixz="0"   iyz="0" />
+      </inertial>
+    </link>
+    <link name="${arm_id}_link8" />
     <joint name="${arm_id}_joint1" type="revolute">
       <safety_controller k_position="100.0" k_velocity="40.0" soft_lower_limit="-2.8973" soft_upper_limit="2.8973"/>
-      <origin rpy="0 0 0" xyz="0 0 0.333"/>
+      <origin rpy="0 0 0" xyz="0 0 0.1"/>
       <parent link="${arm_id}_link0"/>
       <child link="${arm_id}_link1"/>
-      <axis xyz="0 0 1"/>
-      <limit acceleration="15" lower="-2.9671" effort="87" upper="2.9671" velocity="2.5"/>
-      <dynamics D="1" K="7000" mu_coulomb="0" mu_viscous="16" damping="0.003" friction="0.0"/>
-    </joint>
-    <link name="${arm_id}_link2">
-      <visual>
-        <origin rpy="0 0 0" xyz="0 0 0"/>
-        <geometry>
-          <mesh filename="package://franka_description/meshes/visual/link2.dae"/>
-        </geometry>
-      </visual>
-      <collision>
-        <origin rpy="0 0 0" xyz="0 0 0"/>
-        <geometry>
-          <mesh filename="package://franka_description/meshes/collision/link2.stl"/>
-        </geometry>
-      </collision>
-      <inertial>
-        <origin rpy="0 0 0" xyz=" -0.003141 -0.02872  0.003495"/>
-        <mass value="0.646926"/>
-        <inertia ixx="0.0079620" ixy="-3.9250e-3" ixz="1.0254e-02"
-                                 iyy="2.8110e-02" iyz="7.0400e-04"
-                                                  izz="2.5995e-02" />
-      </inertial>
-    </link>
+      <axis xyz="0 1 0"/>
+      <limit acceleration="15" lower="-2.9671" effort="87" upper="2.9671" velocity="2.5"/>
+      <dynamics D="1" K="7000" mu_coulomb="0" mu_viscous="16" damping="0.003" friction="0.0"/>
+    </joint>
     <joint name="${arm_id}_joint2" type="revolute">
-      <safety_controller k_position="100.0" k_velocity="40.0" soft_lower_limit="-1.7628" soft_upper_limit="1.7628"/>
-      <origin rpy="${-pi/2} 0 0" xyz="0 0 0"/>
+      <safety_controller k_position="100.0" k_velocity="40.0" soft_lower_limit="-2.8973" soft_upper_limit="2.8973"/>
+      <origin rpy="0 0 0" xyz="0 0 0.1"/>
       <parent link="${arm_id}_link1"/>
       <child link="${arm_id}_link2"/>
       <axis xyz="0 0 1"/>
-      <limit acceleration="7.5" lower="-1.8326" effort="87" upper="1.8326" velocity="2.5"/>
-      <dynamics D="1" K="7000" mu_coulomb="0" mu_viscous="16" damping="0.003" friction="0.0"/>
-    </joint>
-    <link name="${arm_id}_link3">
-      <visual>
-        <origin rpy="0 0 0" xyz="0 0 0"/>
-        <geometry>
-          <mesh filename="package://franka_description/meshes/visual/link3.dae"/>
-        </geometry>
-      </visual>
-      <collision>
-        <origin rpy="0 0 0" xyz="0 0 0"/>
-        <geometry>
-          <mesh filename="package://franka_description/meshes/collision/link3.stl"/>
-        </geometry>
-      </collision>
-      <inertial>
-        <origin rpy="0 0 0" xyz="2.7518e-02 3.9252e-02 -6.6502e-02"/>
-        <mass value="3.228604"/>
-        <inertia ixx="3.7242e-02" ixy="-4.7610e-03" ixz="-1.1396e-02"
-                                  iyy="3.6155e-02"  iyz="-1.2805e-02"
-                                                    izz="1.0830e-02" />
-      </inertial>
-    </link>
+      <limit acceleration="15" lower="-2.9671" effort="87" upper="2.9671" velocity="2.5"/>
+      <dynamics D="1" K="7000" mu_coulomb="0" mu_viscous="16" damping="0.003" friction="0.0"/>
+    </joint>
     <joint name="${arm_id}_joint3" type="revolute">
       <safety_controller k_position="100.0" k_velocity="40.0" soft_lower_limit="-2.8973" soft_upper_limit="2.8973"/>
-      <origin rpy="${pi/2} 0 0" xyz="0 -0.316 0"/>
+      <origin rpy="0 0 0" xyz="0 0 0.1"/>
       <parent link="${arm_id}_link2"/>
       <child link="${arm_id}_link3"/>
       <axis xyz="0 0 1"/>
-      <limit acceleration="12.5" lower="-2.9671" effort="87" upper="2.9671" velocity="2.5"/>
-      <dynamics D="1" K="7000" mu_coulomb="0" mu_viscous="16" damping="0.003" friction="0.0"/>
-    </joint>
-    <link name="${arm_id}_link4">
-      <visual>
-        <origin rpy="0 0 0" xyz="0 0 0"/>
-        <geometry>
-          <mesh filename="package://franka_description/meshes/visual/link4.dae"/>
-        </geometry>
-      </visual>
-      <collision>
-        <origin rpy="0 0 0" xyz="0 0 0"/>
-        <geometry>
-          <mesh filename="package://franka_description/meshes/collision/link4.stl"/>
-        </geometry>
-      </collision>
-      <inertial>
-        <origin rpy="0 0 0" xyz="-5.317e-02 1.04419e-01 2.7454e-02"/>
-        <mass value="3.587895"/>
-        <inertia ixx="2.5853e-02" ixy="7.7960e-03" ixz="-1.3320e-03"
-                                  iyy="1.9552e-02" iyz="8.6410e-03"
-                                                   izz="2.8323e-02" />
-      </inertial>
-    </link>
+      <limit acceleration="15" lower="-2.9671" effort="87" upper="2.9671" velocity="2.5"/>
+      <dynamics D="1" K="7000" mu_coulomb="0" mu_viscous="16" damping="0.003" friction="0.0"/>
+    </joint>
     <joint name="${arm_id}_joint4" type="revolute">
-      <safety_controller k_position="100.0" k_velocity="40.0" soft_lower_limit="-3.0718" soft_upper_limit="-0.0698"/>
-      <origin rpy="${pi/2} 0 0" xyz="0.0825 0 0"/>
+      <safety_controller k_position="100.0" k_velocity="40.0" soft_lower_limit="-2.8973" soft_upper_limit="2.8973"/>
+      <origin rpy="0 0 0" xyz="0 0 0.1"/>
       <parent link="${arm_id}_link3"/>
       <child link="${arm_id}_link4"/>
       <axis xyz="0 0 1"/>
-      <limit acceleration="12.5" lower="-3.1416" effort="87" upper="-0.4" velocity="2.5"/>
-      <dynamics D="1" K="7000" mu_coulomb="0" mu_viscous="16" damping="0.003" friction="0.0"/>
-    </joint>
-    <link name="${arm_id}_link5">
-      <visual>
-        <origin rpy="0 0 0" xyz="0 0 0"/>
-        <geometry>
-          <mesh filename="package://franka_description/meshes/visual/link5.dae"/>
-        </geometry>
-      </visual>
-      <collision>
-        <origin rpy="0 0 0" xyz="0 0 0"/>
-        <geometry>
-          <mesh filename="package://franka_description/meshes/collision/link5.stl"/>
-        </geometry>
-      </collision>
-      <inertial>
-        <origin rpy="0 0 0" xyz="-1.1953e-02 4.1065e-02 -3.8437e-02"/>
-        <mass value="1.225946"/>
-        <inertia ixx="3.5549e-02" ixy="-2.1170e-03" ixz="-4.0370e-03"
-                                  iyy="2.9474e-02"  iyz="2.2900e-04"
-                                                    izz="8.6270e-03" />
-      </inertial>
-    </link>
+      <limit acceleration="15" lower="-2.9671" effort="87" upper="2.9671" velocity="2.5"/>
+      <dynamics D="1" K="7000" mu_coulomb="0" mu_viscous="16" damping="0.003" friction="0.0"/>
+    </joint>
     <joint name="${arm_id}_joint5" type="revolute">
       <safety_controller k_position="100.0" k_velocity="40.0" soft_lower_limit="-2.8973" soft_upper_limit="2.8973"/>
-      <origin rpy="${-pi/2} 0 0" xyz="-0.0825 0.384 0"/>
+      <origin rpy="0 0 0" xyz="0 0 0.1"/>
       <parent link="${arm_id}_link4"/>
       <child link="${arm_id}_link5"/>
       <axis xyz="0 0 1"/>
-      <limit acceleration="15" lower="-2.9671" effort="12" upper="2.9671" velocity="3"/>
-      <dynamics D="1" K="7000" mu_coulomb="0" mu_viscous="16" damping="0.003" friction="0.0"/>
-    </joint>
-    <link name="${arm_id}_link6">
-      <visual>
-        <origin rpy="0 0 0" xyz="0 0 0"/>
-        <geometry>
-          <mesh filename="package://franka_description/meshes/visual/link6.dae"/>
-        </geometry>
-      </visual>
-      <collision>
-        <origin rpy="0 0 0" xyz="0 0 0"/>
-        <geometry>
-          <mesh filename="package://franka_description/meshes/collision/link6.stl"/>
-        </geometry>
-      </collision>
-      <inertial>
-        <origin rpy="0 0 0" xyz="6.0149e-02 -1.4117e-02 -1.0517e-02"/>
-        <mass value="1.666555"/>
-        <inertia ixx="1.9640e-03" ixy="1.0900e-04" ixz="-1.1580e-03"
-                                  iyy="4.3540e-03" iyz="3.4100e-04"
-                                                   izz="5.4330e-03" />
-      </inertial>
-    </link>
+      <limit acceleration="15" lower="-2.9671" effort="87" upper="2.9671" velocity="2.5"/>
+      <dynamics D="1" K="7000" mu_coulomb="0" mu_viscous="16" damping="0.003" friction="0.0"/>
+    </joint>
+    <!-- Joint 6 WITHOUT Rotation -->
     <joint name="${arm_id}_joint6" type="revolute">
-      <safety_controller k_position="100.0" k_velocity="40.0" soft_lower_limit="-0.0175" soft_upper_limit="3.7525"/>
-      <origin rpy="${pi/2} 0 0" xyz="0 0 0"/>
+      <safety_controller k_position="100.0" k_velocity="40.0" soft_lower_limit="-2.8973" soft_upper_limit="2.8973"/>
+      <origin rpy="0 0 0" xyz="0 0 0.1"/>
       <parent link="${arm_id}_link5"/>
       <child link="${arm_id}_link6"/>
-      <axis xyz="0 0 1"/>
-      <limit acceleration="20" lower="-0.0873" effort="12" upper="3.8223" velocity="3"/>
-      <dynamics D="1" K="7000" mu_coulomb="0" mu_viscous="16" damping="0.003" friction="0.0"/>
-    </joint>
-    <link name="${arm_id}_link7">
-      <visual>
-        <origin rpy="0 0 0" xyz="0 0 0"/>
-        <geometry>
-          <mesh filename="package://franka_description/meshes/visual/link7.dae"/>
-        </geometry>
-      </visual>
-      <collision>
-        <origin rpy="0 0 0" xyz="0 0 0"/>
-        <geometry>
-          <mesh filename="package://franka_description/meshes/collision/link7.stl"/>
-        </geometry>
-      </collision>
-      <inertial>
-        <origin rpy="0 0 0" xyz="1.0517e-02 -4.252e-03 6.1597e-02"/>
-        <mass value="7.35522e-01"/>
-        <inertia ixx="1.2516e-02" ixy="-4.2800e-04" ixz="-1.1960e-03"
-                                  iyy="1.0027e-02"  iyz="-7.4100e-04"
-                                                    izz="4.8150e-03"/>
-      </inertial>
-    </link>
+      <axis xyz="0 1 0"/>
+      <limit acceleration="15" lower="-2.9671" effort="87" upper="2.9671" velocity="2.5"/>
+      <dynamics D="1" K="7000" mu_coulomb="0" mu_viscous="16" damping="0.003" friction="0.0"/>
+    </joint>
+    <!-- Joint 6 WITH Rotation -->
+    <!-- <joint name="${arm_id}_joint6" type="revolute"> -->
+    <!--   <safety_controller k_position="100.0" k_velocity="40.0" soft_lower_limit="-2.8973" soft_upper_limit="2.8973"/> -->
+    <!--   <origin rpy="${pi/2} 0 0" xyz="0 0 0.1"/> -->
+    <!--   <parent link="${arm_id}_link5"/> -->
+    <!--   <child link="${arm_id}_link6"/> -->
+    <!--   <axis xyz="0 0 1"/> -->
+    <!--   <limit acceleration="15" lower="-2.9671" effort="87" upper="2.9671" velocity="2.5"/> -->
+    <!--   <dynamics D="1" K="7000" mu_coulomb="0" mu_viscous="16" damping="0.003" friction="0.0"/> -->
+    <!-- </joint> -->
     <joint name="${arm_id}_joint7" type="revolute">
       <safety_controller k_position="100.0" k_velocity="40.0" soft_lower_limit="-2.8973" soft_upper_limit="2.8973"/>
-      <origin rpy="${pi/2} 0 0" xyz="0.088 0 0"/>
+      <origin rpy="${pi/2} 0 0" xyz="0 0 0.1"/>
       <parent link="${arm_id}_link6"/>
       <child link="${arm_id}_link7"/>
       <axis xyz="0 0 1"/>
-      <limit acceleration="20" lower="-2.9671" effort="12" upper="2.9671" velocity="3"/>
-      <dynamics D="1" K="7000" mu_coulomb="0" mu_viscous="16" damping="0.003" friction="0.0"/>
-    </joint>
-    <link name="${arm_id}_link8" />
+      <limit acceleration="15" lower="-2.9671" effort="87" upper="2.9671" velocity="2.5"/>
+      <dynamics D="1" K="7000" mu_coulomb="0" mu_viscous="16" damping="0.003" friction="0.0"/>
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
Commit message: CHANGE: Finger collision meshes to primitive boxes
With the mesh shape with the 28 vertices Gazebo struggles in contact
situations. When closing the fingers once they touch they become very unstable
and jiggle around. Reverting the finger collision into a primitive
compromised of boxes solves the problem.

File: franka_description/robots/panda_gazebo.xacro (robot description, xacro)
@@ -286,7 +286,30 @@
         </geometry>
       </visual>
-      <collision>
-        <geometry>
-          <mesh filename="package://franka_description/meshes/collision/finger.stl" />
+      <!-- screw mount -->
+      <collision>
+        <origin xyz="0 18.5e-3 11e-3" rpy="0 0 0"/>
+        <geometry>
+          <box size="22e-3 15e-3 20e-3" />
+        </geometry>
+      </collision>
+      <!-- cartriage sledge -->
+      <collision>
+        <origin xyz="0 6.8e-3 2.2e-3" rpy="0 0 0"/>
+        <geometry>
+          <box size="22e-3 8.8e-3 3.8e-3" />
+        </geometry>
+      </collision>
+      <!-- diagonal finger -->
+      <collision>
+        <origin xyz="0 15.9e-3 28.35e-3" rpy="${pi/6} 0 0"/>
+        <geometry>
+          <box size="17.5e-3 7e-3 23.5e-3" />
+        </geometry>
+      </collision>
+      <!-- rubber tip with which to grasp -->
+      <collision>
+        <origin xyz="0 7.58e-3 45.25e-3" rpy="0 0 0"/>
+        <geometry>
+          <box size="17.5e-3 15.2e-3 18.5e-3" />
         </geometry>
       </collision>
@@ -300,8 +323,30 @@
         </geometry>
       </visual>
-      <collision>
-        <origin xyz="0 0 0" rpy="0 0 ${pi}"/>
-        <geometry>
-          <mesh filename="package://franka_description/meshes/collision/finger.stl" />
+      <!-- screw mount -->
+      <collision>
+        <origin xyz="0 -18.5e-3 11e-3" rpy="0 0 0"/>
+        <geometry>
+          <box size="22e-3 15e-3 20e-3" />
+        </geometry>
+      </collision>
+      <!-- cartriage sledge -->
+      <collision>
+        <origin xyz="0 -6.8e-3 2.2e-3" rpy="0 0 0"/>
+        <geometry>
+          <box size="22e-3 8.8e-3 3.8e-3" />
+        </geometry>
+      </collision>
+      <!-- diagonal finger -->
+      <collision>
+        <origin xyz="0 -15.9e-3 28.35e-3" rpy="${-pi/6} 0 0"/>
+        <geometry>
+          <box size="17.5e-3 7e-3 23.5e-3" />
+        </geometry>
+      </collision>
+      <!-- rubber tip with which to grasp -->
+      <collision>
+        <origin xyz="0 -7.58e-3 45.25e-3" rpy="0 0 0"/>
+        <geometry>
+          <box size="17.5e-3 15.2e-3 18.5e-3" />
         </geometry>
       </collision>

Commit message: Rename panda_arm.xacro -> arm.xacro
... and xacro:panda_arm -> xacro:arm
to be consistent with hand.xacro

File: franka_description/robots/panda_gazebo.xacro (robot description, xacro)
@@ -10,5 +10,5 @@
   <!-- || Paolo Robuffo Giordano, Alessandro de Luca                || -->
   <!-- =============================================================== -->
-  <xacro:macro name="panda_arm" params="arm_id:='panda'">
+  <xacro:macro name="arm" params="arm_id:='panda'">
     <link name="${arm_id}_link0">
       <visual>

Commit message: FIX: Tune parameter for fingers to grasp successful in franka_gazebo
With very light fingers (~15g) the PID controller of `franka_gripper_sim` is
tuned way too aggressively. It makes the fingers oscillate in contact situations
(e.g. after a grasping action). This oscillation won't make the gripper change
to the HOLDING state, which eventually makes the grasp action hang forever.

Relaxing the D and I gains makes the control much more stable, while keeping
overall sufficient accuracy.

Also for opening grasps, since there is no contact the velocity oscillates much
more then for closing grasps. Slightly increasing the resting threshold makes
the action also succeed here.

File: franka_description/robots/panda_gazebo.xacro (robot description, xacro)
@@ -362,5 +362,5 @@
       <axis xyz="0 1 0"/>
       <limit effort="20" lower="0.0" upper="0.04" velocity="0.2"/>
-      <dynamics damping="0.3"/>
+      <dynamics friction="0.0" damping="0.03"/>
     </joint>
     <joint name="${ns}_finger_joint2" type="prismatic">
@@ -370,5 +370,5 @@
       <axis xyz="0 -1 0"/>
       <limit effort="20" lower="0.0" upper="0.04" velocity="0.2"/>
-      <dynamics damping="0.3"/>
+      <dynamics friction="0.0" damping="0.03"/>
     </joint>
   </xacro:macro>
