Commit message: CHANGE: Refactor finger collision models to macro

File: franka_description/robots/panda_gazebo.xacro (robot description, xacro)
@@ -279,4 +279,34 @@
       </inertial>
     </link>
+    <xacro:macro name="finger-collision" params="sign">
+      <!-- screw mount -->
+      <collision>
+        <origin xyz="0 ${sign}18.5e-3 11e-3" rpy="0 0 0"/>
+        <geometry>
+          <box size="22e-3 15e-3 20e-3" />
+        </geometry>
+      </collision>
+      <!-- cartriage sledge -->
+      <collision>
+        <origin xyz="0 ${sign}6.8e-3 2.2e-3" rpy="0 0 0"/>
+        <geometry>
+          <box size="22e-3 8.8e-3 3.8e-3" />
+        </geometry>
+      </collision>
+      <!-- diagonal finger -->
+      <collision>
+	      <origin xyz="0 ${sign}15.9e-3 28.35e-3" rpy="${sign}${pi/6} 0 0"/>
+        <geometry>
+          <box size="17.5e-3 7e-3 23.5e-3" />
+        </geometry>
+      </collision>
+      <!-- rubber tip with which to grasp -->
+      <collision>
+        <origin xyz="0 ${sign}7.58e-3 45.25e-3" rpy="0 0 0"/>
+        <geometry>
+          <box size="17.5e-3 15.2e-3 18.5e-3" />
+        </geometry>
+      </collision>
+    </xacro:macro>
     <link name="${ns}_leftfinger">
       <xacro:inertia-cylinder mass="15e-3" radius="0.01" h="0.04"/>
@@ -286,32 +316,5 @@
         </geometry>
       </visual>
-      <!-- screw mount -->
-      <collision>
-        <origin xyz="0 18.5e-3 11e-3" rpy="0 0 0"/>
-        <geometry>
-          <box size="22e-3 15e-3 20e-3" />
-        </geometry>
-      </collision>
-      <!-- cartriage sledge -->
-      <collision>
-        <origin xyz="0 6.8e-3 2.2e-3" rpy="0 0 0"/>
-        <geometry>
-          <box size="22e-3 8.8e-3 3.8e-3" />
-        </geometry>
-      </collision>
-      <!-- diagonal finger -->
-      <collision>
-        <origin xyz="0 15.9e-3 28.35e-3" rpy="${pi/6} 0 0"/>
-        <geometry>
-          <box size="17.5e-3 7e-3 23.5e-3" />
-        </geometry>
-      </collision>
-      <!-- rubber tip with which to grasp -->
-      <collision>
-        <origin xyz="0 7.58e-3 45.25e-3" rpy="0 0 0"/>
-        <geometry>
-          <box size="17.5e-3 15.2e-3 18.5e-3" />
-        </geometry>
-      </collision>
+      <xacro:finger-collision sign="+" />
     </link>
     <link name="${ns}_rightfinger">
@@ -323,32 +326,5 @@
         </geometry>
       </visual>
-      <!-- screw mount -->
-      <collision>
-        <origin xyz="0 -18.5e-3 11e-3" rpy="0 0 0"/>
-        <geometry>
-          <box size="22e-3 15e-3 20e-3" />
-        </geometry>
-      </collision>
-      <!-- cartriage sledge -->
-      <collision>
-        <origin xyz="0 -6.8e-3 2.2e-3" rpy="0 0 0"/>
-        <geometry>
-          <box size="22e-3 8.8e-3 3.8e-3" />
-        </geometry>
-      </collision>
-      <!-- diagonal finger -->
-      <collision>
-        <origin xyz="0 -15.9e-3 28.35e-3" rpy="${-pi/6} 0 0"/>
-        <geometry>
-          <box size="17.5e-3 7e-3 23.5e-3" />
-        </geometry>
-      </collision>
-      <!-- rubber tip with which to grasp -->
-      <collision>
-        <origin xyz="0 -7.58e-3 45.25e-3" rpy="0 0 0"/>
-        <geometry>
-          <box size="17.5e-3 15.2e-3 18.5e-3" />
-        </geometry>
-      </collision>
+      <xacro:finger-collision sign="-" />
     </link>
     <!-- Friction specific material for Rubber/Rubber contact -->

Commit message: feat(gazebo): add hand_tcp frame to gazebo robot description
This commit adds the `hand_tcp` frame that was defined in
97e73fabdeed69bc8deb8686f1973f0e03b6400f to the Gazebo robot
description. This frame is positioned in the center between and
aligned with the fingers.

File: franka_description/robots/panda_gazebo.xacro (robot description, xacro)
@@ -309,4 +309,11 @@
       </collision>
     </xacro:macro>
+    <!-- Define the hand_tcp frame -->
+    <link name="${ns}_hand_tcp" />
+    <joint name="${ns}_hand_tcp_joint" type="fixed">
+      <origin xyz="0 0 0.1034" rpy="0 0 0" />
+      <parent link="${ns}_hand" />
+      <child link="${ns}_hand_tcp" />
+    </joint>
     <link name="${ns}_leftfinger">
       <xacro:inertia-cylinder mass="15e-3" radius="0.01" h="0.04"/>

Commit message: Adds optional joint to connect the panda, similar to panda_arm.xacro

File: franka_description/robots/panda_gazebo.xacro (robot description, xacro)
@@ -10,5 +10,12 @@
   <!-- || Paolo Robuffo Giordano, Alessandro de Luca                || -->
   <!-- =============================================================== -->
-  <xacro:macro name="panda_arm" params="arm_id:='panda'">
+  <xacro:macro name="panda_arm" params="arm_id:='panda' connected_to=''">
+    <xacro:unless value="${not connected_to}">
+      <joint name="${arm_id}_joint_${connected_to}" type="fixed">
+        <parent link="${connected_to}"/>
+        <child link="${arm_id}_link0"/>
+        <origin rpy="0 0 0" xyz="0 0 0"/>
+      </joint>
+    </xacro:unless>
     <link name="${arm_id}_link0">
       <visual>

Commit message: ADD: `connected_to` optional arg to `panda_gazebo.xacro`
This provides a similar interface to `panda_arm.xacro`

File: franka_description/robots/panda_gazebo.xacro (robot description, xacro)
@@ -10,5 +10,12 @@
   <!-- || Paolo Robuffo Giordano, Alessandro de Luca                || -->
   <!-- =============================================================== -->
-  <xacro:macro name="panda_arm" params="arm_id:='panda'">
+  <xacro:macro name="panda_arm" params="arm_id:='panda' connected_to:='' xyz:='0 0 0' rpy:='0 0 0'">
+    <xacro:unless value="${not connected_to}">
+      <joint name="${arm_id}_joint_${connected_to}" type="fixed">
+        <parent link="${connected_to}"/>
+        <child link="${arm_id}_link0"/>
+        <origin rpy="${rpy}" xyz="${xyz}"/>
+      </joint>
+    </xacro:unless>
     <link name="${arm_id}_link0">
       <visual>
@@ -296,5 +303,5 @@
       <!-- diagonal finger -->
       <collision>
-	      <origin xyz="0 ${sign}15.9e-3 28.35e-3" rpy="${sign}${pi/6} 0 0"/>
+        <origin xyz="0 ${sign}15.9e-3 28.35e-3" rpy="${sign}${pi/6} 0 0"/>
         <geometry>
           <box size="17.5e-3 7e-3 23.5e-3" />
