Commit message: Adjust soft limits.

File: franka_description/robots/panda_arm.xacro (robot description, xacro)
@@ -44,10 +44,10 @@
     </link>
     <joint name="${arm_id}_joint1" type="revolute">
-      <safety_controller k_position="100.0" k_velocity="40.0" soft_lower_limit="-2.818745" soft_upper_limit="2.818745"/>
+      <safety_controller k_position="100.0" k_velocity="40.0" soft_lower_limit="-2.8973" soft_upper_limit="2.8973"/>
       <origin rpy="0 0 0" xyz="0 0 0.333"/>
       <parent link="${arm_id}_link0"/>
       <child link="${arm_id}_link1"/>
       <axis xyz="0 0 1"/>
-      <limit effort="87" lower="-2.9671" upper="2.9671" velocity="2.5"/>
+      <limit effort="87" lower="-2.9671" upper="2.9671" velocity="2.3925"/>
     </joint>
     <link name="${arm_id}_link2">
@@ -69,10 +69,10 @@
     </link>
     <joint name="${arm_id}_joint2" type="revolute">
-      <safety_controller k_position="100.0" k_velocity="40.0" soft_lower_limit="-1.74097" soft_upper_limit="1.74097"/>
+      <safety_controller k_position="100.0" k_velocity="40.0" soft_lower_limit="-1.7628" soft_upper_limit="1.7628"/>
       <origin rpy="-1.570796326794897 0 0" xyz="0 0 0"/>
       <parent link="${arm_id}_link1"/>
       <child link="${arm_id}_link2"/>
       <axis xyz="0 0 1"/>
-      <limit effort="87" lower="-1.8326" upper="1.8326" velocity="2.5"/>
+      <limit effort="87" lower="-1.8326" upper="1.8326" velocity="2.3925"/>
     </joint>
     <link name="${arm_id}_link3">
@@ -94,10 +94,10 @@
     </link>
     <joint name="${arm_id}_joint3" type="revolute">
-      <safety_controller k_position="100.0" k_velocity="40.0" soft_lower_limit="-2.818745" soft_upper_limit="2.818745"/>
+      <safety_controller k_position="100.0" k_velocity="40.0" soft_lower_limit="-2.8973" soft_upper_limit="2.8973"/>
       <origin rpy="1.570796326794897 0 0" xyz="0 -0.316 0"/>
       <parent link="${arm_id}_link2"/>
       <child link="${arm_id}_link3"/>
       <axis xyz="0 0 1"/>
-      <limit effort="87" lower="-2.9671" upper="2.9671" velocity="2.5"/>
+      <limit effort="87" lower="-2.9671" upper="2.9671" velocity="2.3925"/>
     </joint>
     <link name="${arm_id}_link4">
@@ -119,10 +119,10 @@
     </link>
     <joint name="${arm_id}_joint4" type="revolute">
-      <safety_controller k_position="100.0" k_velocity="40.0" soft_lower_limit="-2.98452" soft_upper_limit="0.082935"/>
+      <safety_controller k_position="100.0" k_velocity="40.0" soft_lower_limit="-3.0718" soft_upper_limit="0.0175"/>
       <origin rpy="1.570796326794897 0 0" xyz="0.0825 0 0"/>
       <parent link="${arm_id}_link3"/>
       <child link="${arm_id}_link4"/>
       <axis xyz="0 0 1"/>
-      <limit effort="87" lower="-3.1416" upper="0.0873" velocity="2.5"/>
+      <limit effort="87" lower="-3.1416" upper="0.0873" velocity="2.3925"/>
     </joint>
     <link name="${arm_id}_link5">
@@ -144,10 +144,10 @@
     </link>
     <joint name="${arm_id}_joint5" type="revolute">
-      <safety_controller k_position="100.0" k_velocity="40.0" soft_lower_limit="-2.818745" soft_upper_limit="2.818745"/>
+      <safety_controller k_position="100.0" k_velocity="40.0" soft_lower_limit="-2.8973" soft_upper_limit="2.8973"/>
       <origin rpy="-1.570796326794897 0 0" xyz="-0.0825 0.384 0"/>
       <parent link="${arm_id}_link4"/>
       <child link="${arm_id}_link5"/>
       <axis xyz="0 0 1"/>
-      <limit effort="12" lower="-2.9671" upper="2.9671" velocity="3"/>
+      <limit effort="12" lower="-2.9671" upper="2.9671" velocity="2.8710"/>
     </joint>
     <link name="${arm_id}_link6">
@@ -169,10 +169,10 @@
     </link>
     <joint name="${arm_id}_joint6" type="revolute">
-      <safety_controller k_position="100.0" k_velocity="40.0" soft_lower_limit="-0.082935" soft_upper_limit="3.631185"/>
+      <safety_controller k_position="100.0" k_velocity="40.0" soft_lower_limit="-0.0175" soft_upper_limit="3.7525"/>
       <origin rpy="1.570796326794897 0 0" xyz="0 0 0"/>
       <parent link="${arm_id}_link5"/>
       <child link="${arm_id}_link6"/>
       <axis xyz="0 0 1"/>
-      <limit effort="12" lower="-0.0873" upper="3.8223" velocity="3"/>
+      <limit effort="12" lower="-0.0873" upper="3.8223" velocity="2.8710"/>
     </joint>
     <link name="${arm_id}_link7">
@@ -194,10 +194,10 @@
     </link>
     <joint name="${arm_id}_joint7" type="revolute">
-      <safety_controller k_position="100.0" k_velocity="40.0" soft_lower_limit="-2.818745" soft_upper_limit="2.818745"/>
+      <safety_controller k_position="100.0" k_velocity="40.0" soft_lower_limit="-2.8973" soft_upper_limit="2.8973"/>
       <origin rpy="1.570796326794897 0 0" xyz="0.088 0 0"/>
       <parent link="${arm_id}_link6"/>
       <child link="${arm_id}_link7"/>
       <axis xyz="0 0 1"/>
-      <limit effort="12" lower="-2.9671" upper="2.9671" velocity="3"/>
+      <limit effort="12" lower="-2.9671" upper="2.9671" velocity="2.8710"/>
     </joint>
     <link name="${arm_id}_link8"/>

Commit message: Adjust maximum joint velocity in URDF.

File: franka_description/robots/panda_arm.xacro (robot description, xacro)
@@ -39,5 +39,5 @@
       <child link="${arm_id}_link1"/>
       <axis xyz="0 0 1"/>
-      <limit effort="87" lower="-2.9671" upper="2.9671" velocity="2.3925"/>
+      <limit effort="87" lower="-2.9671" upper="2.9671" velocity="2.1750"/>
     </joint>
     <link name="${arm_id}_link2">
@@ -59,5 +59,5 @@
       <child link="${arm_id}_link2"/>
       <axis xyz="0 0 1"/>
-      <limit effort="87" lower="-1.8326" upper="1.8326" velocity="2.3925"/>
+      <limit effort="87" lower="-1.8326" upper="1.8326" velocity="2.1750"/>
     </joint>
     <link name="${arm_id}_link3">
@@ -79,5 +79,5 @@
       <child link="${arm_id}_link3"/>
       <axis xyz="0 0 1"/>
-      <limit effort="87" lower="-2.9671" upper="2.9671" velocity="2.3925"/>
+      <limit effort="87" lower="-2.9671" upper="2.9671" velocity="2.1750"/>
     </joint>
     <link name="${arm_id}_link4">
@@ -99,5 +99,5 @@
       <child link="${arm_id}_link4"/>
       <axis xyz="0 0 1"/>
-      <limit effort="87" lower="-3.1416" upper="0.0873" velocity="2.3925"/>
+      <limit effort="87" lower="-3.1416" upper="0.0873" velocity="2.1750"/>
     </joint>
     <link name="${arm_id}_link5">
@@ -119,5 +119,5 @@
       <child link="${arm_id}_link5"/>
       <axis xyz="0 0 1"/>
-      <limit effort="12" lower="-2.9671" upper="2.9671" velocity="2.8710"/>
+      <limit effort="12" lower="-2.9671" upper="2.9671" velocity="2.6100"/>
     </joint>
     <link name="${arm_id}_link6">
@@ -139,5 +139,5 @@
       <child link="${arm_id}_link6"/>
       <axis xyz="0 0 1"/>
-      <limit effort="12" lower="-0.0873" upper="3.8223" velocity="2.8710"/>
+      <limit effort="12" lower="-0.0873" upper="3.8223" velocity="2.6100"/>
     </joint>
     <link name="${arm_id}_link7">
@@ -159,5 +159,5 @@
       <child link="${arm_id}_link7"/>
       <axis xyz="0 0 1"/>
-      <limit effort="12" lower="-2.9671" upper="2.9671" velocity="2.8710"/>
+      <limit effort="12" lower="-2.9671" upper="2.9671" velocity="2.6100"/>
     </joint>
     <link name="${arm_id}_link8"/>

Commit message: Update axis 4 hard limit in URDF.

File: franka_description/robots/panda_arm.xacro (robot description, xacro)
@@ -99,5 +99,5 @@
       <child link="${arm_id}_link4"/>
       <axis xyz="0 0 1"/>
-      <limit effort="87" lower="-3.1416" upper="0.0873" velocity="2.1750"/>
+      <limit effort="87" lower="-3.1416" upper="0.0" velocity="2.1750"/>
     </joint>
     <link name="${arm_id}_link5">

Commit message: Adjust hard limits

File: franka_description/robots/panda_arm.xacro (robot description, xacro)
@@ -39,5 +39,5 @@
       <child link="${arm_id}_link1"/>
       <axis xyz="0 0 1"/>
-      <limit effort="87" lower="-2.9671" upper="2.9671" velocity="2.1750"/>
+      <limit effort="87" lower="-2.8973" upper="2.8973" velocity="2.1750"/>
     </joint>
     <link name="${arm_id}_link2">
@@ -59,5 +59,5 @@
       <child link="${arm_id}_link2"/>
       <axis xyz="0 0 1"/>
-      <limit effort="87" lower="-1.8326" upper="1.8326" velocity="2.1750"/>
+      <limit effort="87" lower="-1.7628" upper="1.7628" velocity="2.1750"/>
     </joint>
     <link name="${arm_id}_link3">
@@ -79,5 +79,5 @@
       <child link="${arm_id}_link3"/>
       <axis xyz="0 0 1"/>
-      <limit effort="87" lower="-2.9671" upper="2.9671" velocity="2.1750"/>
+      <limit effort="87" lower="-2.8973" upper="2.8973" velocity="2.1750"/>
     </joint>
     <link name="${arm_id}_link4">
@@ -99,5 +99,5 @@
       <child link="${arm_id}_link4"/>
       <axis xyz="0 0 1"/>
-      <limit effort="87" lower="-3.1416" upper="0.0" velocity="2.1750"/>
+      <limit effort="87" lower="-3.0718" upper="-0.0698" velocity="2.1750"/>
     </joint>
     <link name="${arm_id}_link5">
@@ -119,5 +119,5 @@
       <child link="${arm_id}_link5"/>
       <axis xyz="0 0 1"/>
-      <limit effort="12" lower="-2.9671" upper="2.9671" velocity="2.6100"/>
+      <limit effort="12" lower="-2.8973" upper="2.8973" velocity="2.6100"/>
     </joint>
     <link name="${arm_id}_link6">
@@ -139,5 +139,5 @@
       <child link="${arm_id}_link6"/>
       <axis xyz="0 0 1"/>
-      <limit effort="12" lower="-0.0873" upper="3.8223" velocity="2.6100"/>
+      <limit effort="12" lower="-0.0175" upper="3.7525" velocity="2.6100"/>
     </joint>
     <link name="${arm_id}_link7">
@@ -159,5 +159,5 @@
       <child link="${arm_id}_link7"/>
       <axis xyz="0 0 1"/>
-      <limit effort="12" lower="-2.9671" upper="2.9671" velocity="2.6100"/>
+      <limit effort="12" lower="-2.8973" upper="2.8973" velocity="2.6100"/>
     </joint>
     <link name="${arm_id}_link8"/>

Commit message: Adds rcu collision volumes to robot URDF.

File: franka_description/robots/panda_arm.xacro (robot description, xacro)
@@ -16,6 +16,19 @@
       </visual>
       <collision>
-        <geometry>
-          <mesh filename="package://${description_pkg}/meshes/collision/link0.stl"/>
+        <origin xyz="-0.075 0 0.06" rpy="0 ${pi/2} 0"/>
+        <geometry>
+          <cylinder radius="0.06" length="0.03" />
+        </geometry>
+      </collision>
+      <collision>
+        <origin xyz="-0.06 0 0.06" rpy="0 0 0"/>
+        <geometry>
+          <sphere radius="0.06" />
+        </geometry>
+      </collision>
+      <collision>
+        <origin xyz="-0.09 0 0.06" rpy="0 0 0"/>
+        <geometry>
+          <sphere radius="0.06" />
         </geometry>
       </collision>
@@ -28,6 +41,19 @@
       </visual>
       <collision>
-        <geometry>
-          <mesh filename="package://${description_pkg}/meshes/collision/link1.stl"/>
+        <origin xyz="0 0 -0.1915" rpy="0 0 0"/>
+        <geometry>
+          <cylinder radius="0.06" length="0.2830" />
+        </geometry>
+      </collision>
+      <collision>
+        <origin xyz="0 0 -0.333" rpy="0 0 0"/>
+        <geometry>
+          <sphere radius="0.06" />
+        </geometry>
+      </collision>
+      <collision>
+        <origin xyz="0 0 -0.05" rpy="0 0 0"/>
+        <geometry>
+          <sphere radius="0.06" />
         </geometry>
       </collision>
@@ -48,6 +74,19 @@
       </visual>
       <collision>
-        <geometry>
-          <mesh filename="package://${description_pkg}/meshes/collision/link2.stl"/>
+        <origin xyz="0 0 0" rpy="0 0 0"/>
+        <geometry>
+          <cylinder radius="0.06" length="0.12" />
+        </geometry>
+      </collision>
+      <collision>
+        <origin xyz="0 0 -0.06" rpy="0 0 0"/>
+        <geometry>
+          <sphere radius="0.06" />
+        </geometry>
+      </collision>
+      <collision>
+        <origin xyz="0 0 0.06" rpy="0 0 0"/>
+        <geometry>
+          <sphere radius="0.06" />
         </geometry>
       </collision>
@@ -68,6 +107,19 @@
       </visual>
       <collision>
-        <geometry>
-          <mesh filename="package://${description_pkg}/meshes/collision/link3.stl"/>
+        <origin xyz="0 0 -0.145" rpy="0 0 0"/>
+        <geometry>
+          <cylinder radius="0.06" length="0.15" />
+        </geometry>
+      </collision>
+      <collision>
+        <origin xyz="0 0 -0.22" rpy="0 0 0"/>
+        <geometry>
+          <sphere radius="0.06" />
+        </geometry>
+      </collision>
+      <collision>
+        <origin xyz="0 0 -0.07" rpy="0 0 0"/>
+        <geometry>
+          <sphere radius="0.06" />
         </geometry>
       </collision>
@@ -88,6 +140,19 @@
       </visual>
       <collision>
-        <geometry>
-          <mesh filename="package://${description_pkg}/meshes/collision/link4.stl"/>
+        <origin xyz="0 0 0" rpy="0 0 0"/>
+        <geometry>
+          <cylinder radius="0.06" length="0.12" />
+        </geometry>
+      </collision>
+      <collision>
+        <origin xyz="0 0 0.06" rpy="0 0 0"/>
+        <geometry>
+          <sphere radius="0.06" />
+        </geometry>
+      </collision>
+      <collision>
+        <origin xyz="0 0 -0.06" rpy="0 0 0"/>
+        <geometry>
+          <sphere radius="0.06" />
         </geometry>
       </collision>
@@ -108,6 +173,37 @@
       </visual>
       <collision>
-        <geometry>
-          <mesh filename="package://${description_pkg}/meshes/collision/link5.stl"/>
+        <origin xyz="0 0 -0.26" rpy="0 0 0"/>
+        <geometry>
+          <cylinder radius="0.06" length="0.1" />
+        </geometry>
+      </collision>
+      <collision>
+        <origin xyz="0 0 -0.31" rpy="0 0 0"/>
+        <geometry>
+          <sphere radius="0.06" />
+        </geometry>
+      </collision>
+      <collision>
+        <origin xyz="0 0 -0.21" rpy="0 0 0"/>
+        <geometry>
+          <sphere radius="0.06" />
+        </geometry>
+      </collision>
+      <collision>
+        <origin xyz="0 0.08 -0.13" rpy="0 0 0"/>
+        <geometry>
+          <cylinder radius="0.025" length="0.14" />
+        </geometry>
+      </collision>
+      <collision>
+        <origin xyz="0 0.08 -0.06" rpy="0 0 0"/>
+        <geometry>
+          <sphere radius="0.025" />
+        </geometry>
+      </collision>
+      <collision>
+        <origin xyz="0 0.08 -0.20" rpy="0 0 0"/>
+        <geometry>
+          <sphere radius="0.025" />
         </geometry>
       </collision>
@@ -128,6 +224,19 @@
       </visual>
       <collision>
-        <geometry>
-          <mesh filename="package://${description_pkg}/meshes/collision/link6.stl"/>
+        <origin xyz="0 0 -0.03" rpy="0 0 0"/>
+        <geometry>
+          <cylinder radius="0.05" length="0.08" />
+        </geometry>
+      </collision>
+      <collision>
+        <origin xyz="0 0 0.01" rpy="0 0 0"/>
+        <geometry>
+          <sphere radius="0.05" />
+        </geometry>
+      </collision>
+      <collision>
+        <origin xyz="0 0 -0.07" rpy="0 0 0"/>
+        <geometry>
+          <sphere radius="0.05" />
         </geometry>
       </collision>
@@ -148,6 +257,19 @@
       </visual>
       <collision>
-        <geometry>
-          <mesh filename="package://${description_pkg}/meshes/collision/link7.stl"/>
+        <origin xyz="0 0 0.01" rpy="0 0 0"/>
+        <geometry>
+          <cylinder radius="0.04" length="0.14" />
+        </geometry>
+      </collision>
+      <collision>
+        <origin xyz="0 0 0.08" rpy="0 0 0"/>
+        <geometry>
+          <sphere radius="0.04" />
+        </geometry>
+      </collision>
+      <collision>
+        <origin xyz="0 0 -0.06" rpy="0 0 0"/>
+        <geometry>
+          <sphere radius="0.04" />
         </geometry>
       </collision>
@@ -161,5 +283,24 @@
       <limit effort="12" lower="-2.8973" upper="2.8973" velocity="2.6100"/>
     </joint>
-    <link name="${arm_id}_link8"/>
+    <link name="${arm_id}_link8">
+      <collision>
+        <origin xyz="0.0424 0.0424 -0.0250" rpy="${-pi/4} ${pi/2} 0"/>
+        <geometry>
+          <cylinder radius="0.03" length="0.01" />
+        </geometry>
+      </collision>
+      <collision>
+        <origin xyz="0.0424 0.0424 -0.02" rpy="0 0 0"/>
+        <geometry>
+          <sphere radius="0.03" />
+        </geometry>
+      </collision>
+      <collision>
+        <origin xyz="0.0424 0.0424 -0.03" rpy="0 0 0"/>
+        <geometry>
+          <sphere radius="0.03" />
+        </geometry>
+      </collision>
+    </link>
     <joint name="${arm_id}_joint8" type="fixed">
       <origin rpy="0 0 0" xyz="0 0 0.107"/>

Commit message: changes link 7 collision volume to an equivalent description.

File: franka_description/robots/panda_arm.xacro (robot description, xacro)
@@ -285,5 +285,5 @@
     <link name="${arm_id}_link8">
       <collision>
-        <origin xyz="0.0424 0.0424 -0.0250" rpy="${-pi/4} ${pi/2} 0"/>
+        <origin xyz="0.0424 0.0424 -0.0250" rpy="${pi} ${pi/2} ${pi/2}"/>
         <geometry>
           <cylinder radius="0.03" length="0.01" />

Commit message: Adds inital value to safety_distance in panda_arm.xacro

File: franka_description/robots/panda_arm.xacro (robot description, xacro)
@@ -1,5 +1,5 @@
 <?xml version='1.0' encoding='utf-8'?>
 <robot xmlns:xacro="http://www.ros.org/wiki/xacro" name="panda">
-  <xacro:macro name="panda_arm" params="arm_id:='panda' description_pkg:='franka_description' connected_to:='' xyz:='0 0 0' rpy:='0 0 0' safety_distance:=''">
+  <xacro:macro name="panda_arm" params="arm_id:='panda' description_pkg:='franka_description' connected_to:='' xyz:='0 0 0' rpy:='0 0 0' safety_distance:='0'">
     <xacro:unless value="${not connected_to}">
       <joint name="${arm_id}_joint_${connected_to}" type="fixed">

Commit message: :sparkles: Adds more realistic inertias, masses and damping ratios to the robot description

File: franka_description/robots/panda_arm.xacro (robot description, xacro)
@@ -9,4 +9,23 @@
       </joint>
     </xacro:unless>
+    <!-- Masses, COG and inertias -->
+    <xacro:property name="link0_mass" value="3.06357" />
+    <xacro:property name="link1_mass" value="2.34471" />
+    <xacro:property name="link2_mass" value="2.36414" />
+    <xacro:property name="link3_mass" value="2.38050" />
+    <xacro:property name="link4_mass" value="2.42754" />
+    <xacro:property name="link5_mass" value="3.49611" />
+    <xacro:property name="link6_mass" value="1.46736" />
+    <xacro:property name="link7_mass" value="0.45606" />
+    <xacro:property name="link8_mass" value="0.001" /> --
+    <xacro:property name="link0_cog" value="-0.029190 -0.000879 0.056603" />
+    <xacro:property name="link1_cog" value="0.000011 -0.031266 -0.069373" />
+    <xacro:property name="link2_cog" value="-0.000013 -0.070322 0.031178" />
+    <xacro:property name="link3_cog" value="0.044348 0.024928 -0.038130" />
+    <xacro:property name="link4_cog" value="-0.038550 0.039526 0.024716" />
+    <xacro:property name="link5_cog" value="-0.000064 0.038412 -0.109970" />
+    <xacro:property name="link6_cog" value="0.051002 0.006933 0.006169" />
+    <xacro:property name="link7_cog" value="0.010361 0.010360 0.079108" />
+    <xacro:property name="link8_cog" value="0.0 0.0 0.0" />
     <!-- for simulation -->
     <link name="world" />
@@ -31,7 +50,7 @@
       <!-- for simulation -->
       <inertial>
-        <origin xyz="0 0 0" rpy="0 0 0" />
-        <mass value="3.06" />
-        <inertia ixx="0.3" ixy="0.0" ixz="0.0" iyy="0.3" iyz="0.0" izz="0.3" />
+        <origin xyz="${link0_cog}" rpy="0 0 0" />
+        <mass value="${link0_mass}" />
+        <inertia ixx="0.009" iyy="0.0122" izz="0.0122" ixy="0.0" ixz="-0.00010" iyz="0.0" />
       </inertial>
       <!-- end for simulation -->
@@ -50,7 +69,7 @@
       <!-- for simulation -->
       <inertial>
-        <origin xyz="0 0 0" rpy="0 0 0" />
-        <mass value="2.34" />
-        <inertia ixx="0.3" ixy="0.0" ixz="0.0" iyy="0.3" iyz="0.0" izz="0.3" />
+        <origin xyz="${link1_cog}" rpy="0 0 0" />
+        <mass value="${link1_mass}" />
+        <inertia ixx="0.01418" iyy="0.01181" izz="0.005515" ixy="0.0" ixz="0.0" iyz="0.00236" />
       </inertial>
       <!-- end for simulation -->
@@ -80,7 +99,7 @@
       <!-- for simulation -->
       <inertial>
-        <origin xyz="0 0 0" rpy="0 0 0" />
-        <mass value="2.36" />
-        <inertia ixx="0.3" ixy="0.0" ixz="0.0" iyy="0.3" iyz="0.0" izz="0.3" />
+        <origin xyz="${link2_cog}" rpy="0 0 0" />
+        <mass value="${link2_mass}" />
+        <inertia ixx="0.014" ixy="0.0" ixz="0.0" iyy="0.0055" iyz="-0.0023" izz="0.01259" />
       </inertial>
       <!-- end for simulation -->
@@ -110,7 +129,7 @@
       <!-- for simulation -->
       <inertial>
-        <origin xyz="0 0 0" rpy="0 0 0" />
-        <mass value="2.38" />
-        <inertia ixx="0.3" ixy="0.0" ixz="0.0" iyy="0.3" iyz="0.0" izz="0.3" />
+        <origin xyz="${link3_cog}" rpy="0 0 0" />
+        <mass value="${link3_mass}" />
+        <inertia ixx="0.00716" ixy="-0.00102" ixz="-0.02040" iyy="0.00920" iyz="-0.00102" izz="0.007159" />
       </inertial>
       <!-- end for simulation -->
@@ -140,7 +159,7 @@
       <!-- for simulation -->
       <inertial>
-        <origin xyz="0 0 0" rpy="0 0 0" />
-        <mass value="2.43" />
-        <inertia ixx="0.3" ixy="0.0" ixz="0.0" iyy="0.3" iyz="0.0" izz="0.3" />
+        <origin xyz="${link4_cog}" rpy="0 0 0" />
+        <mass value="${link4_mass}" />
+        <inertia ixx="0.008164" ixy="0.003061" ixz="0.00102" iyy="0.008165" iyz="0.00102" izz="0.009185" />
       </inertial>
       <!-- end for simulation -->
@@ -170,7 +189,7 @@
       <!-- for simulation -->
       <inertial>
-        <origin xyz="0 0 0" rpy="0 0 0" />
-        <mass value="3.5" />
-        <inertia ixx="0.3" ixy="0.0" ixz="0.0" iyy="0.3" iyz="0.0" izz="0.3" />
+        <origin xyz="${link5_cog}" rpy="0 0 0" />
+        <mass value="${link5_mass}" />
+        <inertia ixx="0.0307" ixy="0.0" ixz="0.0" iyy="0.02761" iyz="-0.0613" izz="0.00818" />
       </inertial>
       <!-- end for simulation -->
@@ -200,7 +219,7 @@
       <!-- for simulation -->
       <inertial>
-        <origin xyz="0 0 0" rpy="0 0 0" />
-        <mass value="1.47" />
-        <inertia ixx="0.3" ixy="0.0" ixz="0.0" iyy="0.3" iyz="0.0" izz="0.3" />
+        <origin xyz="${link6_cog}" rpy="0 0 0" />
+        <mass value="${link6_mass}" />
+        <inertia ixx="0.00205" ixy="0.0" ixz="0.0" iyy="0.004089" iyz="0" izz="0.00490" />
       </inertial>
       <!-- end for simulation -->
@@ -230,6 +249,6 @@
       <!-- for simulation -->
       <inertial>
-        <origin xyz="0 0 0" rpy="0 0 0" />
-        <mass value="0.45" />
+        <origin xyz="${link7_cog}" rpy="0 0 0" />
+        <mass value="${link7_mass}" />
         <inertia ixx="0.3" ixy="0.0" ixz="0.0" iyy="0.3" iyz="0.0" izz="0.3" />
       </inertial>
@@ -250,6 +269,6 @@
       <!-- for simulation -->
       <inertial>
-        <origin xyz="0 0 0" rpy="0 0 0" />
-        <mass value="0.0" />
+        <origin xyz="${link8_cog}" rpy="0 0 0" />
+        <mass value="${link8_mass}" />
         <inertia ixx="0.3" ixy="0.0" ixz="0.0" iyy="0.3" iyz="0.0" izz="0.3" />
       </inertial>
