Commit message: Update and improve usage

File: franka_description/robots/panda_arm.xacro (robot description, xacro)
@@ -2,20 +2,13 @@
 <robot xmlns:xacro="http://www.ros.org/wiki/xacro" name="panda">
   <xacro:macro name="panda_arm" params="arm_id:='panda' description_pkg:='franka_description' connected_to:='' xyz:='0 0 0' rpy:='0 0 0'">
+    <link name="world" />
     <xacro:unless value="${not connected_to}">
-      <joint name="${arm_id}_joint_${connected_to}" type="fixed">
+      <joint name="virtual_joint" type="fixed">
         <parent link="${connected_to}"/>
         <child link="${arm_id}_link0"/>
         <origin rpy="${rpy}" xyz="${xyz}"/>
+        <dynamics damping="1.0"/>
       </joint>
     </xacro:unless>
-    <!-- for simulation -->
-    <link name="world" />
-    <joint name="robot_to_world" type="fixed">
-      <parent link="world" />
-      <child link="${arm_id}_link0" />
-      <origin xyz="0.0 0.0 0.0" rpy="0.0 0.0 0.0" />
-    </joint>
-    <xacro:property name="joint_damping" value="1.0"/>
-    <!-- end for simulation -->
     <link name="${arm_id}_link0">
       <visual>
@@ -64,5 +57,5 @@
       <limit effort="87" lower="-2.8973" upper="2.8973" velocity="2.1750"/>
       <!-- for simulation -->
-      <dynamics damping="${joint_damping}"/>
+      <dynamics damping="1.0"/>
       <!-- end for simulation -->
     </joint>
@@ -94,5 +87,5 @@
       <limit effort="87" lower="-1.7628" upper="1.7628" velocity="2.1750"/>
       <!-- for simulation -->
-      <dynamics damping="${joint_damping}"/>
+      <dynamics damping="1.0"/>
       <!-- end for simulation -->
     </joint>
@@ -124,5 +117,5 @@
       <limit effort="87" lower="-2.8973" upper="2.8973" velocity="2.1750"/>
       <!-- for simulation -->
-      <dynamics damping="${joint_damping}"/>
+      <dynamics damping="1.0"/>
       <!-- end for simulation -->
     </joint>
@@ -154,5 +147,5 @@
       <limit effort="87" lower="-3.0718" upper="-0.0698" velocity="2.1750"/>
       <!-- for simulation -->
-      <dynamics damping="${joint_damping}"/>
+      <dynamics damping="1.0"/>
       <!-- end for simulation -->
     </joint>
@@ -184,5 +177,5 @@
       <limit effort="12" lower="-2.8973" upper="2.8973" velocity="2.6100"/>
       <!-- for simulation -->
-      <dynamics damping="${joint_damping}"/>
+      <dynamics damping="1.0"/>
       <!-- end for simulation -->
     </joint>
@@ -214,5 +207,5 @@
       <limit effort="12" lower="-0.0175" upper="3.7525" velocity="2.6100"/>
       <!-- for simulation -->
-      <dynamics damping="${joint_damping}"/>
+      <dynamics damping="1.0"/>
       <!-- end for simulation -->
     </joint>
@@ -244,5 +237,5 @@
       <limit effort="12" lower="-2.8973" upper="2.8973" velocity="2.6100"/>
       <!-- for simulation -->
-      <dynamics damping="${joint_damping}"/>
+      <dynamics damping="1.0"/>
       <!-- end for simulation -->
     </joint>

File: franka_description/robots/panda_arm_hand.urdf.xacro (robot description, xacro)
@@ -5,12 +5,11 @@
   <!-- for simulation -->
   <xacro:include filename="$(find franka_description)/robots/panda.gazebo.xacro"/>
-  <xacro:include filename="panda.transmission.xacro"/>
+  <xacro:include filename="$(find franka_description)/robots/panda.control.xacro"/>
   <!-- end for simulation -->
-  <xacro:panda_arm />
+  <xacro:panda_arm xyz="0 0 0" rpy="0 0 0" connected_to="world" arm_id="panda"/>
   <xacro:hand ns="panda" rpy="0 0 ${-pi/4}" connected_to="panda_link8"/>
   <!-- for simulation -->
-  <xacro:arg name="robot_name" default="panda"/>
-  <xacro:panda_gazebo robot_name="$(arg robot_name)" />
-  <xacro:panda_transmission robot_name="$(arg robot_name)" load_hand="true" />
+  <xacro:panda_gazebo arm_id="panda"/>
+  <xacro:panda_control arm_id="panda" load_hand="true" />
   <!-- end for simulation -->
 </robot>

Commit message: Create macro for joints and links.

File: franka_description/robots/panda_arm.xacro (robot description, xacro)
@@ -8,251 +8,94 @@
         <child link="${arm_id}_link0"/>
         <origin rpy="${rpy}" xyz="${xyz}"/>
+        <!-- for simulation -->
+        <dynamics damping="1.0"/>
+        <!-- end for simulation -->
+      </joint>
+    </xacro:unless>
+    <xacro:macro name="arm_link" params="name visual_mesh:='' collision_mesh:='' mass:='0.0'">
+      <link name="${name}">
+        <xacro:unless value="${not visual_mesh}">
+          <visual>
+            <geometry>
+              <mesh filename="${visual_mesh}"/>
+            </geometry>
+          </visual>
+        </xacro:unless>
+        <xacro:unless value="${not collision_mesh}">
+          <collision>
+            <geometry>
+              <mesh filename="${collision_mesh}"/>
+            </geometry>
+          </collision>
+        </xacro:unless>
+        <!-- for simulation -->
+        <inertial>
+          <origin xyz="0 0 0" rpy="0 0 0" />
+          <mass value="${mass}"/>
+          <inertia ixx="0.3" ixy="0.0" ixz="0.0" iyy="0.3" iyz="0.0" izz="0.3" />
+        </inertial>
+        <!-- end for simulation -->
+      </link>
+    </xacro:macro>
+    <xacro:macro name="arm_joint" params="name type:='fixed' rpy xyz soft_lower_limit:='' soft_upper_limit:=''
+                            parent_link child_link limit_effort:='' limit_lower:='' limit_upper:='' limit_velocity:=''">
+      <joint name="${name}" type="${type}">
+        <xacro:if value="${type == 'revolute'}">
+          <safety_controller k_position="100.0" k_velocity="40.0"
+            soft_lower_limit="${soft_lower_limit}" soft_upper_limit="${soft_upper_limit}"/>
+        </xacro:if>
+        <origin rpy="${rpy}" xyz="${xyz}"/>
+        <parent link="${parent_link}"/>
+        <child link="${child_link}"/>
+        <xacro:if value="${type == 'revolute'}">
+          <limit effort="${limit_effort}" lower="${limit_lower}" upper="${limit_upper}" velocity="${limit_velocity}"/>
+          <axis xyz="0 0 1"/>
+        </xacro:if>
+        <xacro:if value="${type == 'fixed'}">
+          <axis xyz="0 0 0"/>
+        </xacro:if>
         <dynamics damping="1.0"/>
       </joint>
-    </xacro:unless>
-    <link name="${arm_id}_link0">
-      <visual>
-        <geometry>
-          <mesh filename="package://${description_pkg}/meshes/visual/link0.dae"/>
-        </geometry>
-      </visual>
-      <collision>
-        <geometry>
-          <mesh filename="package://${description_pkg}/meshes/collision/link0.stl"/>
-        </geometry>
-      </collision>
-      <!-- for simulation -->
-      <inertial>
-        <origin xyz="0 0 0" rpy="0 0 0" />
-        <mass value="3.06" />
-        <inertia ixx="0.3" ixy="0.0" ixz="0.0" iyy="0.3" iyz="0.0" izz="0.3" />
-      </inertial>
-      <!-- end for simulation -->
-    </link>
-    <link name="${arm_id}_link1">
-      <visual>
-        <geometry>
-          <mesh filename="package://${description_pkg}/meshes/visual/link1.dae"/>
-        </geometry>
-      </visual>
-      <collision>
-        <geometry>
-          <mesh filename="package://${description_pkg}/meshes/collision/link1.stl"/>
-        </geometry>
-      </collision>
-      <!-- for simulation -->
-      <inertial>
-        <origin xyz="0 0 0" rpy="0 0 0" />
-        <mass value="2.34" />
-        <inertia ixx="0.3" ixy="0.0" ixz="0.0" iyy="0.3" iyz="0.0" izz="0.3" />
-      </inertial>
-      <!-- end for simulation -->
-    </link>
-    <joint name="${arm_id}_joint1" type="revolute">
-      <safety_controller k_position="100.0" k_velocity="40.0" soft_lower_limit="-2.8973" soft_upper_limit="2.8973"/>
-      <origin rpy="0 0 0" xyz="0 0 0.333"/>
-      <parent link="${arm_id}_link0"/>
-      <child link="${arm_id}_link1"/>
-      <axis xyz="0 0 1"/>
-      <limit effort="87" lower="-2.8973" upper="2.8973" velocity="2.1750"/>
-      <!-- for simulation -->
-      <dynamics damping="1.0"/>
-      <!-- end for simulation -->
-    </joint>
-    <link name="${arm_id}_link2">
-      <visual>
-        <geometry>
-          <mesh filename="package://${description_pkg}/meshes/visual/link2.dae"/>
-        </geometry>
-      </visual>
-      <collision>
-        <geometry>
-          <mesh filename="package://${description_pkg}/meshes/collision/link2.stl"/>
-        </geometry>
-      </collision>
-      <!-- for simulation -->
-      <inertial>
-        <origin xyz="0 0 0" rpy="0 0 0" />
-        <mass value="2.36" />
-        <inertia ixx="0.3" ixy="0.0" ixz="0.0" iyy="0.3" iyz="0.0" izz="0.3" />
-      </inertial>
-      <!-- end for simulation -->
-    </link>
-    <joint name="${arm_id}_joint2" type="revolute">
-      <safety_controller k_position="100.0" k_velocity="40.0" soft_lower_limit="-1.7628" soft_upper_limit="1.7628"/>
-      <origin rpy="${-pi/2} 0 0" xyz="0 0 0"/>
-      <parent link="${arm_id}_link1"/>
-      <child link="${arm_id}_link2"/>
-      <axis xyz="0 0 1"/>
-      <limit effort="87" lower="-1.7628" upper="1.7628" velocity="2.1750"/>
-      <!-- for simulation -->
-      <dynamics damping="1.0"/>
-      <!-- end for simulation -->
-    </joint>
-    <link name="${arm_id}_link3">
-      <visual>
-        <geometry>
-          <mesh filename="package://${description_pkg}/meshes/visual/link3.dae"/>
-        </geometry>
-      </visual>
-      <collision>
-        <geometry>
-          <mesh filename="package://${description_pkg}/meshes/collision/link3.stl"/>
-        </geometry>
-      </collision>
-      <!-- for simulation -->
-      <inertial>
-        <origin xyz="0 0 0" rpy="0 0 0" />
-        <mass value="2.38" />
-        <inertia ixx="0.3" ixy="0.0" ixz="0.0" iyy="0.3" iyz="0.0" izz="0.3" />
-      </inertial>
-      <!-- end for simulation -->
-    </link>
-    <joint name="${arm_id}_joint3" type="revolute">
-      <safety_controller k_position="100.0" k_velocity="40.0" soft_lower_limit="-2.8973" soft_upper_limit="2.8973"/>
-      <origin rpy="${pi/2} 0 0" xyz="0 -0.316 0"/>
-      <parent link="${arm_id}_link2"/>
-      <child link="${arm_id}_link3"/>
-      <axis xyz="0 0 1"/>
-      <limit effort="87" lower="-2.8973" upper="2.8973" velocity="2.1750"/>
-      <!-- for simulation -->
-      <dynamics damping="1.0"/>
-      <!-- end for simulation -->
-    </joint>
-    <link name="${arm_id}_link4">
-      <visual>
-        <geometry>
-          <mesh filename="package://${description_pkg}/meshes/visual/link4.dae"/>
-        </geometry>
-      </visual>
-      <collision>
-        <geometry>
-          <mesh filename="package://${description_pkg}/meshes/collision/link4.stl"/>
-        </geometry>
-      </collision>
-      <!-- for simulation -->
-      <inertial>
-        <origin xyz="0 0 0" rpy="0 0 0" />
-        <mass value="2.43" />
-        <inertia ixx="0.3" ixy="0.0" ixz="0.0" iyy="0.3" iyz="0.0" izz="0.3" />
-      </inertial>
-      <!-- end for simulation -->
-    </link>
-    <joint name="${arm_id}_joint4" type="revolute">
-      <safety_controller k_position="100.0" k_velocity="40.0" soft_lower_limit="-3.0718" soft_upper_limit="-0.0698"/>
-      <origin rpy="${pi/2} 0 0" xyz="0.0825 0 0"/>
-      <parent link="${arm_id}_link3"/>
-      <child link="${arm_id}_link4"/>
-      <axis xyz="0 0 1"/>
-      <limit effort="87" lower="-3.0718" upper="-0.0698" velocity="2.1750"/>
-      <!-- for simulation -->
-      <dynamics damping="1.0"/>
-      <!-- end for simulation -->
-    </joint>
-    <link name="${arm_id}_link5">
-      <visual>
-        <geometry>
-          <mesh filename="package://${description_pkg}/meshes/visual/link5.dae"/>
-        </geometry>
-      </visual>
-      <collision>
-        <geometry>
-          <mesh filename="package://${description_pkg}/meshes/collision/link5.stl"/>
-        </geometry>
-      </collision>
-      <!-- for simulation -->
-      <inertial>
-        <origin xyz="0 0 0" rpy="0 0 0" />
-        <mass value="3.5" />
-        <inertia ixx="0.3" ixy="0.0" ixz="0.0" iyy="0.3" iyz="0.0" izz="0.3" />
-      </inertial>
-      <!-- end for simulation -->
-    </link>
-    <joint name="${arm_id}_joint5" type="revolute">
-      <safety_controller k_position="100.0" k_velocity="40.0" soft_lower_limit="-2.8973" soft_upper_limit="2.8973"/>
-      <origin rpy="${-pi/2} 0 0" xyz="-0.0825 0.384 0"/>
-      <parent link="${arm_id}_link4"/>
-      <child link="${arm_id}_link5"/>
-      <axis xyz="0 0 1"/>
-      <limit effort="12" lower="-2.8973" upper="2.8973" velocity="2.6100"/>
-      <!-- for simulation -->
-      <dynamics damping="1.0"/>
-      <!-- end for simulation -->
-    </joint>
-    <link name="${arm_id}_link6">
-      <visual>
-        <geometry>
-          <mesh filename="package://${description_pkg}/meshes/visual/link6.dae"/>
-        </geometry>
-      </visual>
-      <collision>
-        <geometry>
-          <mesh filename="package://${description_pkg}/meshes/collision/link6.stl"/>
-        </geometry>
-      </collision>
-      <!-- for simulation -->
-      <inertial>
-        <origin xyz="0 0 0" rpy="0 0 0" />
-        <mass value="1.47" />
-        <inertia ixx="0.3" ixy="0.0" ixz="0.0" iyy="0.3" iyz="0.0" izz="0.3" />
-      </inertial>
-      <!-- end for simulation -->
-    </link>
-    <joint name="${arm_id}_joint6" type="revolute">
-      <safety_controller k_position="100.0" k_velocity="40.0" soft_lower_limit="-0.0175" soft_upper_limit="3.7525"/>
-      <origin rpy="${pi/2} 0 0" xyz="0 0 0"/>
-      <parent link="${arm_id}_link5"/>
-      <child link="${arm_id}_link6"/>
-      <axis xyz="0 0 1"/>
-      <limit effort="12" lower="-0.0175" upper="3.7525" velocity="2.6100"/>
-      <!-- for simulation -->
-      <dynamics damping="1.0"/>
-      <!-- end for simulation -->
-    </joint>
-    <link name="${arm_id}_link7">
-      <visual>
-        <geometry>
-          <mesh filename="package://${description_pkg}/meshes/visual/link7.dae"/>
-        </geometry>
-      </visual>
-      <collision>
-        <geometry>
-          <mesh filename="package://${description_pkg}/meshes/collision/link7.stl"/>
-        </geometry>
-      </collision>
-      <!-- for simulation -->
-      <inertial>
-        <origin xyz="0 0 0" rpy="0 0 0" />
-        <mass value="0.45" />
-        <inertia ixx="0.3" ixy="0.0" ixz="0.0" iyy="0.3" iyz="0.0" izz="0.3" />
-      </inertial>
-      <!-- end for simulation -->
-    </link>
-    <joint name="${arm_id}_joint7" type="revolute">
-      <safety_controller k_position="100.0" k_velocity="40.0" soft_lower_limit="-2.8973" soft_upper_limit="2.8973"/>
-      <origin rpy="${pi/2} 0 0" xyz="0.088 0 0"/>
-      <parent link="${arm_id}_link6"/>
-      <child link="${arm_id}_link7"/>
-      <axis xyz="0 0 1"/>
-      <limit effort="12" lower="-2.8973" upper="2.8973" velocity="2.6100"/>
-      <!-- for simulation -->
-      <dynamics damping="1.0"/>
-      <!-- end for simulation -->
-    </joint>
-    <link name="${arm_id}_link8">
-      <!-- for simulation -->
-      <inertial>
-        <origin xyz="0 0 0" rpy="0 0 0" />
-        <mass value="0.0" />
-        <inertia ixx="0.3" ixy="0.0" ixz="0.0" iyy="0.3" iyz="0.0" izz="0.3" />
-      </inertial>
-      <!-- end for simulation -->
-    </link>
-    <joint name="${arm_id}_joint8" type="fixed">
-      <origin rpy="0 0 0" xyz="0 0 0.107"/>
-      <parent link="${arm_id}_link7"/>
-      <child link="${arm_id}_link8"/>
-      <axis xyz="0 0 0"/>
-    </joint>
+    </xacro:macro>
+    <xacro:arm_link name="${arm_id}_link0" visual_mesh="package://${description_pkg}/meshes/visual/link0.dae"
+      collision_mesh="package://${description_pkg}/meshes/collision/link0.stl" mass="3.06"/>
+    <xacro:arm_link name="${arm_id}_link1" visual_mesh="package://${description_pkg}/meshes/visual/link1.dae"
+      collision_mesh="package://${description_pkg}/meshes/collision/link1.stl" mass="2.34"/>
+    <xacro:arm_link name="${arm_id}_link2" visual_mesh="package://${description_pkg}/meshes/visual/link2.dae"
+      collision_mesh="package://${description_pkg}/meshes/collision/link2.stl" mass="2.36"/>
+    <xacro:arm_link name="${arm_id}_link3" visual_mesh="package://${description_pkg}/meshes/visual/link3.dae"
+      collision_mesh="package://${description_pkg}/meshes/collision/link3.stl" mass="2.38"/>
+    <xacro:arm_link name="${arm_id}_link4" visual_mesh="package://${description_pkg}/meshes/visual/link4.dae"
+      collision_mesh="package://${description_pkg}/meshes/collision/link4.stl" mass="2.43"/>
+    <xacro:arm_link name="${arm_id}_link5" visual_mesh="package://${description_pkg}/meshes/visual/link5.dae"
+      collision_mesh="package://${description_pkg}/meshes/collision/link5.stl" mass="3.5"/>
+    <xacro:arm_link name="${arm_id}_link6" visual_mesh="package://${description_pkg}/meshes/visual/link6.dae"
+      collision_mesh="package://${description_pkg}/meshes/collision/link6.stl" mass="1.47"/>
+    <xacro:arm_link name="${arm_id}_link7" visual_mesh="package://${description_pkg}/meshes/visual/link7.dae"
+      collision_mesh="package://${description_pkg}/meshes/collision/link7.stl" mass="0.45"/>
+     <xacro:arm_link name="${arm_id}_link8"/>
+    <xacro:arm_joint name="${arm_id}_joint1" type="revolute" soft_lower_limit="-2.8973" soft_upper_limit="2.8973"
+      rpy="0 0 0" xyz="0 0 0.333" parent_link="${arm_id}_link0" child_link="${arm_id}_link1" limit_effort="87"
+      limit_lower="-2.8973" limit_upper="2.8973" limit_velocity="2.1750"/>
+    <xacro:arm_joint name="${arm_id}_joint2" type="revolute" soft_lower_limit="-1.7628" soft_upper_limit="1.7628"
+      rpy="${-pi/2} 0 0" xyz="0 0 0" parent_link="${arm_id}_link1" child_link="${arm_id}_link2" limit_effort="87"
+      limit_lower="-1.7628" limit_upper="1.7628" limit_velocity="2.1750"/>
+    <xacro:arm_joint name="${arm_id}_joint3" type="revolute" soft_lower_limit="-2.8973" soft_upper_limit="2.8973"
+      rpy="${pi/2} 0 0" xyz="0 -0.316 0" parent_link="${arm_id}_link2" child_link="${arm_id}_link3" limit_effort="87"
+      limit_lower="-2.8973" limit_upper="2.8973" limit_velocity="2.1750"/>
+    <xacro:arm_joint name="${arm_id}_joint4" type="revolute" soft_lower_limit="-3.0718" soft_upper_limit="-0.0698"
+      rpy="${pi/2} 0 0" xyz="0.0825 0 0" parent_link="${arm_id}_link3" child_link="${arm_id}_link4" limit_effort="87"
+      limit_lower="-3.0718" limit_upper="-0.0698" limit_velocity="2.1750"/>
+    <xacro:arm_joint name="${arm_id}_joint5" type="revolute" soft_lower_limit="-2.8973" soft_upper_limit="2.8973"
+      rpy="${-pi/2} 0 0" xyz="-0.0825 0.384 0" parent_link="${arm_id}_link4" child_link="${arm_id}_link5" limit_effort="12"
+      limit_lower="-2.8973" limit_upper="2.8973" limit_velocity="2.6100"/>
+    <xacro:arm_joint name="${arm_id}_joint6" type="revolute" soft_lower_limit="-0.0175" soft_upper_limit="3.7525"
+      rpy="${pi/2} 0 0" xyz="0 0 0" parent_link="${arm_id}_link5" child_link="${arm_id}_link6" limit_effort="12"
+      limit_lower="-0.0175" limit_upper="3.7525" limit_velocity="2.6100"/>
+    <xacro:arm_joint name="${arm_id}_joint7" type="revolute" soft_lower_limit="-2.8973" soft_upper_limit="2.8973"
+      rpy="${pi/2} 0 0" xyz="0.088 0 0" parent_link="${arm_id}_link6" child_link="${arm_id}_link7" limit_effort="12"
+      limit_lower="-2.8973" limit_upper="2.8973" limit_velocity="2.6100"/>
+    <xacro:arm_joint name="${arm_id}_joint8" type="fixed" parent_link="${arm_id}_link7" child_link="${arm_id}_link8"
+      rpy="0 0 0" xyz="0 0 0.107"/>
   </xacro:macro>
 </robot>
