Commit message: CHANGE: Use new `<xacro:collision_capsule>` macro for self collision geometries

File: franka_description/robots/panda_arm.xacro (robot description, xacro)
@@ -13,44 +13,10 @@
     <xacro:link_detailed_coarse name="link0">
       <self_collision_geometries>
-        <collision>
-          <origin xyz="-0.075 0 0.06" rpy="0 ${pi/2} 0" />
-          <geometry>
-            <cylinder radius="${0.06+safety_distance}" length="0.03" />
-          </geometry>
-        </collision>
-        <collision>
-          <origin xyz="-0.06 0 0.06" rpy="0 0 0" />
-          <geometry>
-            <sphere radius="${0.06+safety_distance}" />
-          </geometry>
-        </collision>
-        <collision>
-          <origin xyz="-0.09 0 0.06" rpy="0 0 0" />
-          <geometry>
-            <sphere radius="${0.06+safety_distance}" />
-          </geometry>
-        </collision>
+        <xacro:collision_capsule xyz="-0.075 0 0.06" direction="x" radius="${0.06+safety_distance}" length="0.03" />
       </self_collision_geometries>
     </xacro:link_detailed_coarse>
     <xacro:link_detailed_coarse name="link1">
       <self_collision_geometries>
-        <collision>
-          <origin xyz="0 0 -0.1915" rpy="0 0 0" />
-          <geometry>
-            <cylinder radius="${0.06+safety_distance}" length="0.2830" />
-          </geometry>
-        </collision>
-        <collision>
-          <origin xyz="0 0 -0.333" rpy="0 0 0" />
-          <geometry>
-            <sphere radius="${0.06+safety_distance}" />
-          </geometry>
-        </collision>
-        <collision>
-          <origin xyz="0 0 -0.05" rpy="0 0 0" />
-          <geometry>
-            <sphere radius="${0.06+safety_distance}" />
-          </geometry>
-        </collision>
+        <xacro:collision_capsule xyz="0 0 -191.5e-3" radius="${0.06+safety_distance}" length="0.283" />
       </self_collision_geometries>
     </xacro:link_detailed_coarse>
@@ -66,22 +32,5 @@
     <xacro:link_detailed_coarse name="link2">
       <self_collision_geometries>
-        <collision>
-          <origin xyz="0 0 0" rpy="0 0 0" />
-          <geometry>
-            <cylinder radius="${0.06+safety_distance}" length="0.12" />
-          </geometry>
-        </collision>
-        <collision>
-          <origin xyz="0 0 -0.06" rpy="0 0 0" />
-          <geometry>
-            <sphere radius="${0.06+safety_distance}" />
-          </geometry>
-        </collision>
-        <collision>
-          <origin xyz="0 0 0.06" rpy="0 0 0" />
-          <geometry>
-            <sphere radius="${0.06+safety_distance}" />
-          </geometry>
-        </collision>
+        <xacro:collision_capsule xyz="0 0 0" radius="${0.06+safety_distance}" length="0.12" />
       </self_collision_geometries>
     </xacro:link_detailed_coarse>
@@ -97,22 +46,5 @@
     <xacro:link_detailed_coarse name="link3">
       <self_collision_geometries>
-        <collision>
-          <origin xyz="0 0 -0.145" rpy="0 0 0" />
-          <geometry>
-            <cylinder radius="${0.06+safety_distance}" length="0.15" />
-          </geometry>
-        </collision>
-        <collision>
-          <origin xyz="0 0 -0.22" rpy="0 0 0" />
-          <geometry>
-            <sphere radius="${0.06+safety_distance}" />
-          </geometry>
-        </collision>
-        <collision>
-          <origin xyz="0 0 -0.07" rpy="0 0 0" />
-          <geometry>
-            <sphere radius="${0.06+safety_distance}" />
-          </geometry>
-        </collision>
+        <xacro:collision_capsule xyz="0 0 -0.145" radius="${0.06+safety_distance}" length="0.15" />
       </self_collision_geometries>
     </xacro:link_detailed_coarse>
@@ -128,23 +60,6 @@
     <xacro:link_detailed_coarse name="link4">
       <self_collision_geometries>
-        <collision>
-          <origin xyz="0 0 0" rpy="0 0 0" />
-          <geometry>
-            <cylinder radius="${0.06+safety_distance}" length="0.12" />
-          </geometry>
-        </collision>
-        <collision>
-          <origin xyz="0 0 0.06" rpy="0 0 0" />
-          <geometry>
-            <sphere radius="${0.06+safety_distance}" />
-          </geometry>
-        </collision>
-        <collision>
-          <origin xyz="0 0 -0.06" rpy="0 0 0" />
-          <geometry>
-            <sphere radius="${0.06+safety_distance}" />
-          </geometry>
-        </collision>
-      </self_collision_geometries>
+        <xacro:collision_capsule xyz="0 0 0" radius="${0.06+safety_distance}" length="0.12" />
+     </self_collision_geometries>
     </xacro:link_detailed_coarse>
     <joint name="${arm_id}_joint4" type="revolute">
@@ -159,40 +74,6 @@
     <xacro:link_detailed_coarse name="link5">
       <self_collision_geometries>
-        <collision>
-          <origin xyz="0 0 -0.26" rpy="0 0 0" />
-          <geometry>
-            <cylinder radius="${0.06+safety_distance}" length="0.1" />
-          </geometry>
-        </collision>
-        <collision>
-          <origin xyz="0 0 -0.31" rpy="0 0 0" />
-          <geometry>
-            <sphere radius="${0.06+safety_distance}" />
-          </geometry>
-        </collision>
-        <collision>
-          <origin xyz="0 0 -0.21" rpy="0 0 0" />
-          <geometry>
-            <sphere radius="${0.06+safety_distance}" />
-          </geometry>
-        </collision>
-        <collision>
-          <origin xyz="0 0.08 -0.13" rpy="0 0 0" />
-          <geometry>
-            <cylinder radius="${0.025+safety_distance}" length="0.14" />
-          </geometry>
-        </collision>
-        <collision>
-          <origin xyz="0 0.08 -0.06" rpy="0 0 0" />
-          <geometry>
-            <sphere radius="${0.025+safety_distance}" />
-          </geometry>
-        </collision>
-        <collision>
-          <origin xyz="0 0.08 -0.20" rpy="0 0 0" />
-          <geometry>
-            <sphere radius="${0.025+safety_distance}" />
-          </geometry>
-        </collision>
+        <xacro:collision_capsule xyz="0 0 -0.26"    radius="${0.060+safety_distance}" length="0.10" />
+        <xacro:collision_capsule xyz="0 0.08 -0.13" radius="${0.025+safety_distance}" length="0.14" />
       </self_collision_geometries>
     </xacro:link_detailed_coarse>
@@ -208,22 +89,5 @@
     <xacro:link_detailed_coarse name="link6">
       <self_collision_geometries>
-        <collision>
-          <origin xyz="0 0 -0.03" rpy="0 0 0" />
-          <geometry>
-            <cylinder radius="${0.05+safety_distance}" length="0.08" />
-          </geometry>
-        </collision>
-        <collision>
-          <origin xyz="0 0 0.01" rpy="0 0 0" />
-          <geometry>
-            <sphere radius="${0.05+safety_distance}" />
-          </geometry>
-        </collision>
-        <collision>
-          <origin xyz="0 0 -0.07" rpy="0 0 0" />
-          <geometry>
-            <sphere radius="${0.05+safety_distance}" />
-          </geometry>
-        </collision>
+        <xacro:collision_capsule xyz="0 0 -0.03" radius="${0.05+safety_distance}" length="0.08" />
       </self_collision_geometries>
     </xacro:link_detailed_coarse>
@@ -237,24 +101,7 @@
       <dynamics D="1" K="7000" damping="0.003" friction="0.0" mu_coulomb="0" mu_viscous="16" />
     </joint>
-    <xacro:link_detailed_coarse name="link7">
+    <xacro:link_detailed_coarse name="link7" rpy="0 0 ${pi/4}">
       <self_collision_geometries>
-        <collision>
-          <origin xyz="0 0 0.01" rpy="0 0 0" />
-          <geometry>
-            <cylinder radius="${0.04+safety_distance}" length="0.14" />
-          </geometry>
-        </collision>
-        <collision>
-          <origin xyz="0 0 0.08" rpy="0 0 0" />
-          <geometry>
-            <sphere radius="${0.04+safety_distance}" />
-          </geometry>
-        </collision>
-        <collision>
-          <origin xyz="0 0 -0.06" rpy="0 0 0" />
-          <geometry>
-            <sphere radius="${0.04+safety_distance}" />
-          </geometry>
-        </collision>
+        <xacro:collision_capsule xyz="0 0 0.01" direction="z" radius="${0.04+safety_distance}" length="0.14" />
       </self_collision_geometries>
     </xacro:link_detailed_coarse>

Commit message: CHANGE: Move panda_link8_sc -> panda_link7_sc
The capsule at link8 covers the Pilot which is attached to link7. Though rigidly
connected to link7, link8 is more a "virtual" link without geometry indicating
the flange of the robot. That's why it makes more sense to also have the
collision capsule attached to link7_sc.

File: franka_description/robots/panda_arm.xacro (robot description, xacro)
@@ -104,4 +104,5 @@
       <self_collision_geometries>
         <xacro:collision_capsule xyz="0 0 0.01" direction="z" radius="${0.04+safety_distance}" length="0.14" />
+        <xacro:collision_capsule xyz="0.06 0 0.082" direction="x" radius="${0.03+safety_distance}"  length="0.01" />
       </self_collision_geometries>
     </xacro:link_detailed_coarse>
@@ -116,24 +117,5 @@
     </joint>
     <link name="${arm_id}_link8"/>
-    <link name="${arm_id}_link8_sc">
-      <collision>
-        <origin xyz="0.0424 0.0424 -0.0250" rpy="${pi} ${pi/2} ${pi/2}"/>
-        <geometry>
-          <cylinder radius="${0.03+safety_distance}"  length="0.01" />
-        </geometry>
-      </collision>
-      <collision>
-        <origin xyz="0.0424 0.0424 -0.02" rpy="0 0 0"/>
-        <geometry>
-          <sphere radius="${0.03+safety_distance}"  />
-        </geometry>
-      </collision>
-      <collision>
-        <origin xyz="0.0424 0.0424 -0.03" rpy="0 0 0"/>
-        <geometry>
-          <sphere radius="${0.03+safety_distance}"  />
-        </geometry>
-      </collision>
-    </link>
+    <link name="${arm_id}_link8_sc"/>
     <joint name="${arm_id}_link8_sc_joint" type="fixed">
       <parent link="${arm_id}_link8" />

Commit message: Drop obsolete link8_sc

File: franka_description/robots/panda_arm.xacro (robot description, xacro)
@@ -117,9 +117,4 @@
     </joint>
     <link name="${arm_id}_link8"/>
-    <link name="${arm_id}_link8_sc"/>
-    <joint name="${arm_id}_link8_sc_joint" type="fixed">
-      <parent link="${arm_id}_link8" />
-      <child link="${arm_id}_link8_sc" />
-    </joint>
     <joint name="${arm_id}_joint8" type="fixed">
       <origin rpy="0 0 0" xyz="0 0 0.107"/>
