Commit message: ADD: Proper Friction Parameters for fingers
These parameters make it so that the two fingers are stable and the object in
between does not bounce back and forth between the contact of the left and right
finger. This is accomplished by two parameters mainly:

* `max_vel = 0` inhibits any "snapping" motion, when the object and one finger
go beyond the penetration depth
* `min_depth` defines the allowed penetration depth

NOTE: That these parameter have to be set also on the object to grasp!

File: franka_description/robots/utils.xacro (robot description, xacro)
@@ -21,4 +21,29 @@
       </actuator>
     </transmission>
+  </xacro:macro>
+  <xacro:macro name="gazebo-friction" params="joint mu">
+    <gazebo reference="${joint}">
+      <collision>
+        <max_contacts>10</max_contacts>
+        <surface>
+          <contact>
+            <ode>
+              <!-- These two parameter need application specific tuning. -->
+              <!-- Usually you want no "snap out" velocity and a generous -->
+              <!-- penetration depth to keep the grasping stable -->
+              <max_vel>0</max_vel>
+              <min_depth>0.003</min_depth>
+            </ode>
+          </contact>
+          <friction>
+            <ode>
+              <mu>${mu}</mu>
+              <mu2>${mu}</mu2>
+            </ode>
+          </friction>
+          <bounce/>
+        </surface>
+      </collision>
+    </gazebo>
   </xacro:macro>
   <!-- ========================================================== -->

Commit message: ADD: `rpy` parameter to `<xacro:link_detailed_coarse>`
This way you can specify a rotational offset between panda_link* and panda_link*_sc

File: franka_description/robots/utils.xacro (robot description, xacro)
@@ -28,7 +28,8 @@
   <!--                                                            -->
   <!-- name:  Name of the robot link (without prefix)             -->
+  <!-- rpy:   Rotation of the *_sc link relative to parent [rad]  -->
   <!-- self_collision_geometries:  self <collision> models        -->
   <!-- ========================================================== -->
-  <xacro:macro name="link_detailed_coarse" params="name prefix=${arm_id}_ **self_collision_geometries">
+  <xacro:macro name="link_detailed_coarse" params="name prefix=${arm_id}_ rpy:='0 0 0' **self_collision_geometries">
     <!-- sub-link defining detailed meshes for collision with environment -->
     <link name="${prefix}${name}">
@@ -53,4 +54,5 @@
     <!-- fixed joint between both sub-links -->
     <joint name="${prefix}${name}_sc_joint" type="fixed">
+      <origin rpy="${rpy}" />
       <parent link="${prefix}${name}" />
       <child link="${prefix}${name}_sc" />

Commit message: ADD: `<xacro:collision_capsule>` macro
This macro abstracts the creation of a "collision capsule" from two collision
spheres and a collision cylinder.

Since arbitraty RPY rotations are hard to calculate in XACRO (would require
rotation matrix multiplication and probably reduce redability) for now we only
allow the discrete 6 orientations which are aligned with X/Y/Z axes.

File: franka_description/robots/utils.xacro (robot description, xacro)
@@ -59,4 +59,44 @@
     </joint>
   </xacro:macro>
+  <!-- =========================================================== -->
+  <!-- Add a <collision> tag with a capsule, made from a cylinder  -->
+  <!-- with two spheres at its caps. The capsule will always be    -->
+  <!-- aligned with the axis of 'direction' you pass along.        -->
+  <!--                                                             -->
+  <!-- radius: Radii of both the cylinder and both spheres [m]     -->
+  <!-- length: Length of the cylinder/distance between the centers -->
+  <!--         of the spheres. NOT overall length of capsule!      -->
+  <!-- xyz:    Position of the center of the capsule/cylinder      -->
+  <!-- direction: One of { x, y, z, -x, -y, -z }                   -->
+  <!-- =========================================================== -->
+  <xacro:macro name="collision_capsule" params="radius length xyz:='0 0 0' direction:='z'">
+    <xacro:property name="r" value="${pi/2.0 if 'y' in direction else 0}" />
+    <xacro:property name="p" value="${pi/2.0 if 'x' in direction else 0}" />
+    <xacro:property name="y" value="0" />
+    <xacro:property name="x" value="${xyz.split(' ')[0]}" />
+    <xacro:property name="y" value="${xyz.split(' ')[1]}" />
+    <xacro:property name="z" value="${xyz.split(' ')[2]}" />
+    <xacro:property name="sx" value="${length / 2.0 if 'x' in direction else 0}" />
+    <xacro:property name="sy" value="${length / 2.0 if 'y' in direction else 0}" />
+    <xacro:property name="sz" value="${length / 2.0 if 'z' in direction else 0}" />
+    <collision>
+      <origin xyz="${x} ${y} ${z}" rpy="${r} ${p} ${y}"/>
+      <geometry>
+        <cylinder radius="${radius}" length="${length}" />
+      </geometry>
+    </collision>
+    <collision>
+      <origin xyz="${x+sx} ${y+sy} ${z+sz}" />
+      <geometry>
+        <sphere radius="${radius}" />
+      </geometry>
+    </collision>
+    <collision>
+      <origin xyz="${x-sx} ${y-sy} ${z-sz}" />
+      <geometry>
+        <sphere radius="${radius}" />
+      </geometry>
+    </collision>
+  </xacro:macro>
   <!-- ========================================================== -->
   <!-- Adds the required tags to simulate one joint in gazebo     -->

Commit message: load interial.yaml with relative path

File: franka_description/robots/utils.xacro (robot description, xacro)
@@ -2,5 +2,6 @@
 <robot xmlns:xacro="http://www.ros.org/wiki/xacro">
   <!-- Load interial properties. Property is implicitly passed to macros. -->
-  <xacro:property name="inertial" value="${xacro.load_yaml('inertial.yaml')}" />
+  <xacro:property name="interial_config" value="$(find franka_description)/robots/inertial.yaml"/>
+  <xacro:property name="inertial" value="${xacro.load_yaml(interial_config)}"/>
   <!-- ============================================================== -->
   <!-- Macro to add an <interial> tag based on yaml-load properties   -->

Commit message: FIX: Typo

File: franka_description/robots/utils.xacro (robot description, xacro)
@@ -2,6 +2,6 @@
 <robot xmlns:xacro="http://www.ros.org/wiki/xacro">
   <!-- Load interial properties. Property is implicitly passed to macros. -->
-  <xacro:property name="interial_config" value="$(find franka_description)/robots/inertial.yaml"/>
-  <xacro:property name="inertial" value="${xacro.load_yaml(interial_config)}"/>
+  <xacro:property name="inertial_config" value="$(find franka_description)/robots/inertial.yaml"/>
+  <xacro:property name="inertial" value="${xacro.load_yaml(inertial_config)}"/>
   <!-- ============================================================== -->
   <!-- Macro to add an <interial> tag based on yaml-load properties   -->
