Commit message: Adds the safety distance to the values.

File: franka_description/robots/hand.xacro (robot description, xacro)
@@ -1,5 +1,5 @@
 <?xml version="1.0" encoding="utf-8"?>
 <robot xmlns:xacro="http://www.ros.org/wiki/xacro" name="hand">
-  <xacro:macro name="hand" params="connected_to:='' ns:='' rpy:='0 0 0' xyz:='0 0 0' ">
+  <xacro:macro name="hand" params="connected_to:='' ns:='' rpy:='0 0 0' xyz:='0 0 0' safety_distance:='0'">
     <xacro:unless value="${connected_to == ''}">
       <joint name="${ns}_hand_joint" type="fixed">
@@ -18,5 +18,5 @@
         <origin xyz="0 0 0.04" rpy="0 ${pi/2} ${pi/2}"/>
         <geometry>
-          <cylinder radius="0.04" length="0.1" />
+          <cylinder radius="${0.04+safety_distance}" length="0.1" />
         </geometry>
       </collision>
@@ -24,5 +24,5 @@
         <origin xyz="0 -0.05 0.04" rpy="0 0 0"/>
         <geometry>
-          <sphere radius="0.04" />
+          <sphere radius="${0.04+safety_distance}"  />
         </geometry>
       </collision>
@@ -30,5 +30,5 @@
         <origin xyz="0 0.05 0.04" rpy="0 0 0"/>
         <geometry>
-          <sphere radius="0.04" />
+          <sphere radius="${0.04+safety_distance}"  />
         </geometry>
       </collision>
@@ -36,5 +36,5 @@
         <origin xyz="0 0 0.1" rpy="0 ${pi/2} ${pi/2}"/>
         <geometry>
-          <cylinder radius="0.02" length="0.1" />
+          <cylinder radius="${0.02+safety_distance}" length="0.1" />
         </geometry>
       </collision>
@@ -42,5 +42,5 @@
         <origin xyz="0 -0.05 0.1" rpy="0 0 0"/>
         <geometry>
-          <sphere radius="0.02" />
+          <sphere radius="${0.02+safety_distance}"  />
         </geometry>
       </collision>
@@ -48,5 +48,5 @@
         <origin xyz="0 0.05 0.1" rpy="0 0 0"/>
         <geometry>
-          <sphere radius="0.02" />
+          <sphere radius="${0.02+safety_distance}"  />
         </geometry>
       </collision>

File: franka_description/robots/panda_arm.xacro (robot description, xacro)
@@ -1,5 +1,5 @@
 <?xml version='1.0' encoding='utf-8'?>
 <robot xmlns:xacro="http://www.ros.org/wiki/xacro" name="panda">
-  <xacro:macro name="panda_arm" params="arm_id:='panda' description_pkg:='franka_description' connected_to:='' xyz:='0 0 0' rpy:='0 0 0'">
+  <xacro:macro name="panda_arm" params="arm_id:='panda' description_pkg:='franka_description' connected_to:='' xyz:='0 0 0' rpy:='0 0 0' safety_distance:=''">
     <xacro:unless value="${not connected_to}">
       <joint name="${arm_id}_joint_${connected_to}" type="fixed">
@@ -18,5 +18,5 @@
         <origin xyz="-0.075 0 0.06" rpy="0 ${pi/2} 0"/>
         <geometry>
-          <cylinder radius="0.06" length="0.03" />
+          <cylinder radius="${0.06+safety_distance}" length="0.03" />
         </geometry>
       </collision>
@@ -24,5 +24,5 @@
         <origin xyz="-0.06 0 0.06" rpy="0 0 0"/>
         <geometry>
-          <sphere radius="0.06" />
+          <sphere radius="${0.06+safety_distance}" />
         </geometry>
       </collision>
@@ -30,5 +30,5 @@
         <origin xyz="-0.09 0 0.06" rpy="0 0 0"/>
         <geometry>
-          <sphere radius="0.06" />
+          <sphere radius="${0.06+safety_distance}" />
         </geometry>
       </collision>
@@ -43,5 +43,5 @@
         <origin xyz="0 0 -0.1915" rpy="0 0 0"/>
         <geometry>
-          <cylinder radius="0.06" length="0.2830" />
+          <cylinder radius="${0.06+safety_distance}" length="0.2830" />
         </geometry>
       </collision>
@@ -49,5 +49,5 @@
         <origin xyz="0 0 -0.333" rpy="0 0 0"/>
         <geometry>
-          <sphere radius="0.06" />
+          <sphere radius="${0.06+safety_distance}" />
         </geometry>
       </collision>
@@ -55,5 +55,5 @@
         <origin xyz="0 0 -0.05" rpy="0 0 0"/>
         <geometry>
-          <sphere radius="0.06" />
+          <sphere radius="${0.06+safety_distance}" />
         </geometry>
       </collision>
@@ -76,5 +76,5 @@
         <origin xyz="0 0 0" rpy="0 0 0"/>
         <geometry>
-          <cylinder radius="0.06" length="0.12" />
+          <cylinder radius="${0.06+safety_distance}" length="0.12" />
         </geometry>
       </collision>
@@ -82,5 +82,5 @@
         <origin xyz="0 0 -0.06" rpy="0 0 0"/>
         <geometry>
-          <sphere radius="0.06" />
+          <sphere radius="${0.06+safety_distance}" />
         </geometry>
       </collision>
@@ -88,5 +88,5 @@
         <origin xyz="0 0 0.06" rpy="0 0 0"/>
         <geometry>
-          <sphere radius="0.06" />
+          <sphere radius="${0.06+safety_distance}" />
         </geometry>
       </collision>
@@ -109,5 +109,5 @@
         <origin xyz="0 0 -0.145" rpy="0 0 0"/>
         <geometry>
-          <cylinder radius="0.06" length="0.15" />
+          <cylinder radius="${0.06+safety_distance}" length="0.15" />
         </geometry>
       </collision>
@@ -115,5 +115,5 @@
         <origin xyz="0 0 -0.22" rpy="0 0 0"/>
         <geometry>
-          <sphere radius="0.06" />
+          <sphere radius="${0.06+safety_distance}" />
         </geometry>
       </collision>
@@ -121,5 +121,5 @@
         <origin xyz="0 0 -0.07" rpy="0 0 0"/>
         <geometry>
-          <sphere radius="0.06" />
+          <sphere radius="${0.06+safety_distance}" />
         </geometry>
       </collision>
@@ -142,5 +142,5 @@
         <origin xyz="0 0 0" rpy="0 0 0"/>
         <geometry>
-          <cylinder radius="0.06" length="0.12" />
+          <cylinder radius="${0.06+safety_distance}" length="0.12" />
         </geometry>
       </collision>
@@ -148,5 +148,5 @@
         <origin xyz="0 0 0.06" rpy="0 0 0"/>
         <geometry>
-          <sphere radius="0.06" />
+          <sphere radius="${0.06+safety_distance}" />
         </geometry>
       </collision>
@@ -154,5 +154,5 @@
         <origin xyz="0 0 -0.06" rpy="0 0 0"/>
         <geometry>
-          <sphere radius="0.06" />
+          <sphere radius="${0.06+safety_distance}" />
         </geometry>
       </collision>
@@ -175,5 +175,5 @@
         <origin xyz="0 0 -0.26" rpy="0 0 0"/>
         <geometry>
-          <cylinder radius="0.06" length="0.1" />
+          <cylinder radius="${0.06+safety_distance}" length="0.1" />
         </geometry>
       </collision>
@@ -181,5 +181,5 @@
         <origin xyz="0 0 -0.31" rpy="0 0 0"/>
         <geometry>
-          <sphere radius="0.06" />
+          <sphere radius="${0.06+safety_distance}" />
         </geometry>
       </collision>
@@ -187,5 +187,5 @@
         <origin xyz="0 0 -0.21" rpy="0 0 0"/>
         <geometry>
-          <sphere radius="0.06" />
+          <sphere radius="${0.06+safety_distance}" />
         </geometry>
       </collision>
@@ -193,5 +193,5 @@
         <origin xyz="0 0.08 -0.13" rpy="0 0 0"/>
         <geometry>
-          <cylinder radius="0.025" length="0.14" />
+          <cylinder radius="${0.025+safety_distance}" length="0.14" />
         </geometry>
       </collision>
@@ -199,5 +199,5 @@
         <origin xyz="0 0.08 -0.06" rpy="0 0 0"/>
         <geometry>
-          <sphere radius="0.025" />
+          <sphere radius="${0.025+safety_distance}" />
         </geometry>
       </collision>
@@ -205,5 +205,5 @@
         <origin xyz="0 0.08 -0.20" rpy="0 0 0"/>
         <geometry>
-          <sphere radius="0.025" />
+          <sphere radius="${0.025+safety_distance}" />
         </geometry>
       </collision>
@@ -226,5 +226,5 @@
         <origin xyz="0 0 -0.03" rpy="0 0 0"/>
         <geometry>
-          <cylinder radius="0.05" length="0.08" />
+          <cylinder radius="${0.05+safety_distance}" length="0.08" />
         </geometry>
       </collision>
@@ -232,5 +232,5 @@
         <origin xyz="0 0 0.01" rpy="0 0 0"/>
         <geometry>
-          <sphere radius="0.05" />
+          <sphere radius="${0.05+safety_distance}" />
         </geometry>
       </collision>
@@ -238,5 +238,5 @@
         <origin xyz="0 0 -0.07" rpy="0 0 0"/>
         <geometry>
-          <sphere radius="0.05" />
+          <sphere radius="${0.05+safety_distance}" />
         </geometry>
       </collision>
@@ -259,5 +259,5 @@
         <origin xyz="0 0 0.01" rpy="0 0 0"/>
         <geometry>
-          <cylinder radius="0.04" length="0.14" />
+          <cylinder radius="${0.04+safety_distance}" length="0.14" />
         </geometry>
       </collision>
@@ -265,5 +265,5 @@
         <origin xyz="0 0 0.08" rpy="0 0 0"/>
         <geometry>
-          <sphere radius="0.04" />
+          <sphere radius="${0.04+safety_distance}"  />
         </geometry>
       </collision>
@@ -271,5 +271,5 @@
         <origin xyz="0 0 -0.06" rpy="0 0 0"/>
         <geometry>
-          <sphere radius="0.04" />
+          <sphere radius="${0.04+safety_distance}"  />
         </geometry>
       </collision>
@@ -287,5 +287,5 @@
         <origin xyz="0.0424 0.0424 -0.0250" rpy="${pi} ${pi/2} ${pi/2}"/>
         <geometry>
-          <cylinder radius="0.03" length="0.01" />
+          <cylinder radius="${0.03+safety_distance}"  length="0.01" />
         </geometry>
       </collision>
@@ -293,5 +293,5 @@
         <origin xyz="0.0424 0.0424 -0.02" rpy="0 0 0"/>
         <geometry>
-          <sphere radius="0.03" />
+          <sphere radius="${0.03+safety_distance}"  />
         </geometry>
       </collision>
@@ -299,5 +299,5 @@
         <origin xyz="0.0424 0.0424 -0.03" rpy="0 0 0"/>
         <geometry>
-          <sphere radius="0.03" />
+          <sphere radius="${0.03+safety_distance}"  />
         </geometry>
       </collision>

Commit message: remove quotation marks from default value

File: franka_description/robots/hand.xacro (robot description, xacro)
@@ -2,5 +2,5 @@
 <robot xmlns:xacro="http://www.ros.org/wiki/xacro" name="hand">
   <!-- safety_distance: Minimum safety distance in [m] by which the collision volumes are expanded and which is enforced during robot motions -->
-  <xacro:macro name="hand" params="connected_to:='' ns:='' rpy:='0 0 0' xyz:='0 0 0' safety_distance:='0'">
+  <xacro:macro name="hand" params="connected_to:='' ns:='' rpy:='0 0 0' xyz:='0 0 0' safety_distance:=0">
     <xacro:unless value="${connected_to == ''}">
       <joint name="${ns}_hand_joint" type="fixed">

File: franka_description/robots/panda_arm.xacro (robot description, xacro)
@@ -3,5 +3,5 @@
   <!-- safety_distance: Minimum safety distance in [m] by which the collision volumes are expanded and which is enforced during robot motions -->
   <!-- arm_id: Namespace of the panda arm. Serves to differentiate between arms in case of multiple instances. -->
-  <xacro:macro name="panda_arm" params="arm_id:='panda' description_pkg:='franka_description' connected_to:='' xyz:='0 0 0' rpy:='0 0 0' safety_distance:='0'">
+  <xacro:macro name="panda_arm" params="arm_id:='panda' description_pkg:='franka_description' connected_to:='' xyz:='0 0 0' rpy:='0 0 0' safety_distance:=0">
     <xacro:unless value="${not connected_to}">
       <joint name="${arm_id}_joint_${connected_to}" type="fixed">

Commit message: Panda in Gazebo + MoveIt! motion planning

File: franka_description/robots/hand.xacro (robot description, xacro)
@@ -20,4 +20,11 @@
         </geometry>
       </collision>
+      <!-- for simulation -->
+      <inertial>
+        <origin xyz="0 0 0" rpy="0 0 0" />
+        <mass value="0.68" />
+        <inertia ixx="0.1" ixy="0.0" ixz="0.0" iyy="0.1" iyz="0.0" izz="0.1" />
+      </inertial>
+      <!-- end for simulation -->
     </link>
     <link name="${ns}_leftfinger">
@@ -32,4 +39,11 @@
         </geometry>
       </collision>
+      <!-- for simulation -->
+      <inertial>
+        <origin xyz="0 0 0" rpy="0 0 0" />
+        <mass value="0.01" />
+        <inertia ixx="0.1" ixy="0.0" ixz="0.0" iyy="0.1" iyz="0.0" izz="0.1" />
+      </inertial>
+      <!-- end for simulation -->
     </link>
     <link name="${ns}_rightfinger">
@@ -46,4 +60,11 @@
         </geometry>
       </collision>
+      <!-- for simulation -->
+      <inertial>
+        <origin xyz="0 0 0" rpy="0 0 0" />
+        <mass value="0.01" />
+        <inertia ixx="0.1" ixy="0.0" ixz="0.0" iyy="0.1" iyz="0.0" izz="0.1" />
+      </inertial>
+      <!-- end for simulation -->
     </link>
     <joint name="${ns}_finger_joint1" type="prismatic">

File: franka_description/robots/panda_arm.xacro (robot description, xacro)
@@ -9,4 +9,13 @@
       </joint>
     </xacro:unless>
+    <!-- for simulation -->
+    <link name="world" />
+    <joint name="robot_to_world" type="fixed">
+      <parent link="world" />
+      <child link="${arm_id}_link0" />
+      <origin xyz="0.0 0.0 0.0" rpy="0.0 0.0 0.0" />
+    </joint>
+    <xacro:property name="joint_damping" value="1.0"/>
+    <!-- end for simulation -->
     <link name="${arm_id}_link0">
       <visual>
@@ -20,4 +29,11 @@
         </geometry>
       </collision>
+      <!-- for simulation -->
+      <inertial>
+        <origin xyz="0 0 0" rpy="0 0 0" />
+        <mass value="3.06" />
+        <inertia ixx="0.3" ixy="0.0" ixz="0.0" iyy="0.3" iyz="0.0" izz="0.3" />
+      </inertial>
+      <!-- end for simulation -->
     </link>
     <link name="${arm_id}_link1">
@@ -32,4 +48,11 @@
         </geometry>
       </collision>
+      <!-- for simulation -->
+      <inertial>
+        <origin xyz="0 0 0" rpy="0 0 0" />
+        <mass value="2.34" />
+        <inertia ixx="0.3" ixy="0.0" ixz="0.0" iyy="0.3" iyz="0.0" izz="0.3" />
+      </inertial>
+      <!-- end for simulation -->
     </link>
     <joint name="${arm_id}_joint1" type="revolute">
@@ -40,4 +63,7 @@
       <axis xyz="0 0 1"/>
       <limit effort="87" lower="-2.8973" upper="2.8973" velocity="2.1750"/>
+      <!-- for simulation -->
+      <dynamics damping="${joint_damping}"/>
+      <!-- end for simulation -->
     </joint>
     <link name="${arm_id}_link2">
@@ -52,4 +78,11 @@
         </geometry>
       </collision>
+      <!-- for simulation -->
+      <inertial>
+        <origin xyz="0 0 0" rpy="0 0 0" />
+        <mass value="2.36" />
+        <inertia ixx="0.3" ixy="0.0" ixz="0.0" iyy="0.3" iyz="0.0" izz="0.3" />
+      </inertial>
+      <!-- end for simulation -->
     </link>
     <joint name="${arm_id}_joint2" type="revolute">
@@ -60,4 +93,7 @@
       <axis xyz="0 0 1"/>
       <limit effort="87" lower="-1.7628" upper="1.7628" velocity="2.1750"/>
+      <!-- for simulation -->
+      <dynamics damping="${joint_damping}"/>
+      <!-- end for simulation -->
     </joint>
     <link name="${arm_id}_link3">
@@ -72,4 +108,11 @@
         </geometry>
       </collision>
+      <!-- for simulation -->
+      <inertial>
+        <origin xyz="0 0 0" rpy="0 0 0" />
+        <mass value="2.38" />
+        <inertia ixx="0.3" ixy="0.0" ixz="0.0" iyy="0.3" iyz="0.0" izz="0.3" />
+      </inertial>
+      <!-- end for simulation -->
     </link>
     <joint name="${arm_id}_joint3" type="revolute">
@@ -80,4 +123,7 @@
       <axis xyz="0 0 1"/>
       <limit effort="87" lower="-2.8973" upper="2.8973" velocity="2.1750"/>
+      <!-- for simulation -->
+      <dynamics damping="${joint_damping}"/>
+      <!-- end for simulation -->
     </joint>
     <link name="${arm_id}_link4">
@@ -92,4 +138,11 @@
         </geometry>
       </collision>
+      <!-- for simulation -->
+      <inertial>
+        <origin xyz="0 0 0" rpy="0 0 0" />
+        <mass value="2.43" />
+        <inertia ixx="0.3" ixy="0.0" ixz="0.0" iyy="0.3" iyz="0.0" izz="0.3" />
+      </inertial>
+      <!-- end for simulation -->
     </link>
     <joint name="${arm_id}_joint4" type="revolute">
@@ -100,4 +153,7 @@
       <axis xyz="0 0 1"/>
       <limit effort="87" lower="-3.0718" upper="-0.0698" velocity="2.1750"/>
+      <!-- for simulation -->
+      <dynamics damping="${joint_damping}"/>
+      <!-- end for simulation -->
     </joint>
     <link name="${arm_id}_link5">
@@ -112,4 +168,11 @@
         </geometry>
       </collision>
+      <!-- for simulation -->
+      <inertial>
+        <origin xyz="0 0 0" rpy="0 0 0" />
+        <mass value="3.5" />
+        <inertia ixx="0.3" ixy="0.0" ixz="0.0" iyy="0.3" iyz="0.0" izz="0.3" />
+      </inertial>
+      <!-- end for simulation -->
     </link>
     <joint name="${arm_id}_joint5" type="revolute">
@@ -120,4 +183,7 @@
       <axis xyz="0 0 1"/>
       <limit effort="12" lower="-2.8973" upper="2.8973" velocity="2.6100"/>
+      <!-- for simulation -->
+      <dynamics damping="${joint_damping}"/>
+      <!-- end for simulation -->
     </joint>
     <link name="${arm_id}_link6">
@@ -132,4 +198,11 @@
         </geometry>
       </collision>
+      <!-- for simulation -->
+      <inertial>
+        <origin xyz="0 0 0" rpy="0 0 0" />
+        <mass value="1.47" />
+        <inertia ixx="0.3" ixy="0.0" ixz="0.0" iyy="0.3" iyz="0.0" izz="0.3" />
+      </inertial>
+      <!-- end for simulation -->
     </link>
     <joint name="${arm_id}_joint6" type="revolute">
@@ -140,4 +213,7 @@
       <axis xyz="0 0 1"/>
       <limit effort="12" lower="-0.0175" upper="3.7525" velocity="2.6100"/>
+      <!-- for simulation -->
+      <dynamics damping="${joint_damping}"/>
+      <!-- end for simulation -->
     </joint>
     <link name="${arm_id}_link7">
@@ -152,4 +228,11 @@
         </geometry>
       </collision>
+      <!-- for simulation -->
+      <inertial>
+        <origin xyz="0 0 0" rpy="0 0 0" />
+        <mass value="0.45" />
+        <inertia ixx="0.3" ixy="0.0" ixz="0.0" iyy="0.3" iyz="0.0" izz="0.3" />
+      </inertial>
+      <!-- end for simulation -->
     </link>
     <joint name="${arm_id}_joint7" type="revolute">
@@ -160,6 +243,17 @@
       <axis xyz="0 0 1"/>
       <limit effort="12" lower="-2.8973" upper="2.8973" velocity="2.6100"/>
-    </joint>
-    <link name="${arm_id}_link8"/>
+      <!-- for simulation -->
+      <dynamics damping="${joint_damping}"/>
+      <!-- end for simulation -->
+    </joint>
+    <link name="${arm_id}_link8">
+      <!-- for simulation -->
+      <inertial>
+        <origin xyz="0 0 0" rpy="0 0 0" />
+        <mass value="0.0" />
+        <inertia ixx="0.3" ixy="0.0" ixz="0.0" iyy="0.3" iyz="0.0" izz="0.3" />
+      </inertial>
+      <!-- end for simulation -->
+    </link>
     <joint name="${arm_id}_joint8" type="fixed">
       <origin rpy="0 0 0" xyz="0 0 0.107"/>

File: franka_description/robots/panda_arm_hand.urdf.xacro (robot description, xacro)
@@ -3,5 +3,14 @@
   <xacro:include filename="$(find franka_description)/robots/panda_arm.xacro"/>
   <xacro:include filename="$(find franka_description)/robots/hand.xacro"/>
+  <!-- for simulation -->
+  <xacro:include filename="$(find franka_description)/robots/panda.gazebo.xacro"/>
+  <xacro:include filename="$(find franka_description)/robots/panda.transmission.xacro"/>
+  <!-- end for simulation -->
   <xacro:panda_arm />
   <xacro:hand ns="panda" rpy="0 0 ${-pi/4}" connected_to="panda_link8"/>
+  <!-- for simulation -->
+  <xacro:arg name="robot_name" default="panda"/>
+  <xacro:panda_gazebo robot_name="$(arg robot_name)" />
+  <xacro:panda_transmission robot_name="$(arg robot_name)" />
+  <!-- end for simulation -->
 </robot>
