Commit message: Added inertia values to URDFs of arm and hand. Changed constant in visual mesh files, because they're not displayed in gazebo otherwise. See http://answers.gazebosim.org/question/20068/collada-model-is-not-visible-in-gazebo-89-if-transparent-a_one/

File: franka_description/robots/hand.xacro (robot description, xacro)
@@ -9,9 +9,20 @@
       </joint>
     </xacro:unless>
+    <xacro:arg name="gazebo" default="true"/>
+    <xacro:if value="$(arg gazebo)">
+      <!-- Gazebo Tags -->
+      <xacro:include filename="$(find mopa_description)/robots/hand.gazebo.xacro"/>
+    </xacro:if>
     <link name="${ns}_hand">
+      <inertial>
+        <mass value="0.73" />
+        <origin xyz="0 0.0015244 0.0275912" rpy="0 0 0" />
+        <inertia ixx="0.00278560230025" ixy="0.0" ixz="0.0" iyy="0.000400033405336" iyz="0.0" izz="0.00256378041832" />
+      </inertial>
       <visual>
         <geometry>
           <mesh filename="package://franka_description/meshes/visual/hand.dae"/>
         </geometry>
+        <!-- <origin xyz="0 0 0" rpy="0 0 0" /> -->
       </visual>
       <collision>
@@ -22,4 +33,9 @@
     </link>
     <link name="${ns}_leftfinger">
+      <inertial>
+        <mass value="0.1" />
+        <origin xyz="0 0.0145644 0.0227941" rpy="0 0 0" />
+        <inertia ixx="3.01220925051e-05" ixy="0.0" ixz="0.0" iyy="2.95873808038e-05" iyz="0.0" izz="6.95125211657e-06" />
+      </inertial>
       <visual>
         <geometry>
@@ -34,4 +50,9 @@
     </link>
     <link name="${ns}_rightfinger">
+      <inertial>
+        <mass value="0.1" />
+        <origin xyz="0 0.0145644 0.0227941" rpy="0 0 ${pi}" />
+        <inertia ixx="3.01220925051e-05" ixy="0.0" ixz="0.0" iyy="2.95873808038e-05" iyz="0.0" izz="6.95125211657e-06" />
+      </inertial>
       <visual>
         <origin xyz="0 0 0" rpy="0 0 ${pi}"/>

File: franka_description/robots/panda_arm.xacro (robot description, xacro)
@@ -2,5 +2,5 @@
 <robot xmlns:xacro="http://www.ros.org/wiki/xacro" name="panda">
   <xacro:macro name="panda_arm" params="arm_id:='panda' description_pkg:='franka_description' connected_to:='' xyz:='0 0 0' rpy:='0 0 0'">
-    <xacro:unless value="${not connected_to}">
+    <xacro:unless value="${connected_to == ''}">
       <joint name="${arm_id}_joint_${connected_to}" type="fixed">
         <parent link="${connected_to}"/>
@@ -9,5 +9,15 @@
       </joint>
     </xacro:unless>
+    <xacro:arg name="gazebo" default="true"/>
+    <xacro:if value="$(arg gazebo)">
+      <!-- Gazebo Tags -->
+      <xacro:include filename="$(find mopa_description)/robots/panda_arm.gazebo.xacro"/>
+    </xacro:if>
     <link name="${arm_id}_link0">
+      <inertial>
+        <mass value="2.92" />
+        <origin xyz="-0.025566 -2.88e-05 0.057332" rpy="0 0 0" />
+        <inertia ixx="0.00782229414331" ixy="-1.56191622996e-05" ixz="-0.00126005738123" iyy="0.0109027971813" iyz="1.08233858202e-05" izz="0.0102355503949" />
+      </inertial>
       <visual>
         <geometry>
@@ -22,4 +32,9 @@
     </link>
     <link name="${arm_id}_link1">
+      <inertial>
+        <mass value="2.74" />
+        <origin xyz="0 -0.0324958 -0.0675818" rpy="0 0 0" />
+        <inertia ixx="0.0180416958283" ixy="0.0" ixz="0.0" iyy="0.0159136071891" iyz="0.0046758424612" izz="0.00620690827127" />
+      </inertial>
       <visual>
         <geometry>
@@ -42,4 +57,9 @@
     </joint>
     <link name="${arm_id}_link2">
+      <inertial>
+        <mass value="2.74" />
+        <origin xyz="0 -0.06861 0.0322285" rpy="0 0 0" />
+        <inertia ixx="0.0182856182281" ixy="0.0" ixz="0.0" iyy="0.00621358421175" iyz="-0.00472844221905" izz="0.0161514346309" />
+      </inertial>
       <visual>
         <geometry>
@@ -62,4 +82,9 @@
     </joint>
     <link name="${arm_id}_link3">
+      <inertial>
+        <mass value="2.38" />
+        <origin xyz="0.0469893 0.0316374 -0.031704" rpy="0 0 0" />
+        <inertia ixx="0.00771376630908" ixy="-0.00248490625138" ixz="-0.00332147581033" iyy="0.00989108008727" iyz="-0.00217796151484" izz="0.00811723558464" />
+      </inertial>
       <visual>
         <geometry>
@@ -82,4 +107,9 @@
     </joint>
     <link name="${arm_id}_link4">
+      <inertial>
+        <mass value="2.38" />
+        <origin xyz="-0.0360446 0.0336853 0.031882" rpy="0 0 0" />
+        <inertia ixx="0.00799663881132" ixy="0.00347095570217" ixz="-0.00241222942995" iyy="0.00825390705278" iyz="0.00235774044121" izz="0.0102515004345" />
+      </inertial>
       <visual>
         <geometry>
@@ -102,4 +132,9 @@
     </joint>
     <link name="${arm_id}_link5">
+      <inertial>
+        <mass value="2.74" />
+        <origin xyz="0 0.0610427 -0.104176" rpy="0 0 0" />
+        <inertia ixx="0.030371374513" ixy="6.50283587108e-07" ixz="-1.05129179916e-05" iyy="0.0288752887402" iyz="-0.00775653445787" izz="0.00444134056164" />
+      </inertial>
       <visual>
         <geometry>
@@ -122,4 +157,9 @@
     </joint>
     <link name="${arm_id}_link6">
+      <inertial>
+        <mass value="1.55" />
+        <origin xyz="0.0510509 0.009108 0.0106343" rpy="0 0 0" />
+        <inertia ixx="0.00303336450376" ixy="-0.000437276865508" ixz="0.000629257294877" iyy="0.00404479911567" iyz="0.000130472021025" izz="0.00558234286039" />
+      </inertial>
       <visual>
         <geometry>
@@ -142,4 +182,9 @@
     </joint>
     <link name="${arm_id}_link7">
+      <inertial>
+        <mass value="0.54" />
+        <origin xyz="0.0109695 0.0107965 0.0650411" rpy="0 0 0" />
+        <inertia ixx="0.000888868887021" ixy="-0.00012239074652" ixz="3.98699829666e-05" iyy="0.000888001373233" iyz="-9.33825115206e-05" izz="0.0007176834609" />
+      </inertial>
       <visual>
         <geometry>
