Commit message: Improves hand/finger collision geometries
This commit replaces the finger collision geometries found in the hand
joint with more accurate finger geometries placed in the finger joints.
Further it gives users the ability to set the safety_distance.

File: franka_description/robots/hand.xacro (robot description, xacro)
@@ -17,11 +17,5 @@
       </visual>
       <collision>
-        <origin xyz="0 0 0.04" rpy="0 ${pi/2} ${pi/2}"/>
-        <geometry>
-          <cylinder radius="${0.04+safety_distance}" length="0.1" />
-        </geometry>
-      </collision>
-      <collision>
-        <origin xyz="0 -0.05 0.04" rpy="0 0 0"/>
+        <origin xyz="0 0.065 0.027" rpy="0 0 0"/>
         <geometry>
           <sphere radius="${0.04+safety_distance}"  />
@@ -29,25 +23,13 @@
       </collision>
       <collision>
-        <origin xyz="0 0.05 0.04" rpy="0 0 0"/>
+        <origin xyz="0 0 0.027" rpy="0 ${pi/2} ${pi/2}"/>
         <geometry>
-          <sphere radius="${0.04+safety_distance}"  />
+          <cylinder radius="${0.04+safety_distance}" length="0.135" />
         </geometry>
       </collision>
       <collision>
-        <origin xyz="0 0 0.1" rpy="0 ${pi/2} ${pi/2}"/>
+        <origin xyz="0 -0.065 0.027" rpy="0 0 0"/>
         <geometry>
-          <cylinder radius="${0.02+safety_distance}" length="0.1" />
-        </geometry>
-      </collision>
-      <collision>
-        <origin xyz="0 -0.05 0.1" rpy="0 0 0"/>
-        <geometry>
-          <sphere radius="${0.02+safety_distance}"  />
-        </geometry>
-      </collision>
-      <collision>
-        <origin xyz="0 0.05 0.1" rpy="0 0 0"/>
-        <geometry>
-          <sphere radius="${0.02+safety_distance}"  />
+          <sphere radius="${0.04+safety_distance}"  />
         </geometry>
       </collision>
@@ -59,4 +41,22 @@
         </geometry>
       </visual>
+      <collision>
+        <origin xyz="0 0.0184 0.0101" rpy="0 0 0"/>
+        <geometry>
+          <box size="${0.022+safety_distance} ${0.014+safety_distance} ${0.0177+safety_distance}" />
+        </geometry>
+      </collision>
+      <collision>
+        <origin xyz="0 0.01655 0.02755" rpy="${3.257/(2*pi)} 0 0"/>
+        <geometry>
+          <box size="${0.022+safety_distance} ${0.00686+safety_distance} 0.0237" />
+        </geometry>
+      </collision>
+      <collision>
+        <origin xyz="0 0.0073 0.045" rpy="0 0 0"/>
+        <geometry>
+          <box size="${0.022+safety_distance} ${0.0147+safety_distance} ${0.0178+safety_distance}" />
+        </geometry>
+      </collision>
     </link>
     <link name="${ns}_rightfinger">
@@ -67,5 +67,23 @@
         </geometry>
       </visual>
-   </link>
+      <collision>
+        <origin xyz="0 -0.0184 0.0101" rpy="0 0 0"/>
+        <geometry>
+          <box size="${0.022+safety_distance} ${0.014+safety_distance} ${0.0177+safety_distance}" />
+        </geometry>
+      </collision>
+      <collision>
+        <origin xyz="0 -0.01655 0.02755" rpy="${-3.257/(2*pi)} 0 0"/>
+        <geometry>
+          <box size="${0.022+safety_distance} ${0.00686+safety_distance} 0.0237" />
+        </geometry>
+      </collision>
+      <collision>
+        <origin xyz="0 -0.0073 0.045" rpy="0 0 0"/>
+        <geometry>
+          <box size="${0.022+safety_distance} ${0.0147+safety_distance} ${0.0178+safety_distance}" />
+        </geometry>
+      </collision>
+    </link>
     <joint name="${ns}_finger_joint1" type="prismatic">
       <parent link="${ns}_hand"/>

Commit message: Moves finger collision geometries to the finger joints
This commit moves the finger collision geometries to the finger joints.
This was done to prevent errors in third party libaries. Moveit for
example expects a collision geometry in each joint that can be
controlled.

File: franka_description/robots/hand.xacro (robot description, xacro)
@@ -34,22 +34,4 @@
         </geometry>
       </collision>
-      <collision>
-        <origin xyz="0 0 0.1" rpy="0 ${pi/2} ${pi/2}"/>
-        <geometry>
-          <cylinder radius="${0.02+safety_distance}" length="0.1" />
-        </geometry>
-      </collision>
-      <collision>
-        <origin xyz="0 -0.05 0.1" rpy="0 0 0"/>
-        <geometry>
-          <sphere radius="${0.02+safety_distance}"  />
-        </geometry>
-      </collision>
-      <collision>
-        <origin xyz="0 0.05 0.1" rpy="0 0 0"/>
-        <geometry>
-          <sphere radius="${0.02+safety_distance}"  />
-        </geometry>
-      </collision>
     </link>
     <link name="${ns}_leftfinger">
@@ -59,4 +41,16 @@
         </geometry>
       </visual>
+      <collision>
+        <origin xyz="0 0.01 0.0415" rpy="0 0 0"/>
+        <geometry>
+          <sphere radius="${0.02+safety_distance}"  />
+        </geometry>
+      </collision>
+      <collision>
+        <origin xyz="0 -0.015 0.0416" rpy="0 ${pi/2} ${pi/2}"/>
+        <geometry>
+          <cylinder radius="${0.02+safety_distance}" length="0.05" />
+        </geometry>
+      </collision>
     </link>
     <link name="${ns}_rightfinger">
@@ -67,4 +61,16 @@
         </geometry>
       </visual>
+      <collision>
+        <origin xyz="0 -0.01 0.0415" rpy="0 0 0"/>
+        <geometry>
+          <sphere radius="${0.02+safety_distance}"  />
+        </geometry>
+      </collision>
+      <collision>
+        <origin xyz="0 0.015 0.0416" rpy="0 ${pi/2} ${pi/2}"/>
+        <geometry>
+          <cylinder radius="${0.02+safety_distance}" length="0.05" />
+        </geometry>
+      </collision>
    </link>
     <joint name="${ns}_finger_joint1" type="prismatic">

Commit message: Moves finger collision geometries to the finger joints
This commit moves the finger collision geometries to the finger joints.
This was done to prevent errors in third party libaries. Moveit for
example expects a collision geometry in each joint that can be
controlled.

File: franka_description/robots/hand.xacro (robot description, xacro)
@@ -34,22 +34,4 @@
         </geometry>
       </collision>
-      <collision>
-        <origin xyz="0 0 0.1" rpy="0 ${pi/2} ${pi/2}"/>
-        <geometry>
-          <cylinder radius="${0.02+safety_distance}" length="0.1" />
-        </geometry>
-      </collision>
-      <collision>
-        <origin xyz="0 -0.05 0.1" rpy="0 0 0"/>
-        <geometry>
-          <sphere radius="${0.02+safety_distance}"  />
-        </geometry>
-      </collision>
-      <collision>
-        <origin xyz="0 0.05 0.1" rpy="0 0 0"/>
-        <geometry>
-          <sphere radius="${0.02+safety_distance}"  />
-        </geometry>
-      </collision>
     </link>
     <link name="${ns}_leftfinger">
@@ -59,4 +41,10 @@
         </geometry>
       </visual>
+      <collision>
+        <origin xyz="0 0.01 0.0415" rpy="0 0 0"/>
+        <geometry>
+          <sphere radius="${0.02+safety_distance}"  />
+        </geometry>
+      </collision>
     </link>
     <link name="${ns}_rightfinger">
@@ -67,4 +55,10 @@
         </geometry>
       </visual>
+      <collision>
+        <origin xyz="0 -0.01 0.0415" rpy="0 0 0"/>
+        <geometry>
+          <sphere radius="${0.02+safety_distance}"  />
+        </geometry>
+      </collision>
    </link>
     <joint name="${ns}_finger_joint1" type="prismatic">
