Commit message: Use both, detailed meshes and coarse collision geometries
They serve different purposes:
- coarse collision geometries mimic the internal self-collision checking
  of the real-robot controller
- mesh models should be used for collision checking with environmental objects

File: franka_description/robots/hand.xacro (robot description, xacro)
@@ -2,5 +2,5 @@
 <robot xmlns:xacro="http://www.ros.org/wiki/xacro" name="hand">
   <!-- safety_distance: Minimum safety distance in [m] by which the collision volumes are expanded and which is enforced during robot motions -->
-  <xacro:macro name="hand" params="connected_to:='' arm_id:='panda' rpy:='0 0 0' xyz:='0 0 0' safety_distance:=0">
+  <xacro:macro name="hand" params="connected_to:='' arm_id:='panda' rpy:='0 0 0' xyz:='0 0 0' safety_distance:=0 description_pkg:=franka_description">
     <xacro:unless value="${connected_to == ''}">
       <joint name="${arm_id}_hand_joint" type="fixed">
@@ -10,10 +10,6 @@
       </joint>
     </xacro:unless>
-    <link name="${arm_id}_hand">
-      <visual>
-        <geometry>
-          <mesh filename="package://franka_description/meshes/visual/hand.dae"/>
-        </geometry>
-      </visual>
+    <xacro:link name="hand">
+      <self_collision_geometries>
       <collision>
         <origin xyz="0 0 0.04" rpy="0 ${pi/2} ${pi/2}"/>
@@ -52,5 +48,6 @@
         </geometry>
       </collision>
-    </link>
+      </self_collision_geometries>
+    </xacro:link>
     <!-- Define the hand_tcp frame -->
     <link name="${arm_id}_hand_tcp" />
@@ -63,5 +60,5 @@
       <visual>
         <geometry>
-          <mesh filename="package://franka_description/meshes/visual/finger.dae"/>
+          <mesh filename="package://${description_pkg}/meshes/visual/finger.dae"/>
         </geometry>
       </visual>
@@ -71,5 +68,5 @@
         <origin xyz="0 0 0" rpy="0 0 ${pi}"/>
         <geometry>
-          <mesh filename="package://franka_description/meshes/visual/finger.dae"/>
+          <mesh filename="package://${description_pkg}/meshes/visual/finger.dae"/>
         </geometry>
       </visual>

File: franka_description/robots/panda_arm.urdf.xacro (robot description, xacro)
@@ -9,5 +9,6 @@
   <xacro:unless value="$(arg gazebo)">
     <!-- Create a URDF for a real hardware -->
-    <xacro:include filename="$(find franka_description)/robots/panda_arm.xacro" />
+    <xacro:include filename="utils.xacro" />
+    <xacro:include filename="panda_arm.xacro" />
     <xacro:panda_arm arm_id="$(arg arm_id)" safety_distance="0.03"/>
     <xacro:if value="$(arg hand)">

File: franka_description/robots/panda_arm.xacro (robot description, xacro)
@@ -11,10 +11,6 @@
       </joint>
     </xacro:unless>
-    <link name="${arm_id}_link0">
-      <visual>
-        <geometry>
-          <mesh filename="package://${description_pkg}/meshes/visual/link0.dae"/>
-        </geometry>
-      </visual>
+    <xacro:link name="link0">
+      <self_collision_geometries>
       <collision>
         <origin xyz="-0.075 0 0.06" rpy="0 ${pi/2} 0"/>
@@ -35,11 +31,8 @@
         </geometry>
       </collision>
-    </link>
-    <link name="${arm_id}_link1">
-      <visual>
-        <geometry>
-          <mesh filename="package://${description_pkg}/meshes/visual/link1.dae"/>
-        </geometry>
-      </visual>
+      </self_collision_geometries>
+    </xacro:link>
+    <xacro:link name="link1">
+      <self_collision_geometries>
       <collision>
         <origin xyz="0 0 -0.1915" rpy="0 0 0"/>
@@ -60,5 +53,6 @@
         </geometry>
       </collision>
-    </link>
+      </self_collision_geometries>
+    </xacro:link>
     <joint name="${arm_id}_joint1" type="revolute">
       <safety_controller k_position="100.0" k_velocity="40.0" soft_lower_limit="-2.8973" soft_upper_limit="2.8973"/>
@@ -69,10 +63,6 @@
       <limit effort="87" lower="-2.8973" upper="2.8973" velocity="2.1750"/>
     </joint>
-    <link name="${arm_id}_link2">
-      <visual>
-        <geometry>
-          <mesh filename="package://${description_pkg}/meshes/visual/link2.dae"/>
-        </geometry>
-      </visual>
+    <xacro:link name="link2">
+      <self_collision_geometries>
       <collision>
         <origin xyz="0 0 0" rpy="0 0 0"/>
@@ -93,5 +83,6 @@
         </geometry>
       </collision>
-    </link>
+      </self_collision_geometries>
+    </xacro:link>
     <joint name="${arm_id}_joint2" type="revolute">
       <safety_controller k_position="100.0" k_velocity="40.0" soft_lower_limit="-1.7628" soft_upper_limit="1.7628"/>
@@ -102,10 +93,6 @@
       <limit effort="87" lower="-1.7628" upper="1.7628" velocity="2.1750"/>
     </joint>
-    <link name="${arm_id}_link3">
-      <visual>
-        <geometry>
-          <mesh filename="package://${description_pkg}/meshes/visual/link3.dae"/>
-        </geometry>
-      </visual>
+    <xacro:link name="link3">
+      <self_collision_geometries>
       <collision>
         <origin xyz="0 0 -0.145" rpy="0 0 0"/>
@@ -126,5 +113,6 @@
         </geometry>
       </collision>
-    </link>
+      </self_collision_geometries>
+    </xacro:link>
     <joint name="${arm_id}_joint3" type="revolute">
       <safety_controller k_position="100.0" k_velocity="40.0" soft_lower_limit="-2.8973" soft_upper_limit="2.8973"/>
@@ -135,10 +123,6 @@
       <limit effort="87" lower="-2.8973" upper="2.8973" velocity="2.1750"/>
     </joint>
-    <link name="${arm_id}_link4">
-      <visual>
-        <geometry>
-          <mesh filename="package://${description_pkg}/meshes/visual/link4.dae"/>
-        </geometry>
-      </visual>
+    <xacro:link name="link4">
+      <self_collision_geometries>
       <collision>
         <origin xyz="0 0 0" rpy="0 0 0"/>
@@ -159,5 +143,6 @@
         </geometry>
       </collision>
-    </link>
+      </self_collision_geometries>
+    </xacro:link>
     <joint name="${arm_id}_joint4" type="revolute">
       <safety_controller k_position="100.0" k_velocity="40.0" soft_lower_limit="-3.0718" soft_upper_limit="-0.0698"/>
@@ -168,10 +153,6 @@
       <limit effort="87" lower="-3.0718" upper="-0.0698" velocity="2.1750"/>
     </joint>
-    <link name="${arm_id}_link5">
-      <visual>
-        <geometry>
-          <mesh filename="package://${description_pkg}/meshes/visual/link5.dae"/>
-        </geometry>
-      </visual>
+    <xacro:link name="link5">
+      <self_collision_geometries>
       <collision>
         <origin xyz="0 0 -0.26" rpy="0 0 0"/>
@@ -210,5 +191,6 @@
         </geometry>
       </collision>
-    </link>
+      </self_collision_geometries>
+    </xacro:link>
     <joint name="${arm_id}_joint5" type="revolute">
       <safety_controller k_position="100.0" k_velocity="40.0" soft_lower_limit="-2.8973" soft_upper_limit="2.8973"/>
@@ -219,10 +201,6 @@
       <limit effort="12" lower="-2.8973" upper="2.8973" velocity="2.6100"/>
     </joint>
-    <link name="${arm_id}_link6">
-      <visual>
-        <geometry>
-          <mesh filename="package://${description_pkg}/meshes/visual/link6.dae"/>
-        </geometry>
-      </visual>
+    <xacro:link name="link6">
+      <self_collision_geometries>
       <collision>
         <origin xyz="0 0 -0.03" rpy="0 0 0"/>
@@ -243,5 +221,6 @@
         </geometry>
       </collision>
-    </link>
+      </self_collision_geometries>
+    </xacro:link>
     <joint name="${arm_id}_joint6" type="revolute">
       <safety_controller k_position="100.0" k_velocity="40.0" soft_lower_limit="-0.0175" soft_upper_limit="3.7525"/>
@@ -252,10 +231,6 @@
       <limit effort="12" lower="-0.0175" upper="3.7525" velocity="2.6100"/>
     </joint>
-    <link name="${arm_id}_link7">
-      <visual>
-        <geometry>
-          <mesh filename="package://${description_pkg}/meshes/visual/link7.dae"/>
-        </geometry>
-      </visual>
+    <xacro:link name="link7">
+      <self_collision_geometries>
       <collision>
         <origin xyz="0 0 0.01" rpy="0 0 0"/>
@@ -276,5 +251,6 @@
         </geometry>
       </collision>
-    </link>
+      </self_collision_geometries>
+    </xacro:link>
     <joint name="${arm_id}_joint7" type="revolute">
       <safety_controller k_position="100.0" k_velocity="40.0" soft_lower_limit="-2.8973" soft_upper_limit="2.8973"/>
@@ -285,5 +261,6 @@
       <limit effort="12" lower="-2.8973" upper="2.8973" velocity="2.6100"/>
     </joint>
-    <link name="${arm_id}_link8">
+    <link name="${arm_id}_link8"/>
+    <link name="${arm_id}_link8_sc">
       <collision>
         <origin xyz="0.0424 0.0424 -0.0250" rpy="${pi} ${pi/2} ${pi/2}"/>
@@ -305,4 +282,8 @@
       </collision>
     </link>
+    <joint name="${arm_id}_link8_sc_joint" type="fixed">
+      <parent link="${arm_id}_link8" />
+      <child link="${arm_id}_link8_sc" />
+    </joint>
     <joint name="${arm_id}_joint8" type="fixed">
       <origin rpy="0 0 0" xyz="0 0 0.107"/>

File: franka_description/robots/utils.xacro (robot description, xacro)
@@ -1,4 +1,38 @@
 <?xml version="1.0"?>
 <robot xmlns:xacro="http://www.ros.org/wiki/xacro">
+  <!-- ========================================================== -->
+  <!-- Macro to add a single link, both with                      -->
+  <!--  * detailed meshes for environmental collision checking    -->
+  <!--  * and coarse geometry models for self-collision checking  -->
+  <!--                                                            -->
+  <!-- name:  Name of the robot link (without prefix)             -->
+  <!-- self_collision_geometries:  self <collision> models        -->
+  <!-- ========================================================== -->
+  <xacro:macro name="link" params="name prefix=${arm_id}_ **self_collision_geometries">
+    <!-- sub-link defining detailed meshes for collision with environment -->
+    <link name="${prefix}${name}">
+      <visual>
+        <geometry>
+          <mesh filename="package://${description_pkg}/meshes/visual/${name}.dae" />
+        </geometry>
+      </visual>
+      <collision>
+        <geometry>
+          <mesh filename="package://franka_description/meshes/collision/${name}.stl" />
+        </geometry>
+      </collision>
+    </link>
+    <!-- sub-link defining coarse geometries of real robot's internal self-collision -->
+    <link name="${prefix}${name}_sc">
+      <xacro:unless value="$(arg gazebo)">
+        <xacro:insert_block name="self_collision_geometries" />
+      </xacro:unless>
+    </link>
+    <!-- fixed joint between both sub-links -->
+    <joint name="${prefix}${name}_sc_joint" type="fixed">
+      <parent link="${prefix}${name}" />
+      <child link="${prefix}${name}_sc" />
+    </joint>
+  </xacro:macro>
   <!-- ========================================================== -->
   <!-- Adds the required tags to simulate one joint in gazebo     -->

Commit message: Add detailed collision meshes for fingers

File: franka_description/robots/hand.xacro (robot description, xacro)
@@ -57,4 +57,9 @@
         </geometry>
       </visual>
+      <collision>
+        <geometry>
+          <mesh filename="package://franka_description/meshes/collision/finger.stl" />
+        </geometry>
+      </collision>
     </link>
     <link name="${prefix}rightfinger">
@@ -65,4 +70,10 @@
         </geometry>
       </visual>
+      <collision>
+        <origin xyz="0 0 0" rpy="0 0 ${pi}" />
+        <geometry>
+          <mesh filename="package://franka_description/meshes/collision/finger.stl" />
+        </geometry>
+      </collision>
    </link>
     <joint name="${prefix}finger_joint1" type="prismatic">

Commit message: Unify real-world and Gazebo URDF descriptions
- Declare inertial properties in a yaml file
- Use xacro:inertial macro

File: franka_description/robots/hand.xacro (robot description, xacro)
@@ -62,4 +62,5 @@
         </geometry>
       </collision>
+      <xacro:inertial name="leftfinger" />
     </link>
     <link name="${prefix}rightfinger">
@@ -76,4 +77,5 @@
         </geometry>
       </collision>
+      <xacro:inertial name="rightfinger" />
    </link>
     <joint name="${prefix}finger_joint1" type="prismatic">

File: franka_description/robots/panda_arm.urdf.xacro (robot description, xacro)
@@ -9,26 +9,17 @@
   <!-- Name prefix used for joints and links. Property is implicitly passed to macros. -->
   <xacro:property name="prefix" value="$(arg arm_id)_" />
-  <xacro:unless value="$(arg gazebo)">
-    <!-- Create a URDF for a real hardware -->
-    <xacro:include filename="utils.xacro" />
-    <xacro:include filename="arm.xacro" />
-    <xacro:arm safety_distance="0.03" />
-    <xacro:if value="$(arg hand)">
-      <xacro:include filename="hand.xacro"/>
-      <xacro:hand rpy="0 0 ${-pi/4}" connected_to="${prefix}link8" safety_distance="0.03"/>
-    </xacro:if>
-  </xacro:unless>
+  <!-- Load interial properties. Property is implicitly passed to macros. -->
+  <xacro:property name="inertial" value="${xacro.load_yaml('inertial.yaml')}" />
+  <xacro:include filename="utils.xacro" />
+  <xacro:include filename="arm.xacro" />
+  <xacro:arm safety_distance="0.03" />
+  <xacro:if value="$(arg hand)">
+    <xacro:include filename="hand.xacro"/>
+    <xacro:hand rpy="0 0 ${-pi/4}" connected_to="${prefix}link8" safety_distance="0.03"/>
+  </xacro:if>
+  <!-- Define additional Gazebo tags -->
   <xacro:if value="$(arg gazebo)">
     <xacro:arg name="xyz" default="0 0 0" />
     <xacro:arg name="rpy" default="0 0 0" />
-    <!-- Create a simulatable URDF -->
-    <xacro:include filename="utils.xacro" />
-    <xacro:include filename="panda_gazebo.xacro" />
-    <xacro:arm />
-    <xacro:if value="$(arg hand)">
-      <xacro:hand rpy="0 0 ${-pi/4}" connected_to="${prefix}link8" />
-      <xacro:gazebo-joint joint="${prefix}finger_joint1" transmission="hardware_interface/EffortJointInterface" />
-      <xacro:gazebo-joint joint="${prefix}finger_joint2" transmission="hardware_interface/EffortJointInterface" />
-    </xacro:if>
     <!-- Gazebo requires a joint to a link called "world" for statically mounted robots -->
     <link name="world" />
@@ -45,4 +36,11 @@
     <xacro:gazebo-joint joint="${prefix}joint6" transmission="hardware_interface/EffortJointInterface" />
     <xacro:gazebo-joint joint="${prefix}joint7" transmission="hardware_interface/EffortJointInterface" />
+    <xacro:if value="$(arg hand)">
+      <xacro:gazebo-joint joint="${prefix}finger_joint1" transmission="hardware_interface/EffortJointInterface" />
+      <xacro:gazebo-joint joint="${prefix}finger_joint2" transmission="hardware_interface/EffortJointInterface" />
+      <!-- Friction specific material for Rubber/Rubber contact -->
+      <xacro:gazebo-friction link="${prefix}leftfinger" mu="1.13" />
+      <xacro:gazebo-friction link="${prefix}rightfinger" mu="1.13" />
+    </xacro:if>
     <xacro:transmission-franka-state />
     <xacro:transmission-franka-model root="${prefix}joint1" tip="${prefix}joint8" />

File: franka_description/robots/utils.xacro (robot description, xacro)
@@ -1,4 +1,25 @@
 <?xml version="1.0"?>
 <robot xmlns:xacro="http://www.ros.org/wiki/xacro">
+  <!-- ============================================================ -->
+  <!-- Macro to add an <interial> tag based on yaml-load properties -->
+  <!--                                                              -->
+  <!-- name:     Name of the robot link (without prefix)            -->
+  <!-- inertial: Dictionary of inertia properties                   -->
+  <!-- ============================================================ -->
+  <xacro:macro name="inertial" params="inertial:=^ name:=^">
+    <xacro:if value="$(arg gazebo)">
+      <xacro:unless value="${inertial.get(name, None)}">${xacro.warning('No inertia properties defined for: ' + name)}</xacro:unless>
+      <xacro:if value="${inertial.get(name, None)}">
+        <!-- Access inertia properties of link 'name' -->
+        <xacro:property name="inertial" value="${inertial[name]}" lazy_eval="false" />
+        <inertial>
+          <origin rpy="${inertial.origin.rpy}" xyz="${inertial.origin.xyz}" />
+          <mass value="${inertial.mass}" />
+          <xacro:property name="I" value="${inertial.inertia}" />
+          <inertia ixx="${I.xx}" ixy="${I.xy}" ixz="${I.xz}" iyy="${I.yy}" iyz="${I.yz}" izz="${I.zz}" />
+        </inertial>
+      </xacro:if>
+    </xacro:if>
+  </xacro:macro>
   <!-- ========================================================== -->
   <!-- Macro to add a single link, both with                      -->
@@ -22,4 +43,5 @@
         </geometry>
       </collision>
+      <xacro:inertial />
     </link>
     <!-- sub-link defining coarse geometries of real robot's internal self-collision -->
