Commit message: Restore Melodic compatibility
xacro requires macro names to be different from actual tag names.

File: franka_description/robots/hand.xacro (robot description, xacro)
@@ -10,5 +10,5 @@
       </joint>
     </xacro:unless>
-    <xacro:link name="hand">
+    <xacro:link_detailed_coarse name="hand">
       <self_collision_geometries>
         <collision>
@@ -49,5 +49,5 @@
         </collision>
       </self_collision_geometries>
-    </xacro:link>
+    </xacro:link_detailed_coarse>
     <!-- Define the hand_tcp frame -->
     <link name="${arm_id}_hand_tcp" />
@@ -91,5 +91,5 @@
         </geometry>
       </collision>
-      <xacro:inertial name="leftfinger" />
+      <xacro:inertial_props name="leftfinger" />
     </link>
     <link name="${arm_id}_rightfinger">
@@ -128,5 +128,5 @@
         </geometry>
       </collision>
-      <xacro:inertial name="rightfinger" />
+      <xacro:inertial_props name="rightfinger" />
     </link>
     <joint name="${arm_id}_finger_joint1" type="prismatic">

File: franka_description/robots/panda_arm.xacro (robot description, xacro)
@@ -11,5 +11,5 @@
       </joint>
     </xacro:unless>
-    <xacro:link name="link0">
+    <xacro:link_detailed_coarse name="link0">
       <self_collision_geometries>
       <collision>
@@ -32,6 +32,6 @@
       </collision>
       </self_collision_geometries>
-    </xacro:link>
-    <xacro:link name="link1">
+    </xacro:link_detailed_coarse>
+    <xacro:link_detailed_coarse name="link1">
       <self_collision_geometries>
       <collision>
@@ -54,5 +54,5 @@
       </collision>
       </self_collision_geometries>
-    </xacro:link>
+    </xacro:link_detailed_coarse>
     <joint name="${arm_id}_joint1" type="revolute">
       <safety_controller k_position="100.0" k_velocity="40.0" soft_lower_limit="-2.8973" soft_upper_limit="2.8973"/>
@@ -64,5 +64,5 @@
       <dynamics D="1" K="7000" damping="0.003" friction="0.0" mu_coulomb="0" mu_viscous="16"/>
     </joint>
-    <xacro:link name="link2">
+    <xacro:link_detailed_coarse name="link2">
       <self_collision_geometries>
       <collision>
@@ -85,5 +85,5 @@
       </collision>
       </self_collision_geometries>
-    </xacro:link>
+    </xacro:link_detailed_coarse>
     <joint name="${arm_id}_joint2" type="revolute">
       <safety_controller k_position="100.0" k_velocity="40.0" soft_lower_limit="-1.7628" soft_upper_limit="1.7628"/>
@@ -95,5 +95,5 @@
       <dynamics D="1" K="7000" damping="0.003" friction="0.0" mu_coulomb="0" mu_viscous="16"/>
     </joint>
-    <xacro:link name="link3">
+    <xacro:link_detailed_coarse name="link3">
       <self_collision_geometries>
       <collision>
@@ -116,5 +116,5 @@
       </collision>
       </self_collision_geometries>
-    </xacro:link>
+    </xacro:link_detailed_coarse>
     <joint name="${arm_id}_joint3" type="revolute">
       <safety_controller k_position="100.0" k_velocity="40.0" soft_lower_limit="-2.8973" soft_upper_limit="2.8973"/>
@@ -126,5 +126,5 @@
       <dynamics D="1" K="7000" damping="0.003" friction="0.0" mu_coulomb="0" mu_viscous="16"/>
     </joint>
-    <xacro:link name="link4">
+    <xacro:link_detailed_coarse name="link4">
       <self_collision_geometries>
       <collision>
@@ -147,5 +147,5 @@
       </collision>
       </self_collision_geometries>
-    </xacro:link>
+    </xacro:link_detailed_coarse>
     <joint name="${arm_id}_joint4" type="revolute">
       <safety_controller k_position="100.0" k_velocity="40.0" soft_lower_limit="-3.0718" soft_upper_limit="-0.0698"/>
@@ -157,5 +157,5 @@
       <dynamics D="1" K="7000" damping="0.003" friction="0.0" mu_coulomb="0" mu_viscous="16"/>
     </joint>
-    <xacro:link name="link5">
+    <xacro:link_detailed_coarse name="link5">
       <self_collision_geometries>
       <collision>
@@ -196,5 +196,5 @@
       </collision>
       </self_collision_geometries>
-    </xacro:link>
+    </xacro:link_detailed_coarse>
     <joint name="${arm_id}_joint5" type="revolute">
       <safety_controller k_position="100.0" k_velocity="40.0" soft_lower_limit="-2.8973" soft_upper_limit="2.8973"/>
@@ -206,5 +206,5 @@
       <dynamics D="1" K="7000" damping="0.003" friction="0.0" mu_coulomb="0" mu_viscous="16"/>
     </joint>
-    <xacro:link name="link6">
+    <xacro:link_detailed_coarse name="link6">
       <self_collision_geometries>
       <collision>
@@ -227,5 +227,5 @@
       </collision>
       </self_collision_geometries>
-    </xacro:link>
+    </xacro:link_detailed_coarse>
     <joint name="${arm_id}_joint6" type="revolute">
       <safety_controller k_position="100.0" k_velocity="40.0" soft_lower_limit="-0.0175" soft_upper_limit="3.7525"/>
@@ -237,5 +237,5 @@
       <dynamics D="1" K="7000" damping="0.003" friction="0.0" mu_coulomb="0" mu_viscous="16"/>
     </joint>
-    <xacro:link name="link7">
+    <xacro:link_detailed_coarse name="link7">
       <self_collision_geometries>
       <collision>
@@ -258,5 +258,5 @@
       </collision>
       </self_collision_geometries>
-    </xacro:link>
+    </xacro:link_detailed_coarse>
     <joint name="${arm_id}_joint7" type="revolute">
       <safety_controller k_position="100.0" k_velocity="40.0" soft_lower_limit="-2.8973" soft_upper_limit="2.8973"/>

File: franka_description/robots/utils.xacro (robot description, xacro)
@@ -7,5 +7,5 @@
   <!-- inertial: Dictionary of inertia properties                   -->
   <!-- ============================================================ -->
-  <xacro:macro name="inertial" params="inertial:=^ name:=^">
+  <xacro:macro name="inertial_props" params="inertial:=^ name:=^">
     <xacro:if value="$(arg gazebo)">
       <xacro:unless value="${name in inertial}">${xacro.warning('No inertia properties defined for: ' + name)}</xacro:unless>
@@ -30,5 +30,5 @@
   <!-- self_collision_geometries:  self <collision> models        -->
   <!-- ========================================================== -->
-  <xacro:macro name="link" params="name prefix=${arm_id}_ **self_collision_geometries">
+  <xacro:macro name="link_detailed_coarse" params="name prefix=${arm_id}_ **self_collision_geometries">
     <!-- sub-link defining detailed meshes for collision with environment -->
     <link name="${prefix}${name}">
@@ -43,5 +43,5 @@
         </geometry>
       </collision>
-      <xacro:inertial />
+      <xacro:inertial_props />
     </link>
     <!-- sub-link defining coarse geometries of real robot's internal self-collision -->

Commit message: CHANGE: Use `<xacro:collision_capsule>` also for hand.xacro

File: franka_description/robots/hand.xacro (robot description, xacro)
@@ -12,40 +12,6 @@
     <xacro:link_detailed_coarse name="hand">
       <self_collision_geometries>
-        <collision>
-          <origin xyz="0 0 0.04" rpy="0 ${pi/2} ${pi/2}" />
-          <geometry>
-            <cylinder radius="${0.04+safety_distance}" length="0.1" />
-          </geometry>
-        </collision>
-        <collision>
-          <origin xyz="0 -0.05 0.04" rpy="0 0 0" />
-          <geometry>
-            <sphere radius="${0.04+safety_distance}" />
-          </geometry>
-        </collision>
-        <collision>
-          <origin xyz="0 0.05 0.04" rpy="0 0 0" />
-          <geometry>
-            <sphere radius="${0.04+safety_distance}" />
-          </geometry>
-        </collision>
-        <collision>
-          <origin xyz="0 0 0.1" rpy="0 ${pi/2} ${pi/2}" />
-          <geometry>
-            <cylinder radius="${0.02+safety_distance}" length="0.1" />
-          </geometry>
-        </collision>
-        <collision>
-          <origin xyz="0 -0.05 0.1" rpy="0 0 0" />
-          <geometry>
-            <sphere radius="${0.02+safety_distance}" />
-          </geometry>
-        </collision>
-        <collision>
-          <origin xyz="0 0.05 0.1" rpy="0 0 0" />
-          <geometry>
-            <sphere radius="${0.02+safety_distance}" />
-          </geometry>
-        </collision>
+        <xacro:collision_capsule xyz="0 0 0.04" direction="y" radius="${0.04+safety_distance}" length="0.1" />
+        <xacro:collision_capsule xyz="0 0 0.10" direction="y" radius="${0.02+safety_distance}" length="0.1" />
       </self_collision_geometries>
     </xacro:link_detailed_coarse>

Commit message: CHANGE: Rename xacro:{link_detailed_coarse -> link_with_sc}
The name "detailed_coarse" is a bit contradicting. More suitable might be a name
which indicates that existing `<link>`s are augmented with additional
functionality such as self-collision geometries. This in mind it also should
also be rather consise so I went with `link_with_sc`.

File: franka_description/robots/hand.xacro (robot description, xacro)
@@ -10,10 +10,10 @@
       </joint>
     </xacro:unless>
-    <xacro:link_detailed_coarse name="hand">
+    <xacro:link_with_sc name="hand">
       <self_collision_geometries>
         <xacro:collision_capsule xyz="0 0 0.04" direction="y" radius="${0.04+safety_distance}" length="0.1" />
         <xacro:collision_capsule xyz="0 0 0.10" direction="y" radius="${0.02+safety_distance}" length="0.1" />
       </self_collision_geometries>
-    </xacro:link_detailed_coarse>
+    </xacro:link_with_sc>
     <!-- Define the hand_tcp frame -->
     <link name="${arm_id}_hand_tcp" />

File: franka_description/robots/panda_arm.xacro (robot description, xacro)
@@ -11,14 +11,14 @@
       </joint>
     </xacro:unless>
-    <xacro:link_detailed_coarse name="link0">
+    <xacro:link_with_sc name="link0">
       <self_collision_geometries>
         <xacro:collision_capsule xyz="-0.075 0 0.06" direction="x" radius="${0.06+safety_distance}" length="0.03" />
       </self_collision_geometries>
-    </xacro:link_detailed_coarse>
-    <xacro:link_detailed_coarse name="link1">
+    </xacro:link_with_sc>
+    <xacro:link_with_sc name="link1">
       <self_collision_geometries>
         <xacro:collision_capsule xyz="0 0 -191.5e-3" radius="${0.06+safety_distance}" length="0.283" />
       </self_collision_geometries>
-    </xacro:link_detailed_coarse>
+    </xacro:link_with_sc>
     <joint name="${arm_id}_joint1" type="revolute">
       <safety_controller k_position="100.0" k_velocity="40.0" soft_lower_limit="-2.8973" soft_upper_limit="2.8973" />
@@ -30,9 +30,9 @@
       <dynamics D="1" K="7000" damping="0.003" friction="0.0" mu_coulomb="0" mu_viscous="16" />
     </joint>
-    <xacro:link_detailed_coarse name="link2">
+    <xacro:link_with_sc name="link2">
       <self_collision_geometries>
         <xacro:collision_capsule xyz="0 0 0" radius="${0.06+safety_distance}" length="0.12" />
       </self_collision_geometries>
-    </xacro:link_detailed_coarse>
+    </xacro:link_with_sc>
     <joint name="${arm_id}_joint2" type="revolute">
       <safety_controller k_position="100.0" k_velocity="40.0" soft_lower_limit="-1.7628" soft_upper_limit="1.7628" />
@@ -44,9 +44,9 @@
       <dynamics D="1" K="7000" damping="0.003" friction="0.0" mu_coulomb="0" mu_viscous="16" />
     </joint>
-    <xacro:link_detailed_coarse name="link3">
+    <xacro:link_with_sc name="link3">
       <self_collision_geometries>
         <xacro:collision_capsule xyz="0 0 -0.145" radius="${0.06+safety_distance}" length="0.15" />
       </self_collision_geometries>
-    </xacro:link_detailed_coarse>
+    </xacro:link_with_sc>
     <joint name="${arm_id}_joint3" type="revolute">
       <safety_controller k_position="100.0" k_velocity="40.0" soft_lower_limit="-2.8973" soft_upper_limit="2.8973" />
@@ -58,9 +58,9 @@
       <dynamics D="1" K="7000" damping="0.003" friction="0.0" mu_coulomb="0" mu_viscous="16" />
     </joint>
-    <xacro:link_detailed_coarse name="link4">
+    <xacro:link_with_sc name="link4">
       <self_collision_geometries>
         <xacro:collision_capsule xyz="0 0 0" radius="${0.06+safety_distance}" length="0.12" />
      </self_collision_geometries>
-    </xacro:link_detailed_coarse>
+    </xacro:link_with_sc>
     <joint name="${arm_id}_joint4" type="revolute">
       <safety_controller k_position="100.0" k_velocity="40.0" soft_lower_limit="-3.0718" soft_upper_limit="-0.0698" />
@@ -72,10 +72,10 @@
       <dynamics D="1" K="7000" damping="0.003" friction="0.0" mu_coulomb="0" mu_viscous="16" />
     </joint>
-    <xacro:link_detailed_coarse name="link5">
+    <xacro:link_with_sc name="link5">
       <self_collision_geometries>
         <xacro:collision_capsule xyz="0 0 -0.26"    radius="${0.060+safety_distance}" length="0.10" />
         <xacro:collision_capsule xyz="0 0.08 -0.13" radius="${0.025+safety_distance}" length="0.14" />
       </self_collision_geometries>
-    </xacro:link_detailed_coarse>
+    </xacro:link_with_sc>
     <joint name="${arm_id}_joint5" type="revolute">
       <safety_controller k_position="100.0" k_velocity="40.0" soft_lower_limit="-2.8973" soft_upper_limit="2.8973" />
@@ -87,9 +87,9 @@
       <dynamics D="1" K="7000" damping="0.003" friction="0.0" mu_coulomb="0" mu_viscous="16" />
     </joint>
-    <xacro:link_detailed_coarse name="link6">
+    <xacro:link_with_sc name="link6">
       <self_collision_geometries>
         <xacro:collision_capsule xyz="0 0 -0.03" radius="${0.05+safety_distance}" length="0.08" />
       </self_collision_geometries>
-    </xacro:link_detailed_coarse>
+    </xacro:link_with_sc>
     <joint name="${arm_id}_joint6" type="revolute">
       <safety_controller k_position="100.0" k_velocity="40.0" soft_lower_limit="-0.0175" soft_upper_limit="3.7525" />
@@ -101,10 +101,10 @@
       <dynamics D="1" K="7000" damping="0.003" friction="0.0" mu_coulomb="0" mu_viscous="16" />
     </joint>
-    <xacro:link_detailed_coarse name="link7" rpy="0 0 ${pi/4}">
+    <xacro:link_with_sc name="link7" rpy="0 0 ${pi/4}">
       <self_collision_geometries>
         <xacro:collision_capsule xyz="0 0 0.01" direction="z" radius="${0.04+safety_distance}" length="0.14" />
         <xacro:collision_capsule xyz="0.06 0 0.082" direction="x" radius="${0.03+safety_distance}"  length="0.01" />
       </self_collision_geometries>
-    </xacro:link_detailed_coarse>
+    </xacro:link_with_sc>
     <joint name="${arm_id}_joint7" type="revolute">
       <safety_controller k_position="100.0" k_velocity="40.0" soft_lower_limit="-2.8973" soft_upper_limit="2.8973"/>

File: franka_description/robots/utils.xacro (robot description, xacro)
@@ -26,4 +26,5 @@
   <!--  * detailed meshes for environmental collision checking    -->
   <!--  * and coarse geometry models for self-collision checking  -->
+  <!--    (only if 'gazebo' arg is set)                           -->
   <!--                                                            -->
   <!-- name:  Name of the robot link (without prefix)             -->
@@ -31,5 +32,5 @@
   <!-- self_collision_geometries:  self <collision> models        -->
   <!-- ========================================================== -->
-  <xacro:macro name="link_detailed_coarse" params="name prefix=${arm_id}_ rpy:='0 0 0' **self_collision_geometries">
+  <xacro:macro name="link_with_sc" params="name prefix=${arm_id}_ rpy:='0 0 0' **self_collision_geometries">
     <!-- sub-link defining detailed meshes for collision with environment -->
     <link name="${prefix}${name}">

Commit message: FIX: Also pass `gazebo` arg correctly down into `hand.xacro`

File: franka_description/robots/hand.xacro (robot description, xacro)
@@ -2,5 +2,5 @@
 <robot xmlns:xacro="http://www.ros.org/wiki/xacro" name="hand">
   <!-- safety_distance: Minimum safety distance in [m] by which the collision volumes are expanded and which is enforced during robot motions -->
-  <xacro:macro name="hand" params="connected_to:='' arm_id:='panda' rpy:='0 0 0' xyz:='0 0 0' safety_distance:=0 description_pkg:=franka_description">
+  <xacro:macro name="hand" params="connected_to:='' arm_id:='panda' rpy:='0 0 0' xyz:='0 0 0' safety_distance:=0 gazebo:=false description_pkg:=franka_description">
     <xacro:unless value="${connected_to == ''}">
       <joint name="${arm_id}_hand_joint" type="fixed">
@@ -10,5 +10,5 @@
       </joint>
     </xacro:unless>
-    <xacro:link_with_sc name="hand">
+    <xacro:link_with_sc name="hand" gazebo="${gazebo}">
       <self_collision_geometries>
         <xacro:collision_capsule xyz="0 0 0.04" direction="y" radius="${0.04+safety_distance}" length="0.1" />

File: franka_description/robots/panda_arm.urdf.xacro (robot description, xacro)
@@ -12,5 +12,5 @@
   <xacro:if value="$(arg hand)">
     <xacro:include filename="hand.xacro"/>
-    <xacro:hand arm_id="$(arg arm_id)" rpy="0 0 ${-pi/4}" connected_to="$(arg arm_id)_link8" safety_distance="0.03"/>
+    <xacro:hand arm_id="$(arg arm_id)" rpy="0 0 ${-pi/4}" connected_to="$(arg arm_id)_link8" safety_distance="0.03" gazebo="$(arg gazebo)"/>
   </xacro:if>
   <!-- Define additional Gazebo tags -->

Commit message: ADD: `tcp_xyz` & `tcp_rpy` offsets to XACRO files
This allows to specify a move the TCP for MoveIT's `$(arm_id)_manipulator` move group

File: franka_description/robots/hand.xacro (robot description, xacro)
@@ -2,5 +2,5 @@
 <robot xmlns:xacro="http://www.ros.org/wiki/xacro" name="hand">
   <!-- safety_distance: Minimum safety distance in [m] by which the collision volumes are expanded and which is enforced during robot motions -->
-  <xacro:macro name="hand" params="connected_to:='' arm_id:='panda' rpy:='0 0 0' xyz:='0 0 0' safety_distance:=0 gazebo:=false description_pkg:=franka_description">
+  <xacro:macro name="hand" params="connected_to:='' arm_id:='panda' rpy:='0 0 0' xyz:='0 0 0' tcp_xyz:='0 0 0.1034' tcp_rpy:='0 0 0' safety_distance:=0 gazebo:=false description_pkg:=franka_description">
     <xacro:unless value="${connected_to == ''}">
       <joint name="${arm_id}_hand_joint" type="fixed">
@@ -19,5 +19,5 @@
     <link name="${arm_id}_hand_tcp" />
     <joint name="${arm_id}_hand_tcp_joint" type="fixed">
-      <origin xyz="0 0 0.1034" rpy="0 0 0" />
+      <origin xyz="${tcp_xyz}" rpy="${tcp_rpy}" />
       <parent link="${arm_id}_hand" />
       <child link="${arm_id}_hand_tcp" />

File: franka_description/robots/panda_arm.urdf.xacro (robot description, xacro)
@@ -5,4 +5,8 @@
   <!-- Should a franka_gripper be mounted at the flange?" -->
   <xacro:arg name="hand" default="false" />
+  <!-- Positional offset between $(arm_id)_hand -> $(arm_id)_hand_tcp [m]. Only used when hand:=true -->
+  <xacro:arg name="tcp_xyz" default="0 0 0.1034" />
+  <!-- Rotational offset between $(arm_id)_hand -> $(arm_id)_hand_tcp [rad]. Only used when hand:=true -->
+  <xacro:arg name="tcp_rpy" default="0 0 0" />
   <!-- Is the robot being simulated in gazebo?" -->
   <xacro:arg name="gazebo" default="false" />
@@ -12,5 +16,13 @@
   <xacro:if value="$(arg hand)">
     <xacro:include filename="hand.xacro"/>
-    <xacro:hand arm_id="$(arg arm_id)" rpy="0 0 ${-pi/4}" connected_to="$(arg arm_id)_link8" safety_distance="0.03" gazebo="$(arg gazebo)"/>
+    <xacro:hand
+        arm_id="$(arg arm_id)"
+        rpy="0 0 ${-pi/4}"
+        tcp_xyz="$(arg tcp_xyz)"
+        tcp_rpy="$(arg tcp_rpy)"
+        connected_to="$(arg arm_id)_link8"
+        safety_distance="0.03"
+        gazebo="$(arg gazebo)"
+     />
   </xacro:if>
   <!-- Define additional Gazebo tags -->
