Commit message: CHANGE: Add `gazebo` bool argument to `panda_arm.urdf.xacro`

File: franka_description/robots/panda_arm.urdf.xacro (robot description, xacro)
@@ -1,5 +1,41 @@
 <?xml version='1.0' encoding='utf-8'?>
 <robot xmlns:xacro="http://www.ros.org/wiki/xacro" name="panda">
-  <xacro:include filename="$(find franka_description)/robots/panda_arm.xacro" />
-  <xacro:panda_arm safety_distance="0.03"/>
+  <xacro:arg name="gazebo" default="false" />
+  <xacro:unless value="$(arg gazebo)">
+    <!-- Create a URDF for a real hardware -->
+    <xacro:include filename="$(find franka_description)/robots/panda_arm.xacro" />
+    <xacro:panda_arm safety_distance="0.03"/>
+  </xacro:unless>
+  <xacro:if value="$(arg gazebo)">
+    <!-- Create a simulatable URDF -->
+    <xacro:include filename="$(find franka_description)/robots/utils.xacro" />
+    <xacro:include filename="$(find franka_description)/robots/panda_gazebo.xacro" />
+    <xacro:property name="arm_id" value="panda" />
+    <xacro:panda_arm arm_id="${arm_id}" />
+    <!-- Gazebo requires a joint to a link called "world" for statically mounted robots -->
+    <link name="world" />
+    <joint name="world_joint" type="fixed">
+      <parent link="world" />
+      <child  link="${arm_id}_link0" />
+    </joint>
+    <xacro:gazebo-joint joint="${arm_id}_joint1" transmission="hardware_interface/EffortJointInterface" />
+    <xacro:gazebo-joint joint="${arm_id}_joint2" transmission="hardware_interface/EffortJointInterface" />
+    <xacro:gazebo-joint joint="${arm_id}_joint3" transmission="hardware_interface/EffortJointInterface" />
+    <xacro:gazebo-joint joint="${arm_id}_joint4" transmission="hardware_interface/EffortJointInterface" />
+    <xacro:gazebo-joint joint="${arm_id}_joint5" transmission="hardware_interface/EffortJointInterface" />
+    <xacro:gazebo-joint joint="${arm_id}_joint6" transmission="hardware_interface/EffortJointInterface" />
+    <xacro:gazebo-joint joint="${arm_id}_joint7" transmission="hardware_interface/EffortJointInterface" />
+    <xacro:transmission-franka-state arm_id="${arm_id}" />
+    <xacro:transmission-franka-model arm_id="${arm_id}"
+       root="${arm_id}_joint1"
+       tip="${arm_id}_joint8"
+     />
+    <gazebo>
+      <plugin name="gazebo_ros_control" filename="libgazebo_ros_control.so">
+        <robotNamespace>${arm_id}</robotNamespace>
+        <controlPeriod>0.001</controlPeriod>
+        <robotSimType>franka_gazebo/FrankaHWSim</robotSimType>
+      </plugin>
+    </gazebo>
+  </xacro:if>
 </robot>

Commit message: CHANGE: Let real panda URDF also take arm_id as optional argument

File: franka_description/robots/panda_arm.urdf.xacro (robot description, xacro)
@@ -1,13 +1,15 @@
 <?xml version='1.0' encoding='utf-8'?>
 <robot xmlns:xacro="http://www.ros.org/wiki/xacro" name="panda">
+  <xacro:arg name="arm_id" default="panda" /> <!-- Name of this panda -->
   <xacro:arg name="hand"   default="false" /> <!-- Should a franka_gripper be mounted at the flange?" -->
   <xacro:arg name="gazebo" default="false" /> <!-- Is the robot being simulated in gazebo?" -->
+  <xacro:property name="arm_id" value="$(arg arm_id)" />
   <xacro:unless value="$(arg gazebo)">
     <!-- Create a URDF for a real hardware -->
     <xacro:include filename="$(find franka_description)/robots/panda_arm.xacro" />
-    <xacro:panda_arm safety_distance="0.03"/>
+    <xacro:panda_arm arm_id="${arm_id}" safety_distance="0.03"/>
     <xacro:if value="$(arg hand)">
       <xacro:include filename="$(find franka_description)/robots/hand.xacro"/>
-      <xacro:hand ns="panda" rpy="0 0 ${-pi/4}" connected_to="panda_link8" safety_distance="0.03"/>
+      <xacro:hand ns="${arm_id}" rpy="0 0 ${-pi/4}" connected_to="${arm_id}_link8" safety_distance="0.03"/>
     </xacro:if>
   </xacro:unless>
@@ -16,5 +18,4 @@
     <xacro:include filename="$(find franka_description)/robots/utils.xacro" />
     <xacro:include filename="$(find franka_description)/robots/panda_gazebo.xacro" />
-    <xacro:property name="arm_id" value="panda" />
     <xacro:panda_arm arm_id="${arm_id}" />
     <xacro:if value="$(arg hand)">

Commit message: FIX: Use XYZ/RPY offsets in URDF not in Gazebo Spawner
Problem is, when you hand the parameters to the gazebo model spawner, the models
will appear correctly in gazebo at the specified pose, but Gazebo will publish a
TF from `world` -> `$(arm_id)_link0` with identity. This means that when placing
multiple pandas, they appear correctly in Gazebo, however ROS "thinks" they all
overlap and are attached to the world's origin at (0,0,0).

To fix this, we don't pass the pose to the model spawner, but rather to the URDF
directly. In here, the values specifiy the `<origin>` of the joint from `world`
-> `$(arm_id)_link0`, which then is published correctly as TF in ROS.

File: franka_description/robots/panda_arm.urdf.xacro (robot description, xacro)
@@ -15,4 +15,10 @@
   </xacro:unless>
   <xacro:if value="$(arg gazebo)">
+    <xacro:arg name="x" default="0" />
+    <xacro:arg name="y" default="0" />
+    <xacro:arg name="z" default="0" />
+    <xacro:arg name="R" default="0" />
+    <xacro:arg name="P" default="0" />
+    <xacro:arg name="Y" default="0" />
     <!-- Create a simulatable URDF -->
     <xacro:include filename="$(find franka_description)/robots/utils.xacro" />
@@ -27,4 +33,5 @@
     <link name="world" />
     <joint name="world_joint" type="fixed">
+      <origin xyz="$(arg x) $(arg y) $(arg z)" rpy="$(arg R) $(arg P) $(arg Y)" />
       <parent link="world" />
       <child  link="${arm_id}_link0" />

Commit message: FIX: Make Xacro args for root pose for consistent with `xyz`/`rpy`

File: franka_description/robots/panda_arm.urdf.xacro (robot description, xacro)
@@ -15,10 +15,6 @@
   </xacro:unless>
   <xacro:if value="$(arg gazebo)">
-    <xacro:arg name="x" default="0" />
-    <xacro:arg name="y" default="0" />
-    <xacro:arg name="z" default="0" />
-    <xacro:arg name="R" default="0" />
-    <xacro:arg name="P" default="0" />
-    <xacro:arg name="Y" default="0" />
+    <xacro:arg name="xyz" default="0 0 0" />
+    <xacro:arg name="rpy" default="0 0 0" />
     <!-- Create a simulatable URDF -->
     <xacro:include filename="$(find franka_description)/robots/utils.xacro" />
@@ -33,5 +29,5 @@
     <link name="world" />
     <joint name="world_joint" type="fixed">
-      <origin xyz="$(arg x) $(arg y) $(arg z)" rpy="$(arg R) $(arg P) $(arg Y)" />
+      <origin xyz="$(arg xyz)" rpy="$(arg rpy)" />
       <parent link="world" />
       <child  link="${arm_id}_link0" />

Commit message: Adds the ability to specify the safety_distance

File: franka_description/robots/panda_arm.urdf.xacro (robot description, xacro)
@@ -4,12 +4,14 @@
   <xacro:arg name="hand"   default="false" /> <!-- Should a franka_gripper be mounted at the flange?" -->
   <xacro:arg name="gazebo" default="false" /> <!-- Is the robot being simulated in gazebo?" -->
+  <xacro:arg name="safety_distance" default="0.03" /> <!-- The safety distance that is used for the collisions. Please take care when changing this value!" -->
   <xacro:property name="arm_id" value="$(arg arm_id)" />
+  <xacro:property name="safety_distance" value="$(arg safety_distance)" />
   <xacro:unless value="$(arg gazebo)">
     <!-- Create a URDF for a real hardware -->
     <xacro:include filename="$(find franka_description)/robots/panda_arm.xacro" />
-    <xacro:panda_arm arm_id="${arm_id}" safety_distance="0.03"/>
+    <xacro:panda_arm arm_id="${arm_id}" safety_distance="${safety_distance}"/>
     <xacro:if value="$(arg hand)">
       <xacro:include filename="$(find franka_description)/robots/hand.xacro"/>
-      <xacro:hand ns="${arm_id}" rpy="0 0 ${-pi/4}" connected_to="${arm_id}_link8" safety_distance="0.03"/>
+      <xacro:hand ns="${arm_id}" rpy="0 0 ${-pi/4}" connected_to="${arm_id}_link8" safety_distance="${safety_distance}"/>
     </xacro:if>
   </xacro:unless>

Commit message: Adds the 'transmission' arg to the 'panda_arm.urdf.xacro' file
This commit gives users the ability to set the hardware_interface that
is used in the panda arm joints when loading the 'panda_arm.urdf.xacro'
file.

File: franka_description/robots/panda_arm.urdf.xacro (robot description, xacro)
@@ -1,10 +1,10 @@
 <?xml version='1.0' encoding='utf-8'?>
 <robot xmlns:xacro="http://www.ros.org/wiki/xacro" name="panda">
-  <!-- Name of this panda -->
-  <xacro:arg name="arm_id" default="panda" />
-  <!-- Should a franka_gripper be mounted at the flange?" -->
-  <xacro:arg name="hand" default="false" />
-  <!-- Is the robot being simulated in gazebo?" -->
-  <xacro:arg name="gazebo" default="false" />
+  <xacro:arg name="arm_id" default="panda" /> <!-- Name of this panda -->
+  <xacro:arg name="hand"   default="false" /> <!-- Should a franka_gripper be mounted at the flange?" -->
+  <xacro:arg name="gazebo" default="false" /> <!-- Is the robot being simulated in gazebo?" -->
+  <xacro:arg name="transmission" default="hardware_interface/EffortJointInterface" /> <!-- The transmission that is used in the gazebo joints -->
+  <xacro:property name="arm_id" value="$(arg arm_id)" />
+  <xacro:property name="transmission" value="$(arg transmission)" />
   <xacro:unless value="$(arg gazebo)">
     <!-- Create a URDF for a real hardware -->
@@ -35,11 +35,11 @@
       <child  link="$(arg arm_id)_link0" />
     </joint>
-    <xacro:gazebo-joint joint="$(arg arm_id)_joint1" transmission="hardware_interface/EffortJointInterface" />
-    <xacro:gazebo-joint joint="$(arg arm_id)_joint2" transmission="hardware_interface/EffortJointInterface" />
-    <xacro:gazebo-joint joint="$(arg arm_id)_joint3" transmission="hardware_interface/EffortJointInterface" />
-    <xacro:gazebo-joint joint="$(arg arm_id)_joint4" transmission="hardware_interface/EffortJointInterface" />
-    <xacro:gazebo-joint joint="$(arg arm_id)_joint5" transmission="hardware_interface/EffortJointInterface" />
-    <xacro:gazebo-joint joint="$(arg arm_id)_joint6" transmission="hardware_interface/EffortJointInterface" />
-    <xacro:gazebo-joint joint="$(arg arm_id)_joint7" transmission="hardware_interface/EffortJointInterface" />
+    <xacro:gazebo-joint joint="${arm_id}_joint1" transmission="${transmission}" />
+    <xacro:gazebo-joint joint="${arm_id}_joint2" transmission="${transmission}" />
+    <xacro:gazebo-joint joint="${arm_id}_joint3" transmission="${transmission}" />
+    <xacro:gazebo-joint joint="${arm_id}_joint4" transmission="${transmission}" />
+    <xacro:gazebo-joint joint="${arm_id}_joint5" transmission="${transmission}" />
+    <xacro:gazebo-joint joint="${arm_id}_joint6" transmission="${transmission}" />
+    <xacro:gazebo-joint joint="${arm_id}_joint7" transmission="${transmission}" />
     <xacro:transmission-franka-state arm_id="$(arg arm_id)" />
     <xacro:transmission-franka-model arm_id="$(arg arm_id)"

Commit message: Simplify use of arguments
No need to declare an intermediate property

File: franka_description/robots/panda_arm.urdf.xacro (robot description, xacro)
@@ -4,12 +4,11 @@
   <xacro:arg name="hand"   default="false" /> <!-- Should a franka_gripper be mounted at the flange?" -->
   <xacro:arg name="gazebo" default="false" /> <!-- Is the robot being simulated in gazebo?" -->
-  <xacro:property name="arm_id" value="$(arg arm_id)" />
   <xacro:unless value="$(arg gazebo)">
     <!-- Create a URDF for a real hardware -->
     <xacro:include filename="$(find franka_description)/robots/panda_arm.xacro" />
-    <xacro:panda_arm arm_id="${arm_id}" safety_distance="0.03"/>
+    <xacro:panda_arm arm_id="$(arg arm_id)" safety_distance="0.03"/>
     <xacro:if value="$(arg hand)">
       <xacro:include filename="$(find franka_description)/robots/hand.xacro"/>
-      <xacro:hand ns="${arm_id}" rpy="0 0 ${-pi/4}" connected_to="${arm_id}_link8" safety_distance="0.03"/>
+      <xacro:hand ns="$(arg arm_id)" rpy="0 0 ${-pi/4}" connected_to="$(arg arm_id)_link8" safety_distance="0.03"/>
     </xacro:if>
   </xacro:unless>
@@ -20,9 +19,9 @@
     <xacro:include filename="$(find franka_description)/robots/utils.xacro" />
     <xacro:include filename="$(find franka_description)/robots/panda_gazebo.xacro" />
-    <xacro:panda_arm arm_id="${arm_id}" />
+    <xacro:panda_arm arm_id="$(arg arm_id)" />
     <xacro:if value="$(arg hand)">
-      <xacro:hand ns="${arm_id}" rpy="0 0 ${-pi/4}" connected_to="${arm_id}_link8" />
-      <xacro:gazebo-joint joint="${arm_id}_finger_joint1" transmission="hardware_interface/EffortJointInterface" />
-      <xacro:gazebo-joint joint="${arm_id}_finger_joint2" transmission="hardware_interface/EffortJointInterface" />
+      <xacro:hand ns="$(arg arm_id)" rpy="0 0 ${-pi/4}" connected_to="$(arg arm_id)_link8" />
+      <xacro:gazebo-joint joint="$(arg arm_id)_finger_joint1" transmission="hardware_interface/EffortJointInterface" />
+      <xacro:gazebo-joint joint="$(arg arm_id)_finger_joint2" transmission="hardware_interface/EffortJointInterface" />
     </xacro:if>
     <!-- Gazebo requires a joint to a link called "world" for statically mounted robots -->
@@ -31,21 +30,21 @@
       <origin xyz="$(arg xyz)" rpy="$(arg rpy)" />
       <parent link="world" />
-      <child  link="${arm_id}_link0" />
+      <child  link="$(arg arm_id)_link0" />
     </joint>
-    <xacro:gazebo-joint joint="${arm_id}_joint1" transmission="hardware_interface/EffortJointInterface" />
-    <xacro:gazebo-joint joint="${arm_id}_joint2" transmission="hardware_interface/EffortJointInterface" />
-    <xacro:gazebo-joint joint="${arm_id}_joint3" transmission="hardware_interface/EffortJointInterface" />
-    <xacro:gazebo-joint joint="${arm_id}_joint4" transmission="hardware_interface/EffortJointInterface" />
-    <xacro:gazebo-joint joint="${arm_id}_joint5" transmission="hardware_interface/EffortJointInterface" />
-    <xacro:gazebo-joint joint="${arm_id}_joint6" transmission="hardware_interface/EffortJointInterface" />
-    <xacro:gazebo-joint joint="${arm_id}_joint7" transmission="hardware_interface/EffortJointInterface" />
-    <xacro:transmission-franka-state arm_id="${arm_id}" />
-    <xacro:transmission-franka-model arm_id="${arm_id}"
-       root="${arm_id}_joint1"
-       tip="${arm_id}_joint8"
+    <xacro:gazebo-joint joint="$(arg arm_id)_joint1" transmission="hardware_interface/EffortJointInterface" />
+    <xacro:gazebo-joint joint="$(arg arm_id)_joint2" transmission="hardware_interface/EffortJointInterface" />
+    <xacro:gazebo-joint joint="$(arg arm_id)_joint3" transmission="hardware_interface/EffortJointInterface" />
+    <xacro:gazebo-joint joint="$(arg arm_id)_joint4" transmission="hardware_interface/EffortJointInterface" />
+    <xacro:gazebo-joint joint="$(arg arm_id)_joint5" transmission="hardware_interface/EffortJointInterface" />
+    <xacro:gazebo-joint joint="$(arg arm_id)_joint6" transmission="hardware_interface/EffortJointInterface" />
+    <xacro:gazebo-joint joint="$(arg arm_id)_joint7" transmission="hardware_interface/EffortJointInterface" />
+    <xacro:transmission-franka-state arm_id="$(arg arm_id)" />
+    <xacro:transmission-franka-model arm_id="$(arg arm_id)"
+       root="$(arg arm_id)_joint1"
+       tip="$(arg arm_id)_joint8"
      />
     <gazebo>
       <plugin name="gazebo_ros_control" filename="libgazebo_ros_control.so">
-        <robotNamespace>${arm_id}</robotNamespace>
+        <robotNamespace>$(arg arm_id)</robotNamespace>
         <controlPeriod>0.001</controlPeriod>
         <robotSimType>franka_gazebo/FrankaHWSim</robotSimType>

Commit message: Allow short transmission argument: position, velocity, or effort
Automatically translate into full name, e.g. hardware_interface/PositionJointInterface

File: franka_description/robots/panda_arm.urdf.xacro (robot description, xacro)
@@ -4,7 +4,7 @@
   <xacro:arg name="hand"   default="false" /> <!-- Should a franka_gripper be mounted at the flange?" -->
   <xacro:arg name="gazebo" default="false" /> <!-- Is the robot being simulated in gazebo?" -->
-  <xacro:arg name="transmission" default="hardware_interface/EffortJointInterface" /> <!-- The transmission that is used in the gazebo joints -->
+  <!-- The transmission type that is used to control arm joints in gazebo: position, velocity, or effort -->
+  <xacro:arg name="transmission" default="effort" />
   <xacro:property name="arm_id" value="$(arg arm_id)" />
-  <xacro:property name="transmission" value="$(arg transmission)" />
   <xacro:unless value="$(arg gazebo)">
     <!-- Create a URDF for a real hardware -->
@@ -35,11 +35,18 @@
       <child  link="$(arg arm_id)_link0" />
     </joint>
-    <xacro:gazebo-joint joint="${arm_id}_joint1" transmission="${transmission}" />
-    <xacro:gazebo-joint joint="${arm_id}_joint2" transmission="${transmission}" />
-    <xacro:gazebo-joint joint="${arm_id}_joint3" transmission="${transmission}" />
-    <xacro:gazebo-joint joint="${arm_id}_joint4" transmission="${transmission}" />
-    <xacro:gazebo-joint joint="${arm_id}_joint5" transmission="${transmission}" />
-    <xacro:gazebo-joint joint="${arm_id}_joint6" transmission="${transmission}" />
-    <xacro:gazebo-joint joint="${arm_id}_joint7" transmission="${transmission}" />
+    <xacro:property name="transmission" value="$(arg transmission)" />
+    <!-- sanity check -->
+    <xacro:if value="${transmission.lower() not in ['position', 'velocity', 'effort']}" >
+      ${xacro.fatal("transmission:=" + transmission + " is not one of position, velocity, or effort")}
+    </xacro:if>
+    <!-- Unify transmission argument into title case and expand to full name -->
+    <xacro:property name="transmission" value="hardware_interface/${transmission.title()}JointInterface" lazy_eval="false" />
+    <xacro:gazebo-joint joint="$(arg arm_id)_joint1" transmission="${transmission}" />
+    <xacro:gazebo-joint joint="$(arg arm_id)_joint2" transmission="${transmission}" />
+    <xacro:gazebo-joint joint="$(arg arm_id)_joint3" transmission="${transmission}" />
+    <xacro:gazebo-joint joint="$(arg arm_id)_joint4" transmission="${transmission}" />
+    <xacro:gazebo-joint joint="$(arg arm_id)_joint5" transmission="${transmission}" />
+    <xacro:gazebo-joint joint="$(arg arm_id)_joint6" transmission="${transmission}" />
+    <xacro:gazebo-joint joint="$(arg arm_id)_joint7" transmission="${transmission}" />
     <xacro:transmission-franka-state arm_id="$(arg arm_id)" />
     <xacro:transmission-franka-model arm_id="$(arg arm_id)"

Commit message: Expose transmission argument in franka_gazebo/panda.launch

File: franka_description/robots/panda_arm.urdf.xacro (robot description, xacro)
@@ -1,10 +1,12 @@
 <?xml version='1.0' encoding='utf-8'?>
 <robot xmlns:xacro="http://www.ros.org/wiki/xacro" name="panda">
-  <xacro:arg name="arm_id" default="panda" /> <!-- Name of this panda -->
-  <xacro:arg name="hand"   default="false" /> <!-- Should a franka_gripper be mounted at the flange?" -->
-  <xacro:arg name="gazebo" default="false" /> <!-- Is the robot being simulated in gazebo?" -->
+  <!-- Name of this panda -->
+  <xacro:arg name="arm_id" default="panda" />
+  <!-- Should a franka_gripper be mounted at the flange?" -->
+  <xacro:arg name="hand" default="false" />
+  <!-- Is the robot being simulated in gazebo?" -->
+  <xacro:arg name="gazebo" default="false" />
   <!-- The transmission type that is used to control arm joints in gazebo: position, velocity, or effort -->
   <xacro:arg name="transmission" default="effort" />
-  <xacro:property name="arm_id" value="$(arg arm_id)" />
   <xacro:unless value="$(arg gazebo)">
     <!-- Create a URDF for a real hardware -->
