Commit message: add all transmission types to panda_arm.urdf.xacro

File: franka_description/robots/panda_arm.urdf.xacro (robot description, xacro)
@@ -7,6 +7,4 @@
   <!-- Is the robot being simulated in gazebo?" -->
   <xacro:arg name="gazebo" default="false" />
-  <!-- The transmission type that is used to control arm joints in gazebo: position, velocity, or effort -->
-  <xacro:arg name="transmission" default="effort" />
   <xacro:unless value="$(arg gazebo)">
     <!-- Create a URDF for a real hardware -->
@@ -37,18 +35,25 @@
       <child  link="$(arg arm_id)_link0" />
     </joint>
-    <xacro:property name="transmission" value="$(arg transmission)" />
-    <!-- sanity check -->
-    <xacro:if value="${transmission.lower() not in ['position', 'velocity', 'effort']}" >
-      ${xacro.fatal("transmission:=" + transmission + " is not one of position, velocity, or effort")}
-    </xacro:if>
-    <!-- Unify transmission argument into title case and expand to full name -->
-    <xacro:property name="transmission" value="hardware_interface/${transmission.title()}JointInterface" lazy_eval="false" />
-    <xacro:gazebo-joint joint="$(arg arm_id)_joint1" transmission="${transmission}" />
-    <xacro:gazebo-joint joint="$(arg arm_id)_joint2" transmission="${transmission}" />
-    <xacro:gazebo-joint joint="$(arg arm_id)_joint3" transmission="${transmission}" />
-    <xacro:gazebo-joint joint="$(arg arm_id)_joint4" transmission="${transmission}" />
-    <xacro:gazebo-joint joint="$(arg arm_id)_joint5" transmission="${transmission}" />
-    <xacro:gazebo-joint joint="$(arg arm_id)_joint6" transmission="${transmission}" />
-    <xacro:gazebo-joint joint="$(arg arm_id)_joint7" transmission="${transmission}" />
+    <xacro:gazebo-joint joint="$(arg arm_id)_joint1" transmission="hardware_interface/PositionJointInterface" />
+    <xacro:gazebo-joint joint="$(arg arm_id)_joint2" transmission="hardware_interface/PositionJointInterface" />
+    <xacro:gazebo-joint joint="$(arg arm_id)_joint3" transmission="hardware_interface/PositionJointInterface" />
+    <xacro:gazebo-joint joint="$(arg arm_id)_joint4" transmission="hardware_interface/PositionJointInterface" />
+    <xacro:gazebo-joint joint="$(arg arm_id)_joint5" transmission="hardware_interface/PositionJointInterface" />
+    <xacro:gazebo-joint joint="$(arg arm_id)_joint6" transmission="hardware_interface/PositionJointInterface" />
+    <xacro:gazebo-joint joint="$(arg arm_id)_joint7" transmission="hardware_interface/PositionJointInterface" />
+    <xacro:gazebo-joint joint="$(arg arm_id)_joint1" transmission="hardware_interface/VelocityJointInterface" />
+    <xacro:gazebo-joint joint="$(arg arm_id)_joint2" transmission="hardware_interface/VelocityJointInterface" />
+    <xacro:gazebo-joint joint="$(arg arm_id)_joint3" transmission="hardware_interface/VelocityJointInterface" />
+    <xacro:gazebo-joint joint="$(arg arm_id)_joint4" transmission="hardware_interface/VelocityJointInterface" />
+    <xacro:gazebo-joint joint="$(arg arm_id)_joint5" transmission="hardware_interface/VelocityJointInterface" />
+    <xacro:gazebo-joint joint="$(arg arm_id)_joint6" transmission="hardware_interface/VelocityJointInterface" />
+    <xacro:gazebo-joint joint="$(arg arm_id)_joint7" transmission="hardware_interface/VelocityJointInterface" />
+    <xacro:gazebo-joint joint="$(arg arm_id)_joint1" transmission="hardware_interface/EffortJointInterface" />
+    <xacro:gazebo-joint joint="$(arg arm_id)_joint2" transmission="hardware_interface/EffortJointInterface" />
+    <xacro:gazebo-joint joint="$(arg arm_id)_joint3" transmission="hardware_interface/EffortJointInterface" />
+    <xacro:gazebo-joint joint="$(arg arm_id)_joint4" transmission="hardware_interface/EffortJointInterface" />
+    <xacro:gazebo-joint joint="$(arg arm_id)_joint5" transmission="hardware_interface/EffortJointInterface" />
+    <xacro:gazebo-joint joint="$(arg arm_id)_joint6" transmission="hardware_interface/EffortJointInterface" />
+    <xacro:gazebo-joint joint="$(arg arm_id)_joint7" transmission="hardware_interface/EffortJointInterface" />
     <xacro:transmission-franka-state arm_id="$(arg arm_id)" />
     <xacro:transmission-franka-model arm_id="$(arg arm_id)"

Commit message: CHANGE: Move inertial property to `util.xacro`
Otherwise you get errors when including `util.xacro` in files which don't have
such a property declared

File: franka_description/robots/panda_arm.urdf.xacro (robot description, xacro)
@@ -7,6 +7,4 @@
   <!-- Is the robot being simulated in gazebo?" -->
   <xacro:arg name="gazebo" default="false" />
-  <!-- Load interial properties. Property is implicitly passed to macros. -->
-  <xacro:property name="inertial" value="${xacro.load_yaml('inertial.yaml')}" />
   <xacro:include filename="utils.xacro" />
   <xacro:include filename="panda_arm.xacro" />

File: franka_description/robots/utils.xacro (robot description, xacro)
@@ -1,4 +1,6 @@
 <?xml version="1.0"?>
 <robot xmlns:xacro="http://www.ros.org/wiki/xacro">
+  <!-- Load interial properties. Property is implicitly passed to macros. -->
+  <xacro:property name="inertial" value="${xacro.load_yaml('inertial.yaml')}" />
   <!-- ============================================================== -->
   <!-- Macro to add an <interial> tag based on yaml-load properties   -->

Commit message: CHANGE: Refactor `<xacro:inertial_props>` to be free of global properties

File: franka_description/robots/panda_arm.urdf.xacro (robot description, xacro)
@@ -9,5 +9,5 @@
   <xacro:include filename="utils.xacro" />
   <xacro:include filename="panda_arm.xacro" />
-  <xacro:panda_arm arm_id="$(arg arm_id)" safety_distance="0.03"/>
+  <xacro:panda_arm arm_id="$(arg arm_id)" safety_distance="0.03" gazebo="$(arg gazebo)"/>
   <xacro:if value="$(arg hand)">
     <xacro:include filename="hand.xacro"/>

File: franka_description/robots/panda_arm.xacro (robot description, xacro)
@@ -4,5 +4,5 @@
   <!-- safety_distance: Minimum safety distance in [m] by which the collision volumes are expanded and which is enforced during robot motions -->
   <!-- arm_id: Namespace of the panda arm. Serves to differentiate between arms in case of multiple instances. -->
-  <xacro:macro name="panda_arm" params="arm_id:='panda' description_pkg:='franka_description' connected_to:='' xyz:='0 0 0' rpy:='0 0 0' safety_distance:=0">
+  <xacro:macro name="panda_arm" params="arm_id:='panda' description_pkg:='franka_description' connected_to:='' xyz:='0 0 0' rpy:='0 0 0' gazebo:=false safety_distance:=0">
     <xacro:unless value="${not connected_to}">
       <joint name="${arm_id}_joint_${connected_to}" type="fixed">
@@ -12,10 +12,10 @@
       </joint>
     </xacro:unless>
-    <xacro:link_with_sc name="link0">
+    <xacro:link_with_sc name="link0" gazebo="${gazebo}">
       <self_collision_geometries>
         <xacro:collision_capsule xyz="-0.075 0 0.06" direction="x" radius="${0.06+safety_distance}" length="0.03" />
       </self_collision_geometries>
     </xacro:link_with_sc>
-    <xacro:link_with_sc name="link1">
+    <xacro:link_with_sc name="link1" gazebo="${gazebo}">
       <self_collision_geometries>
         <xacro:collision_capsule xyz="0 0 -191.5e-3" radius="${0.06+safety_distance}" length="0.283" />
@@ -31,5 +31,5 @@
       <dynamics D="1" K="7000" damping="0.003" friction="0.0" mu_coulomb="0" mu_viscous="16" />
     </joint>
-    <xacro:link_with_sc name="link2">
+    <xacro:link_with_sc name="link2" gazebo="${gazebo}">
       <self_collision_geometries>
         <xacro:collision_capsule xyz="0 0 0" radius="${0.06+safety_distance}" length="0.12" />
@@ -45,5 +45,5 @@
       <dynamics D="1" K="7000" damping="0.003" friction="0.0" mu_coulomb="0" mu_viscous="16" />
     </joint>
-    <xacro:link_with_sc name="link3">
+    <xacro:link_with_sc name="link3" gazebo="${gazebo}">
       <self_collision_geometries>
         <xacro:collision_capsule xyz="0 0 -0.145" radius="${0.06+safety_distance}" length="0.15" />
@@ -59,5 +59,5 @@
       <dynamics D="1" K="7000" damping="0.003" friction="0.0" mu_coulomb="0" mu_viscous="16" />
     </joint>
-    <xacro:link_with_sc name="link4">
+    <xacro:link_with_sc name="link4" gazebo="${gazebo}">
       <self_collision_geometries>
         <xacro:collision_capsule xyz="0 0 0" radius="${0.06+safety_distance}" length="0.12" />
@@ -73,5 +73,5 @@
       <dynamics D="1" K="7000" damping="0.003" friction="0.0" mu_coulomb="0" mu_viscous="16" />
     </joint>
-    <xacro:link_with_sc name="link5">
+    <xacro:link_with_sc name="link5" gazebo="${gazebo}">
       <self_collision_geometries>
         <xacro:collision_capsule xyz="0 0 -0.26"    radius="${0.060+safety_distance}" length="0.10" />
@@ -88,5 +88,5 @@
       <dynamics D="1" K="7000" damping="0.003" friction="0.0" mu_coulomb="0" mu_viscous="16" />
     </joint>
-    <xacro:link_with_sc name="link6">
+    <xacro:link_with_sc name="link6" gazebo="${gazebo}">
       <self_collision_geometries>
         <xacro:collision_capsule xyz="0 0 -0.03" radius="${0.05+safety_distance}" length="0.08" />
@@ -102,5 +102,5 @@
       <dynamics D="1" K="7000" damping="0.003" friction="0.0" mu_coulomb="0" mu_viscous="16" />
     </joint>
-    <xacro:link_with_sc name="link7" rpy="0 0 ${pi/4}">
+    <xacro:link_with_sc name="link7" gazebo="${gazebo}" rpy="0 0 ${pi/4}">
       <self_collision_geometries>
         <xacro:collision_capsule xyz="0 0 0.01" direction="z" radius="${0.04+safety_distance}" length="0.14" />

File: franka_description/robots/utils.xacro (robot description, xacro)
@@ -9,6 +9,5 @@
   <!-- inertial: Dictionary of inertia properties (see inertial.yaml) -->
   <!-- ============================================================== -->
-  <xacro:macro name="inertial_props" params="inertial:=^ name:=^">
-    <xacro:if value="$(arg gazebo)">
+  <xacro:macro name="inertial_props" params="name inertial:=^">
       <xacro:unless value="${name in inertial}">${xacro.warning('No inertia properties defined for: ' + name)}</xacro:unless>
       <xacro:if value="${name in inertial}">
@@ -22,5 +21,4 @@
         </inertial>
       </xacro:if>
-    </xacro:if>
   </xacro:macro>
   <!-- ========================================================== -->
@@ -28,5 +26,5 @@
   <!--  * detailed meshes for environmental collision checking    -->
   <!--  * and coarse geometry models for self-collision checking  -->
-  <!--    (only if 'gazebo' arg is set)                           -->
+  <!--    (only if 'gazebo' param is set)                         -->
   <!--                                                            -->
   <!-- name:  Name of the robot link (without prefix)             -->
@@ -34,5 +32,5 @@
   <!-- self_collision_geometries:  self <collision> models        -->
   <!-- ========================================================== -->
-  <xacro:macro name="link_with_sc" params="name prefix=${arm_id}_ rpy:='0 0 0' **self_collision_geometries">
+  <xacro:macro name="link_with_sc" params="name prefix=${arm_id}_ rpy:='0 0 0' **self_collision_geometries gazebo:=false">
     <!-- sub-link defining detailed meshes for collision with environment -->
     <link name="${prefix}${name}">
@@ -47,9 +45,11 @@
         </geometry>
       </collision>
-      <xacro:inertial_props />
+      <xacro:if value="${gazebo}">
+        <xacro:inertial_props name="${name}" />
+      </xacro:if>
     </link>
     <!-- sub-link defining coarse geometries of real robot's internal self-collision -->
     <link name="${prefix}${name}_sc">
-      <xacro:unless value="$(arg gazebo)">
+      <xacro:unless value="${gazebo}">
         <xacro:insert_block name="self_collision_geometries" />
       </xacro:unless>

Commit message: modifications to urdf panda

File: franka_description/robots/panda_arm.urdf.xacro (robot description, xacro)
@@ -26,4 +26,12 @@
       <xacro:gazebo-joint joint="${arm_id}_finger_joint2" transmission="hardware_interface/EffortJointInterface" />
     </xacro:if>
+    <xacro:include filename="$(find open_vico_cameras)/urdf/realsense_d435.xacro"/>
+    <xacro:realsense_d435 parent="${arm_id}_link8"
+        camera_name_prefix="realsense_d435_camera1"
+        enable_pointCloud="true"
+        align_depth="false"
+        enable_gazebo_plugin="true">
+        <origin xyz="-0.045 0.025 -0.04" rpy="0.0 -1.3 -0.75"/>
+    </xacro:realsense_d435>
     <!-- Gazebo requires a joint to a link called "world" for statically mounted robots -->
     <link name="world" />
@@ -53,4 +61,21 @@
       <self_collide>true</self_collide>
     </gazebo>
+    <gazebo>
+      <plugin name="gazebo_grasp_fix" filename="libgazebo_grasp_fix.so">
+       <arm>
+          <arm_name>panda</arm_name>
+          <palm_link> panda_link7  </palm_link>
+          <gripper_link> panda_leftfinger </gripper_link>
+          <gripper_link> panda_rightfinger </gripper_link>
+        </arm>
+      <forces_angle_tolerance>90</forces_angle_tolerance>
+      <update_rate>4</update_rate>
+      <grip_count_threshold>4</grip_count_threshold>
+      <max_grip_count>8</max_grip_count> <!-- this should be at least double than grip_count_threshold -->
+      <release_tolerance>0.00001</release_tolerance>
+      <disable_collisions_on_attach>false</disable_collisions_on_attach>
+      <contact_topic>_default_topic_</contact_topic>
+      </plugin>
+    </gazebo>
   </xacro:if>
 </robot>
