Commit message: refactor franka_description to support for fr3

File: franka_description/robots/common/franka_arm.xacro (robot description, xacro)
@@ -1,8 +1,9 @@
 <?xml version='1.0' encoding='utf-8'?>
 <robot xmlns:xacro="http://www.ros.org/wiki/xacro" name="panda">
-  <xacro:include filename="utils.xacro" />
+  <xacro:include filename="$(find franka_description)/robots/common/utils.xacro" />
   <!-- safety_distance: Minimum safety distance in [m] by which the collision volumes are expanded and which is enforced during robot motions -->
-  <!-- arm_id: Namespace of the panda arm. Serves to differentiate between arms in case of multiple instances. -->
-  <xacro:macro name="panda_arm" params="arm_id:='panda' description_pkg:='franka_description' connected_to:='' xyz:='0 0 0' rpy:='0 0 0' gazebo:=false safety_distance:=0">
+  <!-- arm_id: Namespace of the robot arm. Serves to differentiate between arms in case of multiple instances. -->
+  <xacro:macro name="franka_arm" params="arm_id:='panda' description_pkg:='franka_description' connected_to:='' xyz:='0 0 0' rpy:='0 0 0' gazebo:=false safety_distance:=0 joint_limits_yaml" >
+    <xacro:property name="joint_limits" value="${xacro.load_yaml(joint_limits_yaml)}"/>
     <xacro:unless value="${not connected_to}">
       <joint name="${arm_id}_joint_${connected_to}" type="fixed">
@@ -23,10 +24,11 @@
     </xacro:link_with_sc>
     <joint name="${arm_id}_joint1" type="revolute">
-      <safety_controller k_position="100.0" k_velocity="40.0" soft_lower_limit="-2.8973" soft_upper_limit="2.8973" />
+      <xacro:property name="limits" value="${joint_limits['joint1']}" lazy_eval="false" />
+      <safety_controller k_position="100.0" k_velocity="40.0" soft_lower_limit="${limits.min_position}" soft_upper_limit="${limits.max_position}" />
       <origin rpy="0 0 0" xyz="0 0 0.333" />
       <parent link="${arm_id}_link0" />
       <child link="${arm_id}_link1" />
       <axis xyz="0 0 1" />
-      <limit effort="87" lower="-2.8973" upper="2.8973" velocity="2.1750" />
+      <limit effort="${limits.max_torque}" lower="${limits.min_position}" upper="${limits.max_position}" velocity="${limits.max_velocity}" />
       <dynamics D="1" K="7000" damping="0.003" friction="0.0" mu_coulomb="0" mu_viscous="16" />
     </joint>
@@ -37,10 +39,11 @@
     </xacro:link_with_sc>
     <joint name="${arm_id}_joint2" type="revolute">
-      <safety_controller k_position="100.0" k_velocity="40.0" soft_lower_limit="-1.7628" soft_upper_limit="1.7628" />
+      <xacro:property name="limits" value="${joint_limits['joint2']}" lazy_eval="false" />
+      <safety_controller k_position="100.0" k_velocity="40.0" soft_lower_limit="${limits.min_position}" soft_upper_limit="${limits.max_position}" />
       <origin rpy="${-pi/2} 0 0" xyz="0 0 0" />
       <parent link="${arm_id}_link1" />
       <child link="${arm_id}_link2" />
       <axis xyz="0 0 1" />
-      <limit effort="87" lower="-1.7628" upper="1.7628" velocity="2.1750" />
+      <limit effort="${limits.max_torque}" lower="${limits.min_position}" upper="${limits.max_position}" velocity="${limits.max_velocity}" />
       <dynamics D="1" K="7000" damping="0.003" friction="0.0" mu_coulomb="0" mu_viscous="16" />
     </joint>
@@ -51,10 +54,11 @@
     </xacro:link_with_sc>
     <joint name="${arm_id}_joint3" type="revolute">
-      <safety_controller k_position="100.0" k_velocity="40.0" soft_lower_limit="-2.8973" soft_upper_limit="2.8973" />
+      <xacro:property name="limits" value="${joint_limits['joint3']}" lazy_eval="false" />
+      <safety_controller k_position="100.0" k_velocity="40.0" soft_lower_limit="${limits.min_position}" soft_upper_limit="${limits.max_position}" />
       <origin rpy="${pi/2} 0 0" xyz="0 -0.316 0" />
       <parent link="${arm_id}_link2" />
       <child link="${arm_id}_link3" />
       <axis xyz="0 0 1" />
-      <limit effort="87" lower="-2.8973" upper="2.8973" velocity="2.1750" />
+     <limit effort="${limits.max_torque}" lower="${limits.min_position}" upper="${limits.max_position}" velocity="${limits.max_velocity}" />
       <dynamics D="1" K="7000" damping="0.003" friction="0.0" mu_coulomb="0" mu_viscous="16" />
     </joint>
@@ -65,10 +69,11 @@
     </xacro:link_with_sc>
     <joint name="${arm_id}_joint4" type="revolute">
-      <safety_controller k_position="100.0" k_velocity="40.0" soft_lower_limit="-3.0718" soft_upper_limit="-0.0698" />
+      <xacro:property name="limits" value="${joint_limits['joint4']}" lazy_eval="false" />
+      <safety_controller k_position="100.0" k_velocity="40.0" soft_lower_limit="${limits.min_position}" soft_upper_limit="${limits.max_position}" />
       <origin rpy="${pi/2} 0 0" xyz="0.0825 0 0" />
       <parent link="${arm_id}_link3" />
       <child link="${arm_id}_link4" />
       <axis xyz="0 0 1" />
-      <limit effort="87" lower="-3.0718" upper="-0.0698" velocity="2.1750" />
+      <limit effort="${limits.max_torque}" lower="${limits.min_position}" upper="${limits.max_position}" velocity="${limits.max_velocity}" />
       <dynamics D="1" K="7000" damping="0.003" friction="0.0" mu_coulomb="0" mu_viscous="16" />
     </joint>
@@ -80,10 +85,11 @@
     </xacro:link_with_sc>
     <joint name="${arm_id}_joint5" type="revolute">
-      <safety_controller k_position="100.0" k_velocity="40.0" soft_lower_limit="-2.8973" soft_upper_limit="2.8973" />
+      <xacro:property name="limits" value="${joint_limits['joint5']}" lazy_eval="false" />
+     <safety_controller k_position="100.0" k_velocity="40.0" soft_lower_limit="${limits.min_position}" soft_upper_limit="${limits.max_position}" />
       <origin rpy="${-pi/2} 0 0" xyz="-0.0825 0.384 0" />
       <parent link="${arm_id}_link4" />
       <child link="${arm_id}_link5" />
       <axis xyz="0 0 1" />
-      <limit effort="12" lower="-2.8973" upper="2.8973" velocity="2.6100" />
+      <limit effort="${limits.max_torque}" lower="${limits.min_position}" upper="${limits.max_position}" velocity="${limits.max_velocity}" />
       <dynamics D="1" K="7000" damping="0.003" friction="0.0" mu_coulomb="0" mu_viscous="16" />
     </joint>
@@ -94,10 +100,11 @@
     </xacro:link_with_sc>
     <joint name="${arm_id}_joint6" type="revolute">
-      <safety_controller k_position="100.0" k_velocity="40.0" soft_lower_limit="-0.0175" soft_upper_limit="3.7525" />
+      <xacro:property name="limits" value="${joint_limits['joint6']}" lazy_eval="false" />
+      <safety_controller k_position="100.0" k_velocity="40.0" soft_lower_limit="${limits.min_position}" soft_upper_limit="${limits.max_position}" />
       <origin rpy="${pi/2} 0 0" xyz="0 0 0" />
       <parent link="${arm_id}_link5" />
       <child link="${arm_id}_link6" />
       <axis xyz="0 0 1" />
-      <limit effort="12" lower="-0.0175" upper="3.7525" velocity="2.6100" />
+     <limit effort="${limits.max_torque}" lower="${limits.min_position}" upper="${limits.max_position}" velocity="${limits.max_velocity}" />
       <dynamics D="1" K="7000" damping="0.003" friction="0.0" mu_coulomb="0" mu_viscous="16" />
     </joint>
@@ -109,10 +116,11 @@
     </xacro:link_with_sc>
     <joint name="${arm_id}_joint7" type="revolute">
-      <safety_controller k_position="100.0" k_velocity="40.0" soft_lower_limit="-2.8973" soft_upper_limit="2.8973"/>
+      <xacro:property name="limits" value="${joint_limits['joint7']}" lazy_eval="false" />
+      <safety_controller k_position="100.0" k_velocity="40.0" soft_lower_limit="${limits.min_position}" soft_upper_limit="${limits.max_position}" />
       <origin rpy="${pi/2} 0 0" xyz="0.088 0 0"/>
       <parent link="${arm_id}_link6"/>
       <child link="${arm_id}_link7"/>
       <axis xyz="0 0 1"/>
-      <limit effort="12" lower="-2.8973" upper="2.8973" velocity="2.6100"/>
+     <limit effort="${limits.max_torque}" lower="${limits.min_position}" upper="${limits.max_position}" velocity="${limits.max_velocity}" />
       <dynamics D="1" K="7000" damping="0.003" friction="0.0" mu_coulomb="0" mu_viscous="16"/>
     </joint>

File: franka_description/robots/common/utils.xacro (robot description, xacro)
@@ -1,9 +1,9 @@
 <?xml version="1.0"?>
 <robot xmlns:xacro="http://www.ros.org/wiki/xacro">
-  <!-- Load interial properties. Property is implicitly passed to macros. -->
-  <xacro:property name="inertial_config" value="$(find franka_description)/robots/inertial.yaml"/>
+  <!-- Load inertial properties. Property is implicitly passed to macros. -->
+  <xacro:property name="inertial_config" value="$(find franka_description)/robots/common/inertial.yaml"/>
   <xacro:property name="inertial" value="${xacro.load_yaml(inertial_config)}"/>
   <!-- ============================================================== -->
-  <!-- Macro to add an <interial> tag based on yaml-load properties   -->
+  <!-- Macro to add an <inertial> tag based on yaml-load properties   -->
   <!--                                                                -->
   <!-- name:     Name of the robot link (without prefix)              -->

Commit message: load joint limits directly in top-level URDf

File: franka_description/robots/common/franka_arm.xacro (robot description, xacro)
@@ -4,6 +4,6 @@
   <!-- safety_distance: Minimum safety distance in [m] by which the collision volumes are expanded and which is enforced during robot motions -->
   <!-- arm_id: Namespace of the robot arm. Serves to differentiate between arms in case of multiple instances. -->
-  <xacro:macro name="franka_arm" params="arm_id:='panda' description_pkg:='franka_description' connected_to:='' xyz:='0 0 0' rpy:='0 0 0' gazebo:=false safety_distance:=0 joint_limits_yaml" >
-    <xacro:property name="joint_limits" value="${xacro.load_yaml(joint_limits_yaml)}"/>
+  <!-- joint_limits: description of the joint limits that comes from a YAML file. Example definition: ${xacro.load_yaml('$(find franka_description)/robots/fr3/joint_limits.yaml')} -->
+  <xacro:macro name="franka_arm" params="arm_id:='panda' description_pkg:='franka_description' connected_to:='' xyz:='0 0 0' rpy:='0 0 0' gazebo:=false safety_distance:=0 joint_limits" >
     <xacro:unless value="${not connected_to}">
       <joint name="${arm_id}_joint_${connected_to}" type="fixed">

File: franka_description/robots/common/franka_robot.xacro (robot description, xacro)
@@ -1,5 +1,5 @@
 <?xml version='1.0' encoding='utf-8'?>
 <robot xmlns:xacro="http://www.ros.org/wiki/xacro">
-  <xacro:macro name="franka_robot" params="name joint_limits_yaml">
+  <xacro:macro name="franka_robot" params="name joint_limits">
     <!-- Name of this panda -->
     <xacro:arg name="arm_id" default="panda" />
@@ -14,5 +14,5 @@
     <xacro:include filename="$(find franka_description)/robots/common/utils.xacro" />
     <xacro:include filename="$(find franka_description)/robots/common/franka_arm.xacro" />
-    <xacro:franka_arm arm_id="$(arg arm_id)" safety_distance="0.03" gazebo="$(arg gazebo)" joint_limits_yaml="${joint_limits_yaml}"/>
+    <xacro:franka_arm arm_id="$(arg arm_id)" safety_distance="0.03" gazebo="$(arg gazebo)" joint_limits="${joint_limits}"/>
     <xacro:if value="$(arg hand)">
       <xacro:include filename="$(find franka_description)/robots/common/franka_hand.xacro"/>

File: franka_description/robots/dual_panda/dual_panda_example.urdf.xacro (robot description, xacro)
@@ -24,8 +24,8 @@
   </link>
   <!-- right arm with gripper -->
-  <xacro:franka_arm arm_id="$(arg arm_id_1)" connected_to="base"  xyz="0 -0.5 1" safety_distance="0.03" joint_limits_yaml="$(find franka_description)/robots/panda/joint_limits.yaml"/>
+  <xacro:franka_arm arm_id="$(arg arm_id_1)" connected_to="base"  xyz="0 -0.5 1" safety_distance="0.03" joint_limits="${xacro.load_yaml('$(find franka_description)/robots/panda/joint_limits.yaml')}"/>
   <xacro:franka_hand arm_id="$(arg arm_id_1)" rpy="0 0 ${-pi/4}" connected_to="$(arg arm_id_1)_link8" safety_distance="0.03"/>
   <!-- left arm with gripper -->
-  <xacro:franka_arm arm_id="$(arg arm_id_2)" connected_to="base"  xyz="0 0.5 1" safety_distance="0.03" joint_limits_yaml="$(find franka_description)/robots/panda/joint_limits.yaml"/>
+  <xacro:franka_arm arm_id="$(arg arm_id_2)" connected_to="base"  xyz="0 0.5 1" safety_distance="0.03" joint_limits="${xacro.load_yaml('$(find franka_description)/robots/panda/joint_limits.yaml')}"/>
   <xacro:franka_hand arm_id="$(arg arm_id_2)" rpy="0 0 ${-pi/4}" connected_to="$(arg arm_id_2)_link8" safety_distance="0.03"/>
 </robot>

File: franka_description/robots/fr3/fr3.urdf.xacro (robot description, xacro)
@@ -2,4 +2,4 @@
 <robot xmlns:xacro="http://www.ros.org/wiki/xacro" name="fr3">
   <xacro:include filename="$(find franka_description)/robots/common/franka_robot.xacro"/>
-  <xacro:franka_robot name="fr3" joint_limits_yaml="$(find franka_description)/robots/fr3/joint_limits.yaml"/>
+  <xacro:franka_robot name="fr3" joint_limits="${xacro.load_yaml('$(find franka_description)/robots/fr3/joint_limits.yaml')}"/>
 </robot>

File: franka_description/robots/panda/panda.urdf.xacro (robot description, xacro)
@@ -2,4 +2,4 @@
 <robot xmlns:xacro="http://www.ros.org/wiki/xacro" name="panda">
   <xacro:include filename="$(find franka_description)/robots/common/franka_robot.xacro"/>
-  <xacro:franka_robot name="panda" joint_limits_yaml="$(find franka_description)/robots/panda/joint_limits.yaml"/>
+  <xacro:franka_robot name="panda" joint_limits="${xacro.load_yaml('$(find franka_description)/robots/panda/joint_limits.yaml')}"/>
 </robot>

Commit message: CHANGE: Extract <limits> & <safety_controller> into custom macro

File: franka_description/robots/common/franka_arm.xacro (robot description, xacro)
@@ -24,11 +24,9 @@
     </xacro:link_with_sc>
     <joint name="${arm_id}_joint1" type="revolute">
-      <xacro:property name="limits" value="${joint_limits['joint1']}" lazy_eval="false" />
-      <safety_controller k_position="100.0" k_velocity="40.0" soft_lower_limit="${limits.min_position}" soft_upper_limit="${limits.max_position}" />
       <origin rpy="0 0 0" xyz="0 0 0.333" />
       <parent link="${arm_id}_link0" />
       <child link="${arm_id}_link1" />
       <axis xyz="0 0 1" />
-      <limit effort="${limits.max_torque}" lower="${limits.min_position}" upper="${limits.max_position}" velocity="${limits.max_velocity}" />
+      <xacro:franka-limits name="joint1" config="${joint_limits}" />
       <dynamics D="1" K="7000" damping="0.003" friction="0.0" mu_coulomb="0" mu_viscous="16" />
     </joint>
@@ -39,11 +37,9 @@
     </xacro:link_with_sc>
     <joint name="${arm_id}_joint2" type="revolute">
-      <xacro:property name="limits" value="${joint_limits['joint2']}" lazy_eval="false" />
-      <safety_controller k_position="100.0" k_velocity="40.0" soft_lower_limit="${limits.min_position}" soft_upper_limit="${limits.max_position}" />
       <origin rpy="${-pi/2} 0 0" xyz="0 0 0" />
       <parent link="${arm_id}_link1" />
       <child link="${arm_id}_link2" />
       <axis xyz="0 0 1" />
-      <limit effort="${limits.max_torque}" lower="${limits.min_position}" upper="${limits.max_position}" velocity="${limits.max_velocity}" />
+      <xacro:franka-limits name="joint2" config="${joint_limits}" />
       <dynamics D="1" K="7000" damping="0.003" friction="0.0" mu_coulomb="0" mu_viscous="16" />
     </joint>
@@ -54,11 +50,9 @@
     </xacro:link_with_sc>
     <joint name="${arm_id}_joint3" type="revolute">
-      <xacro:property name="limits" value="${joint_limits['joint3']}" lazy_eval="false" />
-      <safety_controller k_position="100.0" k_velocity="40.0" soft_lower_limit="${limits.min_position}" soft_upper_limit="${limits.max_position}" />
       <origin rpy="${pi/2} 0 0" xyz="0 -0.316 0" />
       <parent link="${arm_id}_link2" />
       <child link="${arm_id}_link3" />
       <axis xyz="0 0 1" />
-     <limit effort="${limits.max_torque}" lower="${limits.min_position}" upper="${limits.max_position}" velocity="${limits.max_velocity}" />
+      <xacro:franka-limits name="joint3" config="${joint_limits}" />
       <dynamics D="1" K="7000" damping="0.003" friction="0.0" mu_coulomb="0" mu_viscous="16" />
     </joint>
@@ -69,11 +63,9 @@
     </xacro:link_with_sc>
     <joint name="${arm_id}_joint4" type="revolute">
-      <xacro:property name="limits" value="${joint_limits['joint4']}" lazy_eval="false" />
-      <safety_controller k_position="100.0" k_velocity="40.0" soft_lower_limit="${limits.min_position}" soft_upper_limit="${limits.max_position}" />
       <origin rpy="${pi/2} 0 0" xyz="0.0825 0 0" />
       <parent link="${arm_id}_link3" />
       <child link="${arm_id}_link4" />
       <axis xyz="0 0 1" />
-      <limit effort="${limits.max_torque}" lower="${limits.min_position}" upper="${limits.max_position}" velocity="${limits.max_velocity}" />
+      <xacro:franka-limits name="joint4" config="${joint_limits}" />
       <dynamics D="1" K="7000" damping="0.003" friction="0.0" mu_coulomb="0" mu_viscous="16" />
     </joint>
@@ -85,11 +77,9 @@
     </xacro:link_with_sc>
     <joint name="${arm_id}_joint5" type="revolute">
-      <xacro:property name="limits" value="${joint_limits['joint5']}" lazy_eval="false" />
-     <safety_controller k_position="100.0" k_velocity="40.0" soft_lower_limit="${limits.min_position}" soft_upper_limit="${limits.max_position}" />
       <origin rpy="${-pi/2} 0 0" xyz="-0.0825 0.384 0" />
       <parent link="${arm_id}_link4" />
       <child link="${arm_id}_link5" />
       <axis xyz="0 0 1" />
-      <limit effort="${limits.max_torque}" lower="${limits.min_position}" upper="${limits.max_position}" velocity="${limits.max_velocity}" />
+      <xacro:franka-limits name="joint5" config="${joint_limits}" />
       <dynamics D="1" K="7000" damping="0.003" friction="0.0" mu_coulomb="0" mu_viscous="16" />
     </joint>
@@ -100,11 +90,9 @@
     </xacro:link_with_sc>
     <joint name="${arm_id}_joint6" type="revolute">
-      <xacro:property name="limits" value="${joint_limits['joint6']}" lazy_eval="false" />
-      <safety_controller k_position="100.0" k_velocity="40.0" soft_lower_limit="${limits.min_position}" soft_upper_limit="${limits.max_position}" />
       <origin rpy="${pi/2} 0 0" xyz="0 0 0" />
       <parent link="${arm_id}_link5" />
       <child link="${arm_id}_link6" />
       <axis xyz="0 0 1" />
-     <limit effort="${limits.max_torque}" lower="${limits.min_position}" upper="${limits.max_position}" velocity="${limits.max_velocity}" />
+      <xacro:franka-limits name="joint6" config="${joint_limits}" />
       <dynamics D="1" K="7000" damping="0.003" friction="0.0" mu_coulomb="0" mu_viscous="16" />
     </joint>
@@ -116,11 +104,9 @@
     </xacro:link_with_sc>
     <joint name="${arm_id}_joint7" type="revolute">
-      <xacro:property name="limits" value="${joint_limits['joint7']}" lazy_eval="false" />
-      <safety_controller k_position="100.0" k_velocity="40.0" soft_lower_limit="${limits.min_position}" soft_upper_limit="${limits.max_position}" />
       <origin rpy="${pi/2} 0 0" xyz="0.088 0 0"/>
       <parent link="${arm_id}_link6"/>
       <child link="${arm_id}_link7"/>
       <axis xyz="0 0 1"/>
-     <limit effort="${limits.max_torque}" lower="${limits.min_position}" upper="${limits.max_position}" velocity="${limits.max_velocity}" />
+      <xacro:franka-limits name="joint7" config="${joint_limits}" />
       <dynamics D="1" K="7000" damping="0.003" friction="0.0" mu_coulomb="0" mu_viscous="16"/>
     </joint>

File: franka_description/robots/common/utils.xacro (robot description, xacro)
@@ -206,3 +206,21 @@
     </inertial>
   </xacro:macro>
+  <!-- ========================================================================= -->
+  <!-- Adds the <limit ... /> & <safety_controller/> tags given a config file    -->
+  <!-- of joint limits                                                           -->
+  <!--                                                                           -->
+  <!-- config - YAML struct defining joint limits (e.g. panda/joint_limits.yaml) -->
+  <!-- name   - Name of the joint for which to add limits to                     -->
+  <!-- ========================================================================= -->
+  <xacro:macro name="franka-limits" params="config name">
+      <xacro:property name="limits" value="${config[name]['limit']}" lazy_eval="false" />
+      <limit lower="${limits.lower}"
+             upper="${limits.upper}"
+             effort="${limits.effort}"
+             velocity="${limits.velocity}" />
+      <safety_controller k_position="100.0"
+                         k_velocity="40.0"
+                         soft_lower_limit="${limits.lower}"
+                         soft_upper_limit="${limits.upper}" />
+  </xacro:macro>
 </robot>

Commit message: adding link9 to franka_arm urdf

File: franka_description/robots/common/franka_arm.xacro (robot description, xacro)
@@ -117,4 +117,10 @@
       <child link="${arm_id}_link8"/>
     </joint>
+    <link name="${arm_id}_link9"/>
+    <joint name="${arm_id}_link9_joint" type="fixed">
+      <origin xyz="0 0 0.103" rpy="0 0 0" />
+      <parent link="${arm_id}_link8" />
+      <child link="${arm_id}_link9" />
+    </joint>
   </xacro:macro>
 </robot>
