Commit message: add end-fingertips-changes-only-to-noetic-devel

File: franka_description/robots/common/franka_hand.xacro (robot description, xacro)
@@ -29,4 +29,21 @@
         </geometry>
       </visual>
+      <!-- end left-fingertip -->
+      <visual>
+        <origin xyz="0 0.0015 0.06" rpy="0 0 0" />
+        <geometry>
+          <box size="0.018 0.003 0.015"/>
+        </geometry>
+        <material name="Grey">
+          <color rgba="0.262 0.262 0.262 1"/>
+        </material>
+      </visual>
+      <!-- end left-fingertip collision -->
+      <collision>
+        <origin xyz="0 0.0015 0.06" rpy="0 0 0" />
+        <geometry>
+          <box size="0.018 0.003 0.015" />
+        </geometry>
+      </collision>
       <!-- screw mount -->
       <collision>
@@ -68,4 +85,21 @@
         </geometry>
       </visual>
+      <!-- end right-fingertip -->
+      <visual>
+        <origin xyz="0 -0.0015 0.06" rpy="0 0 0" />
+        <geometry>
+          <box size="0.018 0.003 0.015"/>
+        </geometry>
+        <material name="Grey">
+          <color rgba="0.262 0.262 0.262 1"/>
+        </material>
+      </visual>
+      <!-- end left-fingertip collision -->
+      <collision>
+        <origin xyz="0 -0.0015 0.06" rpy="0 0 0" />
+        <geometry>
+          <box size="0.018 0.003 0.015" />
+        </geometry>
+      </collision>
       <!-- screw mount -->
       <collision>
