Commit message: allow selecting fr3 urdf for launch files

File: franka_description/robots/common/franka_robot.xacro (robot description, xacro)
@@ -1,7 +1,7 @@
 <?xml version='1.0' encoding='utf-8'?>
 <robot xmlns:xacro="http://www.ros.org/wiki/xacro">
-  <xacro:macro name="franka_robot" params="name joint_limits">
+  <xacro:macro name="franka_robot" params="arm_id joint_limits">
     <!-- Name of this panda -->
-    <xacro:arg name="arm_id" default="panda" />
+    <xacro:arg name="arm_id" default="${arm_id}" />
     <!-- Should a franka_gripper be mounted at the flange?" -->
     <xacro:arg name="hand" default="false" />

File: franka_description/robots/fr3/fr3.urdf.xacro (robot description, xacro)
@@ -2,4 +2,4 @@
 <robot xmlns:xacro="http://www.ros.org/wiki/xacro" name="fr3">
   <xacro:include filename="$(find franka_description)/robots/common/franka_robot.xacro"/>
-  <xacro:franka_robot name="fr3" joint_limits="${xacro.load_yaml('$(find franka_description)/robots/fr3/joint_limits.yaml')}"/>
+  <xacro:franka_robot arm_id="fr3" joint_limits="${xacro.load_yaml('$(find franka_description)/robots/fr3/joint_limits.yaml')}"/>
 </robot>

File: franka_description/robots/panda/panda.urdf.xacro (robot description, xacro)
@@ -2,4 +2,4 @@
 <robot xmlns:xacro="http://www.ros.org/wiki/xacro" name="panda">
   <xacro:include filename="$(find franka_description)/robots/common/franka_robot.xacro"/>
-  <xacro:franka_robot name="panda" joint_limits="${xacro.load_yaml('$(find franka_description)/robots/panda/joint_limits.yaml')}"/>
+  <xacro:franka_robot arm_id="panda" joint_limits="${xacro.load_yaml('$(find franka_description)/robots/panda/joint_limits.yaml')}"/>
 </robot>

Commit message: ADD: `parent` + `{xyz,rpy}` params to franka_robot.xacro
These can be used if you want to simulate the robot on a mobile base. In these
cases the `$(arm_id)_link0` must not be connected to `world` but instead fixed
to a link on the mobile robot instead. You could generate a custom combined
platform + arm URDF like so:

```xml
<robot>
  <xacro:include filename="$(find franka_description)/robots/common/franka_robot.xacro"/>

  <!-- Instantiate a mobile robot here, which defines a "base_link" -->

  <xacro:franka_robot
         robot="fr3"
         parent="base_link"
         xyz="0 0 0.25"
         rpy="0 0 ${pi/2}">
  </xacro:franka_robot>

</robot>
```

File: franka_description/robots/common/franka_robot.xacro (robot description, xacro)
@@ -1,40 +1,33 @@
 <?xml version='1.0' encoding='utf-8'?>
 <robot xmlns:xacro="http://www.ros.org/wiki/xacro">
-  <xacro:macro name="franka_robot" params="arm_id joint_limits">
-    <!-- Name of this panda -->
-    <!-- Should a franka_gripper be mounted at the flange?" -->
-    <xacro:arg name="hand" default="false" />
-    <!-- Positional offset between $(arm_id)_hand -> $(arm_id)_hand_tcp [m]. Only used when hand:=true -->
-    <xacro:arg name="tcp_xyz" default="0 0 0.1034" />
-    <!-- Rotational offset between $(arm_id)_hand -> $(arm_id)_hand_tcp [rad]. Only used when hand:=true -->
-    <xacro:arg name="tcp_rpy" default="0 0 0" />
-    <!-- Is the robot being simulated in gazebo?" -->
-    <xacro:arg name="gazebo" default="false" />
+  <xacro:macro name="franka_robot" params="arm_id joint_limits parent:='world' xyz:='0 0 0' rpy:='0 0 0' hand:=false gazebo:=false tcp_xyz:='0 0 0.1034' tcp_rpy='0 0 0'">
     <xacro:include filename="$(find franka_description)/robots/common/utils.xacro" />
     <xacro:include filename="$(find franka_description)/robots/common/franka_arm.xacro" />
-    <xacro:franka_arm arm_id="${arm_id}" safety_distance="0.03" gazebo="$(arg gazebo)" joint_limits="${joint_limits}"/>
-    <xacro:if value="$(arg hand)">
+    <xacro:franka_arm arm_id="${arm_id}" safety_distance="0.03" gazebo="${gazebo}" joint_limits="${joint_limits}"/>
+    <xacro:if value="${hand}">
       <xacro:include filename="$(find franka_description)/robots/common/franka_hand.xacro"/>
       <xacro:franka_hand
-          arm_id="$(arg arm_id)"
+          arm_id="${arm_id}"
           rpy="0 0 ${-pi/4}"
-          tcp_xyz="$(arg tcp_xyz)"
-          tcp_rpy="$(arg tcp_rpy)"
-          connected_to="$(arg arm_id)_link8"
+          tcp_xyz="${tcp_xyz}"
+          tcp_rpy="${tcp_rpy}"
+          connected_to="${arm_id}_link8"
           safety_distance="0.03"
-          gazebo="$(arg gazebo)"
+          gazebo="${gazebo}"
        />
     </xacro:if>
     <!-- Define additional Gazebo tags -->
-    <xacro:if value="$(arg gazebo)">
-      <xacro:arg name="xyz" default="0 0 0" />
-      <xacro:arg name="rpy" default="0 0 0" />
-      <!-- Gazebo requires a joint to a link called "world" for statically mounted robots -->
-      <link name="world" />
-      <joint name="world_joint" type="fixed">
-        <origin xyz="$(arg xyz)" rpy="$(arg rpy)" />
-        <parent link="world" />
-        <child  link="$(arg arm_id)_link0" />
-      </joint>
+    <xacro:if value="${gazebo}">
+      <xacro:if value="${parent != ''}">
+        <!-- Gazebo requires a joint to a link called "world" for statically mounted robots -->
+        <xacro:if value="${parent == 'world'}">
+          <link name="${parent}" />
+        </xacro:if>
+        <joint name="${parent}_joint" type="fixed">
+          <origin xyz="${xyz}" rpy="${rpy}" />
+          <parent link="${parent}" />
+          <child  link="${arm_id}_link0" />
+        </joint>
+      </xacro:if>
       <xacro:gazebo-joint joint="${arm_id}_joint1" transmission="hardware_interface/PositionJointInterface" />
       <xacro:gazebo-joint joint="${arm_id}_joint2" transmission="hardware_interface/PositionJointInterface" />
